Commit message: try to add obstacles

File: src/first_robot/description/lidar_2d_camera.xacro (robot description, xacro)
@@ -1,45 +1,36 @@
 <?xml version="1.0"?>
-<robot xmlns:xacro="http://www.ros.org/wiki/xacro" name="robot">
-    <joint name="laser joint" type="fixed">
-        <parent link="chassis" />
-        <child link="laser_frame" />
-        <origin xyz="0.1 0 0.175" rpy="0 0 0" />
+<robot xmlns:xacro="http://www.ros.org/wiki/xacro" >
+    <joint name="laser_joint" type="fixed">
+        <parent link="chassis"/>
+        <child link="laser_frame"/>
+        <origin xyz="0.1 0 0.175" rpy="0 0 0"/>
     </joint>
     <link name="laser_frame">
         <visual>
             <geometry>
-                <cylinder radius="0.05" length="0.04" />
+                <cylinder radius="0.05" length="0.04"/>
             </geometry>
-            <material name="orange" />
-        </visual>
-        <visual>
-            <origin xyz="0 0 -0.05" />
-            <geometry>
-                <cylinder radius="0.01" length="0.1" />
-            </geometry>
-            <material name="orange" />
+            <material name="red"/>
         </visual>
         <collision>
             <geometry>
-                <cylinder radius="0.05" length="0.04" />
+                <cylinder radius="0.05" length="0.04"/>
             </geometry>
         </collision>
         <xacro:inertial_cylinder mass="0.1" length="0.04" radius="0.05">
-            <origin xyz="0 0 0" rpy="0 0 0" />
+            <origin xyz="0 0 0" rpy="0 0 0"/>
         </xacro:inertial_cylinder>
     </link>
     <gazebo reference="laser_frame">
-        <material>Gazebo/Black</material>
-        <sensor name="lidar" type="gpu_lidar">
-            <always_on>true</always_on>
+        <material>Gazebo/Red</material>
+        <sensor name="gpu_lidar" type="gpu_lidar">
+            <pose>0 0 0 0 0 0</pose>
             <update_rate>30</update_rate>
             <visualize>true</visualize>
-            <pose>0 0 0 0 0 0</pose>
-            <topic>/lidar_scan</topic>
+            <topic>scan</topic>
             <ray>
                 <scan>
                     <horizontal>
                         <samples>360</samples>
-                        <resolution>1</resolution>
                         <min_angle>-3.14</min_angle>
                         <max_angle>3.14</max_angle>
@@ -47,12 +38,7 @@
                 </scan>
                 <range>
-                    <min>0.1</min>
-                    <max>10.0</max>
+                    <min>0.3</min>
+                    <max>12</max>
                 </range>
-                <noise>
-                    <type>gaussian</type>
-                    <mean>0.0</mean>
-                    <stddev>0.01</stddev>
-                </noise>
             </ray>
         </sensor>

File: src/first_robot/description/robot_core.xacro (robot description, xacro)
@@ -13,4 +13,7 @@
     <material name="black">
         <color rgba="0 0 0 1" />
+    </material>
+    <material name="red">
+        <color rgba="1 0 0 1"/>
     </material>
     <!-- BASE LINK -->
