Commit message: update st

File: src/first_robot/description/robot_core.xacro (robot description, xacro)
@@ -46,4 +46,5 @@
     <!-- LEFT WHEEL LINK -->
     <joint name="left_wheel_joint" type="continuous">
+        <dynamics damping="0.5"/>
         <hardwareInterface>hardware_interface/velocity</hardwareInterface>
         <parent link="base_link" />
@@ -70,4 +71,5 @@
     <!-- RIGHT WHEEL LINK -->
     <joint name="right_wheel_joint" type="continuous">
+        <dynamics damping="0.5"/>
         <hardwareInterface>hardware_interface/velocity</hardwareInterface>
         <parent link="base_link" />
@@ -117,5 +119,5 @@
         <type>transmission_interface/SimpleTransmission</type>
         <actuator name="left_wheel_motor">
-            <mechanicalReduction>1</mechanicalReduction>
+            <mechanicalReduction>3</mechanicalReduction>
         </actuator>
         <joint name="left_wheel_joint" />
@@ -124,5 +126,5 @@
         <type>transmission_interface/SimpleTransmission</type>
         <actuator name="right_wheel_motor">
-            <mechanicalReduction>1</mechanicalReduction>
+            <mechanicalReduction>3</mechanicalReduction>
         </actuator>
         <joint name="right_wheel_joint" />
