Commit message: add mobilenet ssd

File: src/first_robot/description/depth_camera.xacro (robot description, xacro)
@@ -6,4 +6,10 @@
         <origin xyz="0.305 0 0.08" rpy="0 0 0" />
     </joint>
+    <joint name="camera_optical_joint" type="fixed">
+        <parent link="camera_link" />
+        <child link="camera_link_optical" />
+        <origin xyz="0 0 0" rpy="${-pi/2} 0 ${-pi/2}" />
+    </joint>
+    <link name="camera_link_optical"></link>
     <link name="camera_link">
         <visual>
@@ -14,26 +20,19 @@
         </visual>
     </link>
-    <joint name="camera_optical_joint" type="fixed">
-        <parent link="camera_link" />
-        <child link="camera_link_optical" />
-        <origin xyz="0 0 0" rpy="${-pi/2} 0 ${-pi/2}" />
-    </joint>
-    <link name="camera_link_optical"></link>
     <gazebo reference="camera_link">
         <material>Gazebo/Red</material>
-        <sensor name="camera" type="depth">
-            <pose> 0 0 0 0 0 0 </pose>
+        <sensor name="depth_camera" type="depth">
+            <always_on>true</always_on>
+            <update_rate>30</update_rate>
             <visualize>true</visualize>
-            <update_rate>10</update_rate>
             <camera>
-                <horizontal_fov>1.089</horizontal_fov>
+                <horizontal_fov>1.047</horizontal_fov>
                 <image>
-                    <format>B8G8R8</format>
-                    <width>640</width>
-                    <height>480</height>
+                    <width>320</width>
+                    <height>240</height>
                 </image>
                 <clip>
-                    <near>0.05</near>
-                    <far>8.0</far>
+                    <near>0.1</near>
+                    <far>100</far>
                 </clip>
             </camera>
@@ -41,11 +40,11 @@
             <update_rate>30</update_rate>
             <visualize>true</visualize>
-            <topic>camera</topic>
-            <plugin name="camera_controller" filename="libgazebo_ros_camera.so">
-                <camera_name>camera</camera_name>
-                <image_topic_name>image_raw</image_topic_name>
-                <camera_info_topic_name>camera_info</camera_info_topic_name>
-                <frame_name>camera_link</frame_name>
-            </plugin>
+            <topic>depth_camera</topic>
+            <!-- <plugin
+                filename="RosGzPointCloud"
+                name="ros_gz_point_cloud::PointCloud">
+                <topic>points</topic>
+                <frame_id>map</frame_id>
+            </plugin> -->
         </sensor>
     </gazebo>

File: src/first_robot/description/robot.urdf.xacro (robot description, xacro)
@@ -6,5 +6,5 @@
     <xacro:include filename="gz_control.xacro" />
     <xacro:include filename="lidar_2d_camera.xacro" />
-    <xacro:include filename="camera.xacro" />
-    <!-- <xacro:include filename="depth_camera.xacro" /> -->
+    <!-- <xacro:include filename="camera.xacro" /> -->
+    <xacro:include filename="depth_camera.xacro" />
 </robot>
