Commit message: try to add champ

File: src/first_robot/description/imu_link.xacro (robot description, xacro)
@@ -15,14 +15,26 @@
     </joint>
     <gazebo reference="imu_link">
-    <sensor name="imu_sensor" type="imu">
-        <always_on>true</always_on>
-        <update_rate>100</update_rate>
-        <topic>imu/data</topic>
-        <plugin name="gz::sim::systems::Imu" filename="gz-sim-imu-system">
-        <ros>
-            <namespace>/</namespace>
-        </ros>
-        </plugin>
-    </sensor>
+        <sensor name="imu_sensor" type="imu">
+            <always_on>true</always_on>
+            <update_rate>200</update_rate>
+            <topic>imu/data</topic>
+            <plugin name="gz::sim::systems::Imu" filename="gz-sim-imu-system">
+                <ros>
+                    <namespace>/</namespace>
+                </ros>
+            </plugin>
+            <imu>
+                <noise type="gaussian">
+                    <rate>
+                        <mean>0.0</mean>
+                        <stddev>0.005</stddev>                        <!-- Giảm nhiễu -->
+                    </rate>
+                    <accel>
+                        <mean>0.0</mean>
+                        <stddev>0.005</stddev>
+                    </accel>
+                </noise>
+            </imu>
+        </sensor>
     </gazebo>
 </robot>

File: src/first_robot/description/leg_macro.xacro (robot description, xacro)
@@ -32,5 +32,5 @@
         </geometry>
       </collision>
-      <xacro:inertial_box mass="0.2" box_size="${[radius*2, radius*2, length]}" />
+      <xacro:inertial_box mass="0.5" box_size="${[radius*2, radius*2, length]}" />
     </link>
     <joint name="${joint_name}" type="continuous">

File: src/first_robot/description/robot.urdf.xacro (robot description, xacro)
@@ -7,5 +7,5 @@
     <!-- <xacro:include filename="robot_core_ver_four_wheel.xacro" /> -->
     <!-- ROBOT DOG  -->
-    <xacro:include filename="robot_core_ver_snipdog.xacro" />
+    <xacro:include filename="robot_core.xacro" />
     <xacro:include filename="gz_control_snipdog.xacro" />
     <xacro:include filename="lidar_2d_camera.xacro" />

File: src/first_robot/description/robot_core.xacro (robot description, xacro)
@@ -20,5 +20,11 @@
     </material>
     <!-- BASE LINK -->
-    <link name="base_link"></link>
+    <link name="base_link">
+        <inertial>
+        <mass value="0.5"/> <!-- Giảm từ 2.0 -->
+        <origin xyz="0 0 0.1"/>
+        <inertia ixx="0.1" iyy="0.1" izz="0.1" ixy="0" ixz="0" iyz="0"/>
+    </inertial>
+    </link>
     <!-- CHASSIS LINK -->
     <joint name="chassis_joint" type="fixed">
