Commit message: update

File: src/first_robot/description/robot.urdf.xacro (robot description, xacro)
@@ -1,14 +1,11 @@
 <?xml version="1.0"?>
 <robot xmlns:xacro="http://www.ros.org/wiki/xacro" name="my_robot">
-   <!-- need to compose all to single file? run: xacro first_robot/description/robot.urdf.xacro > robot.urdf -->
     <xacro:arg name="prefix" default="" />
     <xacro:arg name="use_mock_hardware" default="true" />
     <xacro:include filename="inertial_base.xacro" />
-    <!-- ROBOT DOG  -->
     <xacro:include filename="robot_core.xacro" />
     <xacro:include filename="gz_control.xacro" />
-    <xacro:include filename="lidar_2d_camera.xacro" />
+    <!-- <xacro:include filename="lidar_2d_camera.xacro" />
     <xacro:include filename="camera.xacro" />
-    <!-- <xacro:include filename="depth_camera.xacro" /> -->
-    <xacro:include filename="imu_link.xacro" />
+    <xacro:include filename="imu_link.xacro" /> -->
 </robot>

File: src/first_robot/description/robot_core.xacro (robot description, xacro)
@@ -51,5 +51,4 @@
         </xacro:inertial_box>
     </link>
-    <!-- FL (Front Left) LEG -->
     <!-- IMPORT LEG PATTERN -->
     <xacro:include filename="$(find first_robot)/description/leg_block.xacro"/>

File: src/robot.urdf (robot description, URDF)
Before this commit: robot my_robot, 31 links, 30 joints
Links:
- removed link camera_link
- removed link camera_link_optical
- removed link imu_link
- removed link lidar_link
Joints:
- removed joint camera_joint
- removed joint camera_optical_joint
- removed joint imu_joint
- removed joint laser_joint
