Commit message: improve urdf

File: src/first_robot/description/leg_block.xacro (robot description, xacro)
@@ -17,5 +17,5 @@
   <link name="${prefix}_hip_motor_link">
     <visual>
-      <origin xyz="0 0 0.02"/>
+      <origin xyz="0 0 0.005"/>
       <geometry>
         <cylinder length="0.02" radius="0.015"/>
@@ -24,5 +24,5 @@
     </visual>
     <collision>
-      <origin xyz="0 0 0.02"/>
+      <origin xyz="0 0 0.005"/>
       <geometry>
         <cylinder length="0.02" radius="0.015"/>
@@ -38,5 +38,5 @@
     <parent link="chassis"/>
     <child link="${prefix}_hip_motor_link"/>
-    <origin xyz="${x} ${y} 0.075"/>
+    <origin xyz="${x} ${y} -0.005"/>
   </joint>
   <!-- Hip Joint -->
@@ -46,22 +46,22 @@
     <origin xyz="0 0 0"/>
     <axis xyz="0 1 0"/>
-    <limit effort="5" velocity="2.0" lower="-1.57" upper="1.57"/>
+    <limit effort="5" velocity="2.0" lower="1.57" upper="-1.57"/><!-- Đảo dấu -->
   </joint>
   <!-- Thigh Link -->
   <link name="${prefix}_thigh">
     <visual>
-      <origin xyz="0 0 -0.075"/>
+      <origin xyz="0 0 -0.06"/>
       <geometry>
-        <box size="0.05 0.05 0.15"/>
+        <box size="0.03 0.03 0.12"/> <!-- Giảm kích thước -->
       </geometry>
       <material name="blue"/>
     </visual>
     <collision>
-      <origin xyz="0 0 -0.075"/>
+      <origin xyz="0 0 -0.06"/>
       <geometry>
-        <box size="0.05 0.05 0.15"/>
+        <box size="0.03 0.03 0.12"/>
       </geometry>
     </collision>
-    <xacro:inertial_box_leg mass="0.2" box_size="${[0.05, 0.05, 0.15]}"/>
+    <xacro:inertial_box_leg mass="0.1" box_size="${[0.03, 0.03, 0.12]}"/> <!-- Giảm khối lượng -->
   </link>
   <!-- Knee Motor Link -->
@@ -89,5 +89,5 @@
     <parent link="${prefix}_thigh"/>
     <child link="${prefix}_knee_motor_link"/>
-    <origin xyz="0 0 -0.15"/>
+    <origin xyz="0 0 -0.12" rpy="0 0.3 0"/> <!-- Thêm góc nghiêng -->
   </joint>
   <!-- Knee Joint -->
@@ -97,22 +97,22 @@
     <origin xyz="0 0 0"/>
     <axis xyz="0 1 0"/>
-    <limit effort="5" velocity="2.0" lower="-1.57" upper="1.57"/>
+    <limit effort="5" velocity="2.0" lower="-2.0" upper="2.0"/> <!-- Mở rộng góc -->
   </joint>
   <!-- Shank Link -->
   <link name="${prefix}_shank">
     <visual>
-      <origin xyz="0 0 -0.075"/>
+      <origin xyz="0 0 -0.06"/>
       <geometry>
-        <box size="0.04 0.04 0.15"/>
+        <box size="0.02 0.02 0.12"/> <!-- Giảm kích thước -->
       </geometry>
       <material name="red"/>
     </visual>
     <collision>
-      <origin xyz="0 0 -0.075"/>
+      <origin xyz="0 0 -0.06"/>
       <geometry>
-        <box size="0.04 0.04 0.15"/>
+        <box size="0.02 0.02 0.12"/>
       </geometry>
     </collision>
-    <xacro:inertial_box_leg mass="0.2" box_size="${[0.04, 0.04, 0.15]}"/>
+    <xacro:inertial_box_leg mass="0.1" box_size="${[0.02, 0.02, 0.12]}"/> <!-- Giảm khối lượng -->
   </link>
   <!-- Ankle Motor Link -->
@@ -140,5 +140,5 @@
     <parent link="${prefix}_shank"/>
     <child link="${prefix}_ankle_motor_link"/>
-    <origin xyz="0 0 -0.15"/>
+    <origin xyz="0 0 -0.12" rpy="0 0.3 0"/> <!-- Thêm góc nghiêng -->
   </joint>
   <!-- Ankle Joint -->
@@ -148,5 +148,5 @@
     <origin xyz="0 0 0"/>
     <axis xyz="0 1 0"/>
-    <limit effort="5" velocity="2.0" lower="-1.57" upper="1.57"/>
+    <limit effort="5" velocity="2.0" lower="-2.0" upper="2.0"/> <!-- Mở rộng góc -->
   </joint>
   <!-- Foot Link -->
@@ -167,4 +167,8 @@
     </xacro:inertial_sphere>
   </link>
+  <gazebo reference="${prefix}_foot">
+    <mu1>1.2</mu1> <!-- Tăng ma sát ngang -->
+    <mu2>1.2</mu2> <!-- Tăng ma sát dọc -->
+  </gazebo>
   <!-- IMPORT LEG PATTERN -->
   <xacro:include filename="$(find first_robot)/description/transmission_block.xacro"/>

File: src/first_robot/description/robot_core.xacro (robot description, xacro)
@@ -42,5 +42,5 @@
         </visual>
         <collision>
-            <origin xyz="0.15 0 0.075" />
+            <origin xyz="0 0 0.075" /> <!-- Sửa tâm va chạm -->
             <geometry>
                 <box size="0.5 0.2 0.15" />

Commit message: temp

File: src/first_robot/description/leg_block.xacro (robot description, xacro)
@@ -108,5 +108,5 @@
       <origin xyz="0 0 0" />
       <axis xyz="0 1 0" /> <!-- Rotation around y axis -->
-      <limit effort="5" velocity="2.0" lower="-2.5" upper="0" /> <!-- Forward motion only -->
+      <limit effort="5" velocity="2.0" lower="-2.8" upper="0" /> <!-- Forward motion only -->
     </joint>
     <!-- Shank link  Box-shaped link connecting knee to ankle -->

File: src/first_robot/description/robot_core.xacro (robot description, xacro)
@@ -22,8 +22,8 @@
     <link name="base_link">
         <inertial>
-        <mass value="0.5"/> <!-- Giảm từ 2.0 -->
-        <origin xyz="0 0 0.1"/>
-        <inertia ixx="0.1" iyy="0.1" izz="0.1" ixy="0" ixz="0" iyz="0"/>
-    </inertial>
+            <mass value="0.25" /> <!-- Giảm từ 2.0 -->
+            <origin xyz="0 0 0.1" />
+            <inertia ixx="0.1" iyy="0.1" izz="0.1" ixy="0" ixz="0" iyz="0" />
+        </inertial>
     </link>
     <!-- CHASSIS LINK -->
@@ -31,5 +31,5 @@
         <parent link="base_link" />
         <child link="chassis" />
-         <origin xyz="0 0 0" />
+        <origin xyz="0 0 0" />
     </joint>
     <link name="chassis">
@@ -37,5 +37,5 @@
             <origin xyz="0 0 0.075" />
             <geometry>
-               <box size="0.5 0.2 0.15" />
+                <box size="0.5 0.15 0.15" />
             </geometry>
             <material name="white" />
@@ -44,18 +44,18 @@
             <origin xyz="0 0 0.075" /> <!-- Sửa tâm va chạm -->
             <geometry>
-                <box size="0.5 0.2 0.15" />
+                <box size="0.5 0.15 0.15" />
             </geometry>
         </collision>
-        <xacro:inertial_box mass="0.5" x="0.5" y="0.2" z="0.15">
-             <origin xyz="0 0 0.075" rpy="0 0 0" />
+        <xacro:inertial_box mass="0.5" x="0.25" y="0.15" z="0.1">
+            <origin xyz="0 0 0.075" rpy="0 0 0" />
         </xacro:inertial_box>
     </link>
     <!-- IMPORT LEG PATTERN -->
-    <xacro:include filename="$(find first_robot)/description/leg_block.xacro"/>
+    <xacro:include filename="$(find first_robot)/description/leg_block.xacro" />
     <!-- Gọi 4 chân: FL, FR, RL, RR -->
-    <xacro:leg prefix="left_front"  x=" 0.15" y=" 0.10" />
+    <xacro:leg prefix="left_front" x=" 0.15" y=" 0.10" />
     <xacro:leg prefix="right_front" x=" 0.15" y="-0.10" />
-    <xacro:leg prefix="left_rear"   x="-0.15" y=" 0.10" />
-    <xacro:leg prefix="right_rear"  x="-0.15" y="-0.10" />
+    <xacro:leg prefix="left_rear" x="-0.15" y=" 0.10" />
+    <xacro:leg prefix="right_rear" x="-0.15" y="-0.10" />
     <!-- HEAD LINK -->
     <joint name="head_joint" type="fixed">
