Commit message: update

File: src/first_robot/description/camera.xacro (robot description, xacro)
@@ -4,10 +4,10 @@
         <parent link="chassis" />
         <child link="camera_link" />
-        <origin xyz="0.305 0 0.08" rpy="0 0 0" />
+        <origin xyz="0.25 0 0.08" rpy="0 0 0" />
     </joint>
     <joint name="camera_optical_joint" type="fixed">
         <parent link="camera_link" />
         <child link="camera_link_optical" />
-        <origin xyz="0 0 0" rpy="${-pi/2} 0 ${-pi/2}" />
+        <origin xyz="0.25 0 0" rpy="${-pi/2} 0 ${-pi/2}" />
     </joint>
     <link name="camera_link_optical"></link>

File: src/first_robot/description/robot_core_ver_snipdog.xacro (robot description, xacro)
@@ -16,4 +16,7 @@
         <color rgba="1 0 0 1" />
     </material>
+    <material name="grey">
+        <color rgba="0.5 0.5 0.5 1" />
+    </material>
     <!-- BASE LINK -->
     <link name="base_link"></link>
@@ -22,11 +25,11 @@
         <parent link="base_link" />
         <child link="chassis" />
-        <origin xyz="-0.1 0 0" />
+         <origin xyz="0 0 0" />
     </joint>
     <link name="chassis">
         <visual>
-            <origin xyz="0.15 0 0.075" />
+            <origin xyz="0 0 0.075" />
             <geometry>
-                <box size="0.3 0.3 0.15" />
+               <box size="0.5 0.2 0.15" />
             </geometry>
             <material name="white" />
@@ -35,18 +38,42 @@
             <origin xyz="0.15 0 0.075" />
             <geometry>
-                <box size="0.3 0.3 0.15" />
+                <box size="0.5 0.2 0.15" />
             </geometry>
         </collision>
-        <xacro:inertial_box mass="0.5" x="0.3" y="0.1" z="0.15">
-            <origin xyz="0.15 0 0.075" rpy="0 0 0" />
+        <xacro:inertial_box mass="0.5" x="0.5" y="0.2" z="0.15">
+             <origin xyz="0 0 0.075" rpy="0 0 0" />
         </xacro:inertial_box>
     </link>
     <!-- FL (Front Left) LEG -->
     <!-- IMPORT LEG PATTERN -->
-    <xacro:include filename="$(find first_robot)/description/leg_macro.xacro"/>
-     <!-- Gọi 4 chân: FL, FR, RL, RR -->
-    <xacro:leg side="left"  pos="front" suffix="" base_link="base_link" hip_pos="0.1 0.05 0" hip_rpy="0 0 0" knee_pos="0 0 -0.05" knee_rpy="0 0 0" ankle_pos="0.0 0.0 -0.08" ankle_rpy="0 0 0" />
-    <xacro:leg side="right" pos="front" suffix="" base_link="base_link" hip_pos="0.1 -0.05 0" hip_rpy="0 0 0" knee_pos="0 0 -0.05" knee_rpy="0 0 0" ankle_pos="0.0 0.0 -0.08" ankle_rpy="0 0 0" />
-    <xacro:leg side="left"  pos="rear"  suffix="" base_link="base_link" hip_pos="-0.1 0.05 0" hip_rpy="0 0 0" knee_pos="0 0 -0.05" knee_rpy="0 0 0" ankle_pos="0.0 0.0 -0.08"  ankle_rpy="0 0 0" />
-    <xacro:leg side="right" pos="rear"  suffix="" base_link="base_link" hip_pos="-0.1 -0.05 0" hip_rpy="0 0 0" knee_pos="0 0 -0.05" knee_rpy="0 0 0" ankle_pos="0.0 0.0 -0.08" ankle_rpy="0 0 0"/>
+    <xacro:include filename="$(find first_robot)/description/leg_block.xacro"/>
+    <!-- Gọi 4 chân: FL, FR, RL, RR -->
+    <xacro:leg prefix="left_front"  x=" 0.15" y=" 0.10" />
+    <xacro:leg prefix="right_front" x=" 0.15" y="-0.10" />
+    <xacro:leg prefix="left_rear"   x="-0.15" y=" 0.10" />
+    <xacro:leg prefix="right_rear"  x="-0.15" y="-0.10" />
+    <!-- HEAD LINK -->
+    <joint name="head_joint" type="fixed">
+        <parent link="base_link" />
+        <child link="head" />
+        <origin xyz="0 0 0.15" />
+    </joint>
+    <link name="head">
+        <visual>
+            <origin xyz="0 0 0.05" />
+            <geometry>
+                <box size="0.1 0.1 0.1" />
+            </geometry>
+            <material name="orange" />
+        </visual>
+        <collision>
+            <origin xyz="0 0 0.05" />
+            <geometry>
+                <box size="0.1 0.1 0.1" />
+            </geometry>
+        </collision>
+        <xacro:inertial_box mass="0.2" x="0.1" y="0.1" z="0.1">
+            <origin xyz="0 0 0.05" rpy="0 0 0" />
+        </xacro:inertial_box>
+    </link>
 </robot>

Commit message: temp update add rviz2

File: src/first_robot/description/camera.xacro (robot description, xacro)
@@ -4,5 +4,5 @@
         <parent link="chassis" />
         <child link="camera_link" />
-        <origin xyz="0.25 0 0.08" rpy="0 0 0" />
+        <origin xyz="0.25 0 0.04" rpy="0 0 0" />
     </joint>
     <joint name="camera_optical_joint" type="fixed">
@@ -15,5 +15,5 @@
         <visual>
             <geometry>
-                <box size="0.010 0.03 0.03" />
+                <box size="0.010 0.03 0.015" />
             </geometry>
             <material name="red" />

File: src/first_robot/description/imu_link.xacro (robot description, xacro)
@@ -11,5 +11,5 @@
         <parent link="base_link"/>
         <child link="imu_link"/>
-        <origin xyz="0 0 0.1"/>
+        <origin xyz="0 0 0.05"/>
         <!-- Đặt IMU gần trọng tâm -->
     </joint>

File: src/first_robot/description/leg_block.xacro (robot description, xacro)
@@ -7,6 +7,5 @@
   <xacro:property name="motor_length" value="0.02" /> <!-- Length of motor cylinders m -->
   <xacro:property name="foot_radius" value="0.03" /> <!-- Radius of foot sphere m -->
-  <!--  INERTIAL MACRO  -->
-  <!-- Macro to calculate inertia for box-shaped links -->
+  <!-- INERTIAL MACRO -->
   <xacro:macro name="inertial_box_leg" params="mass box_size">
     <inertial>
@@ -20,19 +19,29 @@
     </inertial>
   </xacro:macro>
-  <!--  LEG MACRO  -->
-  <!-- Macro to define a single leg with hip thigh knee shank ankle and foot -->
+  <!-- INERTIAL SPHERE MACRO -->
+  <xacro:macro name="inertial_sphere" params="mass radius">
+    <inertial>
+      <mass value="${mass}" />
+      <origin xyz="0 0 0" rpy="0 0 0" />
+      <inertia
+        ixx="${(2/5.0)*mass*pow(radius,2)}"
+        iyy="${(2/5.0)*mass*pow(radius,2)}"
+        izz="${(2/5.0)*mass*pow(radius,2)}"
+        ixy="0.0" ixz="0.0" iyz="0.0" />
+    </inertial>
+  </xacro:macro>
+  <!-- LEG MACRO -->
   <xacro:macro name="leg" params="prefix x y">
-    <!--  HIP SECTION  -->
-    <!-- Hip motor link  Small cylindrical motor attached to chassis -->
+    <!-- HIP SECTION -->
     <link name="${prefix}_hip_motor">
       <visual>
-        <origin xyz="0 0 0.005" />
+        <origin xyz="0 0 0" />
         <geometry>
           <cylinder length="${motor_length}" radius="${motor_radius}" />
         </geometry>
-        <material name="grey" />
+        <material name="red" />
       </visual>
       <collision>
-        <origin xyz="0 0 0.005" />
+        <origin xyz="0 0 0" />
         <geometry>
           <cylinder length="${motor_length}" radius="${motor_radius}" />
@@ -44,22 +53,19 @@
       </inertial>
     </link>
-    <!-- Hip motor mount  Fixed joint attaching hip motor to chassis -->
     <joint name="${prefix}_hip_motor_mount" type="fixed">
       <parent link="chassis" />
       <child link="${prefix}_hip_motor" />
-      <origin xyz="${x} ${y} -0.005" />
+      <origin xyz="${x} ${y} -0.005" rpy="0 0 0" /> <!-- Attach under chassis belly -->
     </joint>
-    <!-- Hip joint  Revolute joint for thigh rotation, limited to forward motion -->
     <joint name="${prefix}_hip_joint" type="revolute">
       <parent link="${prefix}_hip_motor" />
       <child link="${prefix}_thigh" />
-      <origin xyz="0 0 0" />
-      <axis xyz="0 1 0" /> <!-- Rotation around y-axis -->
-      <limit effort="5" velocity="2.0" lower="-1.57" upper="0" /> <!-- Forward motion only -->
+      <origin xyz="0 0 0" rpy="0 0.385 0" /> <!-- -45° for thigh backward -->
+      <axis xyz="0 1 0" />
+      <limit effort="5" velocity="2.0" lower="-1.57" upper="1.57" />
     </joint>
-    <!-- Thigh link  Box-shaped link connecting hip to knee -->
     <link name="${prefix}_thigh">
       <visual>
-        <origin xyz="0 0 -${thigh_length/2}" /> <!-- Center of thigh -->
+        <origin xyz="0 0 -${thigh_length/2}" />
         <geometry>
           <box size="0.03 0.03 ${thigh_length}" />
@@ -75,9 +81,8 @@
       <xacro:inertial_box_leg mass="0.15" box_size="${[0.03, 0.03, thigh_length]}" />
     </link>
-    <!--  KNEE SECTION  -->
-    <!-- Knee motor link  Small cylindrical motor attached to thigh -->
+    <!-- KNEE SECTION -->
     <link name="${prefix}_knee_motor">
       <visual>
-        <origin xyz="0 0 -0.01" />
+        <origin xyz="0 0 0" />
         <geometry>
           <cylinder length="${motor_length}" radius="${motor_radius}" />
@@ -86,5 +91,5 @@
       </visual>
       <collision>
-        <origin xyz="0 0 -0.01" />
+        <origin xyz="0 0 0" />
         <geometry>
           <cylinder length="${motor_length}" radius="${motor_radius}" />
@@ -96,19 +101,16 @@
       </inertial>
     </link>
-    <!-- Knee motor mount  Fixed joint attaching knee motor to thigh -->
     <joint name="${prefix}_knee_motor_mount" type="fixed">
       <parent link="${prefix}_thigh" />
       <child link="${prefix}_knee_motor" />
-      <origin xyz="0 0 -${thigh_length}" rpy="0 -0.3 0" /> <!-- Tilt forward for natural posture -->
+      <origin xyz="0 0 -${thigh_length}" rpy="0 0 0" /> <!-- No rotation here -->
     </joint>
-    <!-- Knee joint  Revolute joint for shank rotation, limited to forward motion -->
     <joint name="${prefix}_knee_joint" type="revolute">
       <parent link="${prefix}_knee_motor" />
       <child link="${prefix}_shank" />
-      <origin xyz="0 0 0" />
-      <axis xyz="0 1 0" /> <!-- Rotation around y axis -->
-      <limit effort="5" velocity="2.0" lower="-2.8" upper="0" /> <!-- Forward motion only -->
+      <origin xyz="0 0 0" rpy="0 -0.385 0" /> <!-- +45° for shank forward -->
+      <axis xyz="0 1 0" />
+      <limit effort="5" velocity="2.0" lower="-2.8" upper="0" />
     </joint>
-    <!-- Shank link  Box-shaped link connecting knee to ankle -->
     <link name="${prefix}_shank">
       <visual>
@@ -127,9 +129,8 @@
       <xacro:inertial_box_leg mass="0.15" box_size="${[0.02, 0.02, shank_length]}" />
     </link>
-    <!--  ANKLE SECTION  -->
-    <!-- Ankle motor link  Small cylindrical motor attached to shank -->
+    <!-- ANKLE SECTION -->
     <link name="${prefix}_ankle_motor">
       <visual>
-        <origin xyz="0 0 -0.01" />
+        <origin xyz="0 0 0" />
         <geometry>
           <cylinder length="${motor_length}" radius="${motor_radius}" />
@@ -138,5 +139,5 @@
       </visual>
       <collision>
-        <origin xyz="0 0 -0.01" />
+        <origin xyz="0 0 0" />
         <geometry>
           <cylinder length="${motor_length}" radius="${motor_radius}" />
@@ -148,19 +149,16 @@
       </inertial>
     </link>
-    <!-- Ankle motor mount  Fixed joint attaching ankle motor to shank -->
     <joint name="${prefix}_ankle_motor_mount" type="fixed">
       <parent link="${prefix}_shank" />
       <child link="${prefix}_ankle_motor" />
-      <origin xyz="0 0 -${shank_length}" rpy="0 -0.3 0" /> <!-- Tilt forward for natural posture -->
+      <origin xyz="0 0 -${shank_length}" rpy="0 0 0" /> <!-- No rotation here -->
     </joint>
-    <!-- Ankle joint  Revolute joint for foot rotation -->
     <joint name="${prefix}_ankle_joint" type="revolute">
       <parent link="${prefix}_ankle_motor" />
       <child link="${prefix}_foot" />
-      <origin xyz="0 0 0" />
-      <axis xyz="0 1 0" /> <!-- Rotation around y-axis -->
+      <origin xyz="0 0 -${motor_length/2}" rpy="0 0 0" /> <!-- No rotation to align foot -->
+      <axis xyz="0 1 0" />
       <limit effort="5" velocity="2.0" lower="-2.0" upper="2.0" />
     </joint>
-    <!-- Foot link  Spherical foot for ground contact -->
     <link name="${prefix}_foot">
       <visual>
@@ -175,13 +173,12 @@
         </geometry>
       </collision>
-      <xacro:inertial_sphere mass="0.1" radius="${foot_radius}">
-        <origin xyz="0 0 0" rpy="0 0 0" />
-      </xacro:inertial_sphere>
+      <xacro:inertial_sphere mass="0.1" radius="${foot_radius}" />
     </link>
     <!-- Gazebo settings for foot friction -->
     <gazebo reference="${prefix}_foot">
-      <mu1>0.8</mu1> <!-- Giảm ma sát ngang -->
-      <mu2>0.8</mu2> <!-- Giảm ma sát dọc -->
+      <mu1>0.8</mu1>
+      <mu2>0.8</mu2>
     </gazebo>
+    <!-- Transmissions -->
     <transmission name="${prefix}_hip_trans">
       <type>transmission_interface/SimpleTransmission</type>

File: src/first_robot/description/lidar_2d_camera.xacro (robot description, xacro)
@@ -4,5 +4,5 @@
         <parent link="base_link" />
         <child link="lidar_link" />
-        <origin xyz="0.1 0 0.175" rpy="0 0 0" />
+        <origin xyz="0.1 0 0.075" rpy="0 0 0" />
     </joint>
     <link name="lidar_link">

File: src/first_robot/description/robot_core.xacro (robot description, xacro)
@@ -22,7 +22,8 @@
     <link name="base_link">
         <inertial>
-            <mass value="0.25" /> <!-- Giảm từ 2.0 -->
-            <origin xyz="0 0 0.1" />
-            <inertia ixx="0.1" iyy="0.1" izz="0.1" ixy="0" ixz="0" iyz="0" />
+            <mass value="0.5"/>
+            <!-- Giảm từ 2.0 -->
+           <origin xyz="0 0 0.05"/>
+            <inertia ixx="0.1" iyy="0.1" izz="0.1" ixy="0" ixz="0" iyz="0"/>
         </inertial>
     </link>
@@ -35,22 +36,23 @@
     <link name="chassis">
         <visual>
-            <origin xyz="0 0 0.075" />
+            <origin xyz="0 0 0.025" />
             <geometry>
-                <box size="0.5 0.15 0.15" />
+                <box size="0.5 0.2 0.1" />
             </geometry>
             <material name="white" />
         </visual>
         <collision>
-            <origin xyz="0 0 0.075" /> <!-- Sửa tâm va chạm -->
+            <origin xyz="0 0 0.025" />
+            <!-- Sửa tâm va chạm -->
             <geometry>
-                <box size="0.5 0.15 0.15" />
+                <box size="0.5 0.2 0.1" />
             </geometry>
         </collision>
-        <xacro:inertial_box mass="0.5" x="0.25" y="0.15" z="0.1">
-            <origin xyz="0 0 0.075" rpy="0 0 0" />
+        <xacro:inertial_box mass="0.5" x="0.5" y="0.2" z="0.1">
+            <origin xyz="0 0 0.025" rpy="0 0 0" />
         </xacro:inertial_box>
     </link>
     <!-- IMPORT LEG PATTERN -->
-    <xacro:include filename="$(find first_robot)/description/leg_block.xacro" />
+    <xacro:include filename="$(find first_robot)/description/leg_block.xacro"/>
     <!-- Gọi 4 chân: FL, FR, RL, RR -->
     <xacro:leg prefix="left_front" x=" 0.15" y=" 0.10" />
@@ -59,12 +61,12 @@
     <xacro:leg prefix="right_rear" x="-0.15" y="-0.10" />
     <!-- HEAD LINK -->
-    <joint name="head_joint" type="fixed">
+    <!-- <joint name="head_joint" type="fixed">
         <parent link="base_link" />
         <child link="head" />
-        <origin xyz="0 0 0.15" />
+        <origin xyz="0.05 0 0.075" />
     </joint>
     <link name="head">
         <visual>
-            <origin xyz="0 0 0.05" />
+            <origin xyz="0.05 0 0.05" />
             <geometry>
                 <box size="0.1 0.1 0.1" />
@@ -73,5 +75,5 @@
         </visual>
         <collision>
-            <origin xyz="0 0 0.05" />
+            <origin xyz="0.05 0 0.05" />
             <geometry>
                 <box size="0.1 0.1 0.1" />
@@ -79,6 +81,6 @@
         </collision>
         <xacro:inertial_box mass="0.2" x="0.1" y="0.1" z="0.1">
-            <origin xyz="0 0 0.05" rpy="0 0 0" />
+            <origin xyz="0.05 0 0.05" rpy="0 0 0" />
         </xacro:inertial_box>
-    </link>
+    </link> -->
 </robot>
