Commit message: update fix leg

File: src/first_robot/description/camera.xacro (robot description, xacro)
@@ -4,10 +4,10 @@
         <parent link="base_link" />
         <child link="camera_link" />
-        <origin xyz="0.25 0 0.04" rpy="0 0 0" />
+        <origin xyz="0.10 0 0.04" rpy="0 0 0" />
     </joint>
     <joint name="camera_optical_joint" type="fixed">
         <parent link="camera_link" />
         <child link="camera_link_optical" />
-        <origin xyz="0.25 0 0" rpy="${-pi/2} 0 ${-pi/2}" />
+        <origin xyz="0.05 0 0" rpy="${-pi/2} 0 ${-pi/2}" />
     </joint>
     <link name="camera_link_optical"></link>
@@ -17,5 +17,5 @@
                 <box size="0.010 0.03 0.015" />
             </geometry>
-            <material name="red" />
+            <material name="cyan" />
         </visual>
     </link>

File: src/first_robot/description/gz_control.xacro (robot description, xacro)
@@ -15,17 +15,17 @@
     </xacro:macro>
     <!-- Front Left Leg -->
-    <!-- <xacro:define_joint_interfaces joint_name="front_left_hip_joint" /> -->
+    <xacro:define_joint_interfaces joint_name="front_left_hip_joint" />
     <xacro:define_joint_interfaces joint_name="front_left_knee_joint" />
     <xacro:define_joint_interfaces joint_name="front_left_ankle_joint" />
     <!-- Front Right Leg -->
-    <!-- <xacro:define_joint_interfaces joint_name="front_right_hip_joint" /> -->
+    <xacro:define_joint_interfaces joint_name="front_right_hip_joint" />
     <xacro:define_joint_interfaces joint_name="front_right_knee_joint" />
     <xacro:define_joint_interfaces joint_name="front_right_ankle_joint" />
     <!-- Rear Left Leg -->
-    <!-- <xacro:define_joint_interfaces joint_name="rear_left_hip_joint" /> -->
+    <xacro:define_joint_interfaces joint_name="rear_left_hip_joint" />
     <xacro:define_joint_interfaces joint_name="rear_left_knee_joint" />
     <xacro:define_joint_interfaces joint_name="rear_left_ankle_joint" />
     <!-- Rear Right Leg -->
-    <!-- <xacro:define_joint_interfaces joint_name="rear_right_hip_joint" /> -->
+    <xacro:define_joint_interfaces joint_name="rear_right_hip_joint" />
     <xacro:define_joint_interfaces joint_name="rear_right_knee_joint" />
     <xacro:define_joint_interfaces joint_name="rear_right_ankle_joint" />

File: src/first_robot/description/leg_block.xacro (robot description, xacro)
@@ -32,8 +32,9 @@
       </inertial>
     </link>
-    <joint name="${prefix}_hip_joint" type="fixed">
+    <joint name="${prefix}_hip_joint" type="revolute">
       <parent link="${pos}_body"/>
       <child link="${prefix}_hip_link"/>
       <origin xyz="0 0 0.0" rpy="0 0 0"/>
+      <limit lower="-1.57" upper="1.57" effort="30" velocity="7.0"/>
       <!-- Vị trí gắn khớp háng vào body-->
     </joint>
@@ -100,5 +101,12 @@
       <!-- Gắn vào motor háng mô phỏng -->
       <child link="${prefix}_knee_link"/>
-      <origin xyz="0 0 0" rpy="0 0.5 0"/>
+      <xacro:if value="${(side == 'left')}">
+         <origin xyz="0 0 0" rpy="0.3 0.1 0"/>
+        <!-- Vị trí đặt link đùi -  so với motor háng mô phỏng -->
+      </xacro:if>
+      <xacro:if value="${(side == 'right')}">
+         <origin xyz="0 0 0" rpy="-0.3 0.1 0"/>
+        <!-- Vị trí đặt link đùi -  so với motor háng mô phỏng -->
+      </xacro:if>
       <axis xyz="0 1 0"/>
       <limit lower="-1.57" upper="1.57" effort="30" velocity="7.0"/>
@@ -141,10 +149,10 @@
         </geometry>
         <xacro:if value="${(side == 'left')}">
-          <origin xyz="0 0 -0.08" rpy="0 -1.0 0"/>
+          <origin xyz="0 0 -0.12" rpy="0 -0.9 0"/>
           <!-- Dịch xuống 1/2 chiều dài -->
           <!-- vị trí đặt link mô phỏng motor khớp háng- trái -->
         </xacro:if>
         <xacro:if value="${(side == 'right')}">
-          <origin xyz="0 0 -0.08" rpy="0 -1.0 0"/>
+          <origin xyz="0 0 -0.12" rpy="0 -0.9 0"/>
           <!-- Dịch xuống 1/2 chiều dài -->
           <!-- vị trí đặt link mô phỏng motor khớp háng- phải -->
@@ -153,5 +161,5 @@
       </visual>
       <collision name="${prefix}_ankle_collision">
-        <origin xyz="0 0 -0.08"/>
+        <origin xyz="0 0 -0.12"/>
         <!-- Khớp visual -->
         <geometry>
@@ -160,5 +168,5 @@
       </collision>
       <inertial>
-        <origin xyz="0 0 -0.08"/>
+        <origin xyz="0 0 -0.12"/>
         <!-- Dịch khối lượng xuống luôn -->
         <mass value="0.2"/>
@@ -167,17 +175,17 @@
     </link>
     <!-- ankle Joint (Cẳng chân, quay về trước 45°) -->
-    <joint name="${prefix}_ankle_joint" type="fixed">
+    <joint name="${prefix}_ankle_joint" type="revolute">
       <parent link="${prefix}_knee_motor_link"/>
       <child link="${prefix}_ankle_link"/>
       <xacro:if value="${(side == 'left')}">
-        <origin xyz="0 0.055 0" rpy="0 -0.60 0"/>
+        <origin xyz="0.08 0.04 0" rpy="0.12 0.45 0"/>
         <!-- Vị trí đặt link đùi -  so với motor háng mô phỏng -->
       </xacro:if>
       <xacro:if value="${(side == 'right')}">
-        <origin xyz="0 -0.055 0" rpy="0 -0.60 0"/>
+        <origin xyz="0.08 -0.04 0" rpy="-0.12 0.45 0"/>
         <!-- Vị trí đặt link đùi -  so với motor háng mô phỏng -->
       </xacro:if>
       <!-- rút ngắn chiều dài -->
-      <axis xyz="0 1 0"/>
+      <axis xyz="1 1 0"/>
       <limit lower="-1.57" upper="1.57" effort="30" velocity="7.0"/>
     </joint>
@@ -186,5 +194,5 @@
     <link name="${prefix}_foot_link">
       <visual name="${prefix}_foot_visual">
-        <origin xyz="0.045 0 -0.055"/>
+        <origin xyz="0.045 0 -0.1"/>
         <geometry>
           <sphere radius="0.02"/>
@@ -193,5 +201,5 @@
       </visual>
       <collision name="${prefix}_foot_collision">
-        <origin xyz="0.045 0 -0.055"/>
+        <origin xyz="0.045 0 -0.1"/>
         <geometry>
           <sphere radius="0.02"/>

File: src/first_robot/description/lidar_2d_camera.xacro (robot description, xacro)
@@ -4,10 +4,10 @@
         <parent link="base_link" />
         <child link="lidar_link" />
-        <origin xyz="0.1 0 0.075" rpy="0 0 0" />
+        <origin xyz="0.05 0 0.045" rpy="0 0 0" />
     </joint>
     <link name="lidar_link">
         <visual>
             <geometry>
-                <cylinder radius="0.05" length="0.04" />
+                <cylinder radius="0.025" length="0.02" />
             </geometry>
             <material name="red" />
@@ -15,8 +15,8 @@
         <collision>
             <geometry>
-                <cylinder radius="0.05" length="0.04" />
+                <cylinder radius="0.025" length="0.02" />
             </geometry>
         </collision>
-        <xacro:inertial_cylinder mass="0.1" length="0.04" radius="0.05">
+        <xacro:inertial_cylinder mass="0.01" length="0.02" radius="0.05">
             <origin xyz="0 0 0" rpy="0 0 0" />
         </xacro:inertial_cylinder>

File: src/first_robot/description/robot_core.xacro (robot description, xacro)
@@ -3,11 +3,10 @@
     <!-- IMPORT MATERIAL -->
     <xacro:include filename="$(find first_robot)/description/constants.xacro"/>
-    <!-- AAAAAAAAAAAAAAAAAAA -->
     <!-- BASE LINK -->
     <link name="base_link">
         <visual name="base_link_visual">
-            <origin xyz="0 0 0.025" />
+            <origin xyz="0 0 0.0125" />
             <geometry>
-                <box size="0.5 0.2 0.1" />
+                <box size="0.2 0.15 0.05" />
             </geometry>
             <material name="white" />
@@ -17,8 +16,8 @@
             <!-- Sửa tâm va chạm -->
             <geometry>
-                <box size="0.5 0.2 0.1" />
+                <box size="0.2 0.15 0.05" />
             </geometry>
         </collision>
-        <xacro:inertial_box mass="0.5" x="0.5" y="0.2" z="0.1">
+        <xacro:inertial_box mass="0.5" x="0.2" y="0.15" z="0.05">
             <origin xyz="0 0 0.025" rpy="0 0 0" />
         </xacro:inertial_box>
@@ -46,5 +45,5 @@
       <parent link="base_link"/>
       <child link="front_body"/>
-      <origin xyz="0.25 0 0" rpy="0 0 0"/> <!-- Đẩy về trước cho cân đối -->
+      <origin xyz="0.1 0 0" rpy="0 0 0"/> <!-- Đẩy về trước cho cân đối -->
     </joint>
     <!-- Rear Body -->
@@ -70,36 +69,12 @@
       <parent link="base_link"/>
       <child link="rear_body"/>
-       <origin xyz="-0.25 0 0" rpy="0 0 0"/> <!-- Đẩy về sau cho cân đối -->
-    </joint>
-    <!-- Chân trước trái FL -->
-    <joint name="front_left_body_hip_joint" type="fixed">
-      <parent link="front_body"/>
-      <child link="front_left_hip_link"/>
-       <origin xyz="0.1 0.1 -0.025" rpy="0 0 0"/> <!-- Ngang 0.1, rộng 0.1, hạ thấp hơn -->
-    </joint>
-    <!-- Chân trước phải FR -->
-    <joint name="front_right_body_hip_joint" type="fixed">
-      <parent link="front_body"/>
-      <child link="front_right_hip_link"/>
-       <origin xyz="0.1 -0.1 -0.025" rpy="0 0 0"/>
-    </joint>
-    <!-- Chân sau trái RL -->
-    <joint name="rear_left_body_hip_joint" type="fixed">
-      <parent link="rear_body"/>
-      <child link="rear_left_hip_link"/>
-      <origin xyz="-0.1 0.1 -0.025" rpy="0 0 0"/>
-    </joint>
-    <!-- Chân sau phải RR -->
-    <joint name="rear_right_body_hip_joint" type="fixed">
-      <parent link="rear_body"/>
-      <child link="rear_right_hip_link"/>
-      <origin xyz="-0.1 -0.1 -0.025" rpy="0 0 0"/>
+       <origin xyz="-0.1 0 0" rpy="0 0 0"/> <!-- Đẩy về sau cho cân đối -->
     </joint>
     <!-- IMPORT LEG PATTERN -->
     <xacro:include filename="$(find first_robot)/description/leg_block.xacro"/>
     <!-- Gọi macro leg cho từng chân -->
-    <xacro:leg prefix="front_left" pos="front" side="left" x=" 0.15" y=" 0.10" />
-    <xacro:leg prefix="front_right" pos="front" side="right" x=" 0.15" y="-0.10" />
-    <xacro:leg prefix="rear_left" pos="rear" side="left" x="-0.15" y=" 0.10" />
-    <xacro:leg prefix="rear_right" pos="rear" side="right" x="-0.15" y="-0.10" />
+    <xacro:leg prefix="front_left" pos="front" side="left" x=" 0.075" y=" 0.05" />
+    <xacro:leg prefix="front_right" pos="front" side="right" x=" 0.075" y="-0.05" />
+    <xacro:leg prefix="rear_left" pos="rear" side="left" x="-0.075" y=" 0.05" />
+    <xacro:leg prefix="rear_right" pos="rear" side="right" x="-0.075" y="-0.05" />
 </robot>

File: src/robot.urdf (robot description, URDF)
Before this commit: robot my_robot, 31 links, 34 joints
Links:
- link base_link: geometry collision box size=0.2 0.15 0.05; visual box size=0.2 0.15 0.05
- link lidar_link: mass 0.1 -> 0.01; geometry collision cylinder length=0.02 radius=0.025; visual cylinder length=0.02 radius=0.025
Joints:
- removed joint front_left_body_hip_joint
- removed joint front_right_body_hip_joint
- removed joint rear_left_body_hip_joint
- removed joint rear_right_body_hip_joint
- joint camera_joint: origin xyz=0.25 0 0.04 rpy=0 0 0 -> xyz=0.10 0 0.04 rpy=0 0 0
- joint camera_optical_joint: origin xyz=0.25 0 0 rpy=-1.5707963267948966 0 -1.5707963267948966 -> xyz=0.05 0 0 rpy=-1.5707963267948966 0 -1.5707963267948966
- joint front_body_joint: origin xyz=0.25 0 0 rpy=0 0 0 -> xyz=0.1 0 0 rpy=0 0 0
- joint front_left_ankle_joint: axis 0 1 0 -> 1 1 0; origin xyz=0 0.055 0 rpy=0 -0.60 0 -> xyz=0.08 0.04 0 rpy=0.12 0.45 0; type fixed -> revolute
- joint front_left_hip_joint: limit (none) -> lower=-1.57 upper=1.57 effort=30 velocity=7.0; type fixed -> revolute
- joint front_left_knee_joint: origin xyz=0 0 0 rpy=0 0.5 0 -> xyz=0 0 0 rpy=0.3 0.1 0
- joint front_right_ankle_joint: axis 0 1 0 -> 1 1 0; origin xyz=0 -0.055 0 rpy=0 -0.60 0 -> xyz=0.08 -0.04 0 rpy=-0.12 0.45 0; type fixed -> revolute
- joint front_right_hip_joint: limit (none) -> lower=-1.57 upper=1.57 effort=30 velocity=7.0; type fixed -> revolute
- joint front_right_knee_joint: origin xyz=0 0 0 rpy=0 0.5 0 -> xyz=0 0 0 rpy=-0.3 0.1 0
- joint laser_joint: origin xyz=0.1 0 0.075 rpy=0 0 0 -> xyz=0.05 0 0.045 rpy=0 0 0
- joint rear_body_joint: origin xyz=-0.25 0 0 rpy=0 0 0 -> xyz=-0.1 0 0 rpy=0 0 0
- joint rear_left_ankle_joint: axis 0 1 0 -> 1 1 0; origin xyz=0 0.055 0 rpy=0 -0.60 0 -> xyz=0.08 0.04 0 rpy=0.12 0.45 0; type fixed -> revolute
- joint rear_left_hip_joint: limit (none) -> lower=-1.57 upper=1.57 effort=30 velocity=7.0; type fixed -> revolute
- joint rear_left_knee_joint: origin xyz=0 0 0 rpy=0 0.5 0 -> xyz=0 0 0 rpy=0.3 0.1 0
- joint rear_right_ankle_joint: axis 0 1 0 -> 1 1 0; origin xyz=0 -0.055 0 rpy=0 -0.60 0 -> xyz=0.08 -0.04 0 rpy=-0.12 0.45 0; type fixed -> revolute
- joint rear_right_hip_joint: limit (none) -> lower=-1.57 upper=1.57 effort=30 velocity=7.0; type fixed -> revolute
- joint rear_right_knee_joint: origin xyz=0 0 0 rpy=0 0.5 0 -> xyz=0 0 0 rpy=-0.3 0.1 0
