Commit message: convert design to unitree go2 formating

File: src/first_robot/description/camera.xacro (robot description, xacro)
@@ -4,5 +4,5 @@
         <parent link="base_link" />
         <child link="camera_link" />
-        <origin xyz="0.10 0 0.04" rpy="0 0 0" />
+        <origin xyz="0.326 0 0.043"  rpy="0 0 0"/>
     </joint>
     <joint name="camera_optical_joint" type="fixed">
@@ -14,9 +14,21 @@
     <link name="camera_link">
         <visual>
+            <origin rpy="0 0 0" xyz="0 0 0"/>
             <geometry>
-                <box size="0.010 0.03 0.015" />
+                <sphere radius="0.001"/>
             </geometry>
             <material name="cyan" />
         </visual>
+        <collision>
+            <origin rpy="0 0 0" xyz="0 0 0"/>
+            <geometry>
+                <sphere radius="0.001"/>
+            </geometry>
+        </collision>
+        <inertial>
+            <mass value="0.001"/>
+            <origin rpy="0 0 0" xyz="0 0 0"/>
+            <inertia ixx="0.0001" ixy="0" ixz="0" iyy="0.0001" iyz="0" izz="0.0001"/>
+        </inertial>
     </link>
     <gazebo reference="camera_link">

File: src/first_robot/description/constants.xacro (robot description, xacro)
@@ -3,7 +3,4 @@
     <material name="white">
         <color rgba="1 1 1 1" />
-    </material>
-    <material name="orange">
-        <color rgba="1 0.3 0.1 1" />
     </material>
     <material name="blue">
@@ -28,12 +25,141 @@
         <color rgba="0 0 0 1" />
     </material>
+    <material name="silver">
+        <color rgba="${233/255} ${233/255} ${216/255} 1.0"/>
+    </material>
+    <material name="orange">
+        <color rgba="${255/255} ${108/255} ${10/255} 1.0"/>
+    </material>
+    <material name="brown">
+        <color rgba="${222/255} ${207/255} ${195/255} 1.0"/>
+    </material>
     <material name="red">
-        <color rgba="1 0 0 1" />
+        <color rgba="0.8 0.0 0.0 1.0"/>
     </material>
-    <material name="grey">
-        <color rgba="0.5 0.5 0.5 1" />
-    </material>
-    <material name="silver">
-        <color rgba="0.75 0.75 0.75 1" />
-    </material>
+    <!-- Constants for robot dimensions -->
+    <xacro:property name="PI" value="3.1415926535897931"/>
+    <xacro:property name="stick_mass" value="0.00001"/>
+    <!-- simplified collision value -->
+    <xacro:property name="trunk_width" value="0.0935"/>
+    <xacro:property name="trunk_length" value="0.3762"/>
+    <xacro:property name="trunk_height" value="0.114"/>
+    <xacro:property name="hip_radius" value="0.046"/>
+    <xacro:property name="hip_length" value="0.04"/>
+    <xacro:property name="knee_shoulder_radius" value="0.041"/>
+    <xacro:property name="knee_shoulder_length" value="0.032"/>
+    <xacro:property name="knee_width" value="0.0245"/>
+    <xacro:property name="knee_height" value="0.034"/>
+    <xacro:property name="ankle_width" value="0.016"/>
+    <xacro:property name="ankle_height" value="0.016"/>
+    <xacro:property name="foot_radius" value="0.02"/>
+    <xacro:property name="stick_radius" value="0.01"/>
+    <xacro:property name="stick_length" value="0.2"/>
+    <!-- dynamics inertial value -->
+    <!-- trunk -->
+    <xacro:property name="trunk_mass" value="6.921"/>
+    <xacro:property name="trunk_com_x" value="0.021112"/>
+    <xacro:property name="trunk_com_y" value="0.00"/>
+    <xacro:property name="trunk_com_z" value="-0.005366"/>
+    <xacro:property name="trunk_ixx" value="0.02448"/>
+    <xacro:property name="trunk_ixy" value="0.00012166"/>
+    <xacro:property name="trunk_ixz" value="0.0014849"/>
+    <xacro:property name="trunk_iyy" value="0.098077"/>
+    <xacro:property name="trunk_iyz" value="-3.12E-05"/>
+    <xacro:property name="trunk_izz" value="0.107"/>
+    <!-- simplified collision value -->
+    <xacro:property name="trunk_width" value="0.0935"/>
+    <xacro:property name="trunk_length" value="0.3762"/>
+    <xacro:property name="trunk_height" value="0.114"/>
+    <xacro:property name="hip_radius" value="0.046"/>
+    <xacro:property name="hip_length" value="0.04"/>
+    <xacro:property name="knee_shoulder_radius" value="0.041"/>
+    <xacro:property name="knee_shoulder_length" value="0.032"/>
+    <xacro:property name="knee_width" value="0.0245"/>
+    <xacro:property name="knee_height" value="0.034"/>
+    <xacro:property name="ankle_width" value="0.016"/>
+    <xacro:property name="ankle_height" value="0.016"/>
+    <xacro:property name="foot_radius" value="0.02"/>
+    <xacro:property name="stick_radius" value="0.01"/>
+    <xacro:property name="stick_length" value="0.2"/>
+    <!-- kinematic value -->
+    <xacro:property name="knee_offset" value="0.0955"/>
+    <xacro:property name="knee_length" value="0.213"/>
+    <xacro:property name="ankle_length" value="0.213"/>
+    <!-- leg offset from trunk center value -->
+    <xacro:property name="leg_offset_x" value="0.1934"/>
+    <xacro:property name="leg_offset_y" value="0.0465"/>
+    <!-- <xacro:property name="trunk_offset_z" value="0.01675"/> -->
+    <xacro:property name="hip_offset" value="0.0955"/>
+    <!-- offset of link locations (left front) -->
+    <xacro:property name="hip_offset_x" value="0.1934"/>
+    <xacro:property name="hip_offset_y" value="0.0465"/>
+    <xacro:property name="hip_offset_z" value="0.0"/>
+    <xacro:property name="knee_offset_x" value="0"/>
+    <xacro:property name="knee_offset_y" value="0.0955"/>
+    <xacro:property name="knee_offset_z" value="0.0"/>
+    <xacro:property name="ankle_offset_x" value="0.0"/>
+    <xacro:property name="ankle_offset_y" value="0.0"/>
+    <xacro:property name="ankle_offset_z" value="-0.213"/>
+    <!-- joint limits -->
+    <xacro:property name="damping" value="0.01"/>
+    <xacro:property name="friction" value="0.2"/>
+    <xacro:property name="hip_position_max" value="1.0472"/>
+    <xacro:property name="hip_position_min" value="-1.0472"/>
+    <xacro:property name="hip_velocity_max" value="30.1"/>
+    <xacro:property name="hip_torque_max" value="23.7"/>
+    <xacro:property name="knee_position_max" value="3.4907"/>
+    <xacro:property name="knee_position_min" value="-1.5708"/>
+    <xacro:property name="knee_velocity_max" value="30.1"/>
+    <xacro:property name="knee_torque_max" value="23.7"/>
+    <xacro:property name="ankle_position_max" value="1.0"/>
+    <xacro:property name="ankle_position_min" value="-1.0"/>
+    <xacro:property name="ankle_velocity_max" value="20.06"/>
+    <xacro:property name="ankle_torque_max" value="35.55"/>
+    <!-- dynamics inertial value -->
+    <!-- trunk -->
+    <xacro:property name="trunk_mass" value="6.921"/>
+    <xacro:property name="trunk_com_x" value="0.021112"/>
+    <xacro:property name="trunk_com_y" value="0.00"/>
+    <xacro:property name="trunk_com_z" value="-0.005366"/>
+    <xacro:property name="trunk_ixx" value="0.02448"/>
+    <xacro:property name="trunk_ixy" value="0.00012166"/>
+    <xacro:property name="trunk_ixz" value="0.0014849"/>
+    <xacro:property name="trunk_iyy" value="0.098077"/>
+    <xacro:property name="trunk_iyz" value="-3.12E-05"/>
+    <xacro:property name="trunk_izz" value="0.107"/>
+    <!-- hip (left front) -->
+    <xacro:property name="hip_mass" value="0.678"/>
+    <xacro:property name="hip_com_x" value="-0.0054"/>
+    <xacro:property name="hip_com_y" value="0.00194"/>
+    <xacro:property name="hip_com_z" value="-0.000105"/>
+    <xacro:property name="hip_ixx" value="0.00048"/>
+    <xacro:property name="hip_ixy" value="-3.01E-06"/>
+    <xacro:property name="hip_ixz" value="1.11E-06"/>
+    <xacro:property name="hip_iyy" value="0.000884"/>
+    <xacro:property name="hip_iyz" value="-1.42E-06"/>
+    <xacro:property name="hip_izz" value="0.000596"/>
+    <!-- knee -->
+    <xacro:property name="knee_mass" value="1.152"/>
+    <xacro:property name="knee_com_x" value="-0.00374"/>
+    <xacro:property name="knee_com_y" value="-0.0223"/>
+    <xacro:property name="knee_com_z" value="-0.0327"/>
+    <xacro:property name="knee_ixx" value="0.00584"/>
+    <xacro:property name="knee_ixy" value="8.72E-05"/>
+    <xacro:property name="knee_ixz" value="-0.000289"/>
+    <xacro:property name="knee_iyy" value="0.0058"/>
+    <xacro:property name="knee_iyz" value="0.000808"/>
+    <xacro:property name="knee_izz" value="0.00103"/>
+    <!-- ankle -->
+    <xacro:property name="ankle_mass" value="0.154"/>
+    <xacro:property name="ankle_com_x" value="0.00548"/>
+    <xacro:property name="ankle_com_y" value="-0.000975"/>
+    <xacro:property name="ankle_com_z" value="-0.115"/>
+    <xacro:property name="ankle_ixx" value="0.00108"/>
+    <xacro:property name="ankle_ixy" value="3.4E-07"/>
+    <xacro:property name="ankle_ixz" value="1.72E-05"/>
+    <xacro:property name="ankle_iyy" value="0.0011"/>
+    <xacro:property name="ankle_iyz" value="8.28E-06"/>
+    <xacro:property name="ankle_izz" value="3.29E-05"/>
+    <!-- foot -->
+    <xacro:property name="foot_mass" value="0.06"/>
 </robot>

File: src/first_robot/description/gz_control.xacro (robot description, xacro)
@@ -14,20 +14,4 @@
       </joint>
     </xacro:macro>
-    <!-- Front Left Leg -->
-    <xacro:define_joint_interfaces joint_name="front_left_hip_joint" />
-    <xacro:define_joint_interfaces joint_name="front_left_knee_joint" />
-    <xacro:define_joint_interfaces joint_name="front_left_ankle_joint" />
-    <!-- Front Right Leg -->
-    <xacro:define_joint_interfaces joint_name="front_right_hip_joint" />
-    <xacro:define_joint_interfaces joint_name="front_right_knee_joint" />
-    <xacro:define_joint_interfaces joint_name="front_right_ankle_joint" />
-    <!-- Rear Left Leg -->
-    <xacro:define_joint_interfaces joint_name="rear_left_hip_joint" />
-    <xacro:define_joint_interfaces joint_name="rear_left_knee_joint" />
-    <xacro:define_joint_interfaces joint_name="rear_left_ankle_joint" />
-    <!-- Rear Right Leg -->
-    <xacro:define_joint_interfaces joint_name="rear_right_hip_joint" />
-    <xacro:define_joint_interfaces joint_name="rear_right_knee_joint" />
-    <xacro:define_joint_interfaces joint_name="rear_right_ankle_joint" />
   </ros2_control>
   <gazebo>

File: src/first_robot/description/imu_link.xacro (robot description, xacro)
@@ -3,13 +3,25 @@
     <link name="imu_link">
         <inertial>
-            <mass value="0.01"/>
-            <origin xyz="0 0 0"/>
-            <inertia ixx="0.001" iyy="0.001" izz="0.001" ixy="0" ixz="0" iyz="0"/>
+            <mass value="0.001"/>
+            <origin rpy="0 0 0" xyz="0 0 0"/>
+            <inertia ixx="0.0001" ixy="0" ixz="0" iyy="0.0001" iyz="0" izz="0.0001"/>
         </inertial>
+        <visual>
+            <origin rpy="0 0 0" xyz="0 0 0"/>
+            <geometry>
+                <box size="0.001 0.001 0.001"/>
+            </geometry>
+        </visual>
+        <collision>
+            <origin rpy="0 0 0" xyz="0 0 0"/>
+            <geometry>
+                <box size=".001 .001 .001"/>
+            </geometry>
+        </collision>
     </link>
     <joint name="imu_joint" type="fixed">
-        <parent link="base_link"/>
+        <parent link="trunk"/>
         <child link="imu_link"/>
-        <origin xyz="0 0 0.05"/>
+        <origin xyz="0 0 0.05" rpy="0 0 0" />
         <!-- Đặt IMU gần trọng tâm -->
     </joint>
@@ -28,5 +40,5 @@
                     <rate>
                         <mean>0.0</mean>
-                        <stddev>0.005</stddev>                        <!-- Giảm nhiễu -->
+                        <stddev>0.005</stddev> <!-- Giảm nhiễu -->
                     </rate>
                     <accel>

File: src/first_robot/description/robot.urdf.xacro (robot description, xacro)
@@ -3,4 +3,5 @@
     <xacro:arg name="prefix" default="" />
     <xacro:arg name="use_mock_hardware" default="true" />
+    <xacro:include filename="$(find first_robot)/description/constants.xacro"/>
     <xacro:include filename="inertial_base.xacro" />
     <xacro:include filename="robot_core.xacro" />

File: src/first_robot/description/robot_core.xacro (robot description, xacro)
@@ -1,43 +1,58 @@
 <?xml version="1.0"?>
 <robot xmlns:xacro="http://www.ros.org/wiki/xacro">
-    <!-- IMPORT MATERIAL -->
-    <xacro:include filename="$(find first_robot)/description/constants.xacro"/>
-    <!-- BASE LINK -->
-    <link name="base_link">
-        <visual name="base_link_visual">
-            <origin xyz="0 0 0.0125" />
-            <geometry>
-                <box size="0.2 0.15 0.05" />
-            </geometry>
-            <material name="white" />
-        </visual>
-        <collision name="base_link_collision">
-            <origin xyz="0 0 0.025" />
-            <!-- Sửa tâm va chạm -->
-            <geometry>
-                <box size="0.2 0.15 0.05" />
-            </geometry>
-        </collision>
-        <xacro:inertial_box mass="0.5" x="0.2" y="0.15" z="0.05">
-            <origin xyz="0 0 0.025" rpy="0 0 0" />
-        </xacro:inertial_box>
+  <!-- Base -->
+  <link name="base_link">
+    <visual name="base_link_visual">
+      <origin rpy="0 0 0" xyz="0 0 0"/>
+      <geometry>
+        <box size="0.001 0.001 0.001"/>
+      </geometry>
+      <material name="white" />
+    </visual>
+    <!-- collision & inertial -->
+  </link>
+  <joint name="floating_base" type="fixed">
+    <parent link="base_link"/>
+    <child link="trunk"/>
+    <origin xyz="0 0 0" rpy="0 0 0"/>
+  </joint>
+  <!-- Trunk : Thân robot -->
+  <link name="trunk">
+    <visual name="trunk_visual">
+      <origin rpy="0 0 0" xyz="0 0 0"/>
+      <geometry>
+        <box size="${trunk_length} ${trunk_width} ${trunk_height}"/>
+      </geometry>
+      <material name="silver"/>
+    </visual>
+    <collision name="trunk_collision">
+      <origin rpy="0 0 0" xyz="0 0 0"/>
+      <geometry>
+        <box size="${trunk_length} ${trunk_width} ${trunk_height}"/>
+      </geometry>
+    </collision>
+    <inertial>
+      <origin rpy="0 0 0" xyz="${trunk_com_x} ${trunk_com_y} ${trunk_com_z}"/>
+      <mass value="${trunk_mass}"/>
+      <inertia ixx="${trunk_ixx}" ixy="${trunk_ixy}" ixz="${trunk_ixz}" iyy="${trunk_iyy}" iyz="${trunk_iyz}" izz="${trunk_izz}"/>
+    </inertial>
     </link>
     <!-- Front Body -->
     <link name="front_body">
-        <visual name="front_body_visual">
-            <geometry>
-                 <box size="0.05 0.1 0.05"/>
-            </geometry>
-            <material name="pink"/>
-        </visual>
-        <collision name="front_body_collision">
-            <geometry>
-                 <box size="0.05 0.1 0.025"/>
-            </geometry>
-        </collision>
-        <inertial>
-            <mass value="1.0"/>
-            <inertia ixx="0.01" ixy="0" ixz="0" iyy="0.01" iyz="0" izz="0.01"/>
-        </inertial>
+      <visual name="front_body_visual">
+        <geometry>
+          <box size="0.05 0.1 0.05"/>
+        </geometry>
+        <material name="pink"/>
+      </visual>
+      <collision name="front_body_collision">
+        <geometry>
+          <box size="0.05 0.1 0.025"/>
+        </geometry>
+      </collision>
+      <inertial>
+        <mass value="1.0"/>
+        <inertia ixx="0.01" ixy="0" ixz="0" iyy="0.01" iyz="0" izz="0.01"/>
+      </inertial>
     </link>
     <!-- Joint nối base_link và front_body -->
@@ -45,5 +60,6 @@
       <parent link="base_link"/>
       <child link="front_body"/>
-      <origin xyz="0.1 0 0" rpy="0 0 0"/> <!-- Đẩy về trước cho cân đối -->
+      <origin xyz="0.1 0 0" rpy="0 0 0"/>
+      <!-- Đẩy về trước cho cân đối -->
     </joint>
     <!-- Rear Body -->
@@ -69,12 +85,13 @@
       <parent link="base_link"/>
       <child link="rear_body"/>
-       <origin xyz="-0.1 0 0" rpy="0 0 0"/> <!-- Đẩy về sau cho cân đối -->
+      <origin xyz="-0.1 0 0" rpy="0 0 0"/>
+      <!-- Đẩy về sau cho cân đối -->
     </joint>
     <!-- IMPORT LEG PATTERN -->
-    <xacro:include filename="$(find first_robot)/description/leg_block.xacro"/>
+    <xacro:include filename="$(find first_robot)/description/leg_block_v2.xacro"/>
     <!-- Gọi macro leg cho từng chân -->
-    <xacro:leg prefix="front_left" pos="front" side="left" x=" 0.075" y=" 0.05" />
-    <xacro:leg prefix="front_right" pos="front" side="right" x=" 0.075" y="-0.05" />
-    <xacro:leg prefix="rear_left" pos="rear" side="left" x="-0.075" y=" 0.05" />
-    <xacro:leg prefix="rear_right" pos="rear" side="right" x="-0.075" y="-0.05" />
-</robot>
+    <xacro:leg prefix="front_left" side="-1" use_dae="False" pos="1" />
+    <xacro:leg prefix="front_right" side="1" use_dae="False" pos="1"/>
+    <xacro:leg prefix="rear_left" side="-1" use_dae="False" pos="-1" />
+    <xacro:leg prefix="rear_right" side="1" use_dae="False" pos="-1" />
+  </robot>
