Commit message: convert design to unitree go2 formating

File: src/robot.urdf (robot description, URDF)
Before this commit: robot my_robot, 31 links, 30 joints
Links:
- removed link front_left_hip_motor_link
- removed link front_left_knee_motor_link
- removed link front_right_hip_motor_link
- removed link front_right_knee_motor_link
- removed link rear_left_hip_motor_link
- removed link rear_left_knee_motor_link
- removed link rear_right_hip_motor_link
- removed link rear_right_knee_motor_link
- added link trunk, mass 6.921; collision box size=0.3762 0.0935 0.114; visual box size=0.3762 0.0935 0.114
- link base_link: mass 0.5 -> None; geometry visual box size=0.001 0.001 0.001
- link camera_link: mass None -> 0.001; geometry collision sphere radius=0.001; visual sphere radius=0.001
- link front_left_ankle_link: mass 0.2 -> 0.154; geometry collision box size=0.223 0.026000000000000002 0.026000000000000002; visual box size=0.213 0.016 0.016
- link front_left_foot_link: mass 0.05 -> 0.06; geometry collision sphere radius=0.02; visual sphere radius=0.01
- link front_left_hip_link: mass 0.2 -> 0.678; geometry collision cylinder length=0.05 radius=0.056; visual cylinder length=0.04 radius=0.046
- link front_left_knee_link: mass 0.5 -> 1.152; geometry collision box size=0.223 0.0345 0.044000000000000004; visual box size=0.213 0.0245 0.034
- link front_right_ankle_link: mass 0.2 -> 0.154; geometry collision box size=0.223 0.026000000000000002 0.026000000000000002; visual box size=0.213 0.016 0.016
- link front_right_foot_link: mass 0.05 -> 0.06; geometry collision sphere radius=0.02; visual sphere radius=0.01
- link front_right_hip_link: mass 0.2 -> 0.678; geometry collision cylinder length=0.05 radius=0.056; visual cylinder length=0.04 radius=0.046
- link front_right_knee_link: mass 0.5 -> 1.152; geometry collision box size=0.223 0.0345 0.044000000000000004; visual box size=0.213 0.0245 0.034
- link imu_link: mass 0.01 -> 0.001; geometry collision box size=.001 .001 .001; visual box size=0.001 0.001 0.001
- link rear_left_ankle_link: mass 0.2 -> 0.154; geometry collision box size=0.223 0.026000000000000002 0.026000000000000002; visual box size=0.213 0.016 0.016
- link rear_left_foot_link: mass 0.05 -> 0.06; geometry collision sphere radius=0.02; visual sphere radius=0.01
- link rear_left_hip_link: mass 0.2 -> 0.678; geometry collision cylinder length=0.05 radius=0.056; visual cylinder length=0.04 radius=0.046
- link rear_left_knee_link: mass 0.5 -> 1.152; geometry collision box size=0.223 0.0345 0.044000000000000004; visual box size=0.213 0.0245 0.034
- link rear_right_ankle_link: mass 0.2 -> 0.154; geometry collision box size=0.223 0.026000000000000002 0.026000000000000002; visual box size=0.213 0.016 0.016
- link rear_right_foot_link: mass 0.05 -> 0.06; geometry collision sphere radius=0.02; visual sphere radius=0.01
- link rear_right_hip_link: mass 0.2 -> 0.678; geometry collision cylinder length=0.05 radius=0.056; visual cylinder length=0.04 radius=0.046
- link rear_right_knee_link: mass 0.5 -> 1.152; geometry collision box size=0.223 0.0345 0.044000000000000004; visual box size=0.213 0.0245 0.034
Joints:
- removed joint front_left_hip_motor_fixed
- removed joint front_left_knee_motor_fixed
- removed joint front_right_hip_motor_fixed
- removed joint front_right_knee_motor_fixed
- removed joint rear_left_hip_motor_fixed
- removed joint rear_left_knee_motor_fixed
- removed joint rear_right_hip_motor_fixed
- removed joint rear_right_knee_motor_fixed
- added joint floating_base: type fixed, parent base_link, child trunk, origin xyz=0 0 0 rpy=0 0 0
- joint camera_joint: origin xyz=0.10 0 0.04 rpy=0 0 0 -> xyz=0.326 0 0.043 rpy=0 0 0
- joint front_left_ankle_joint: axis 1 1 0 -> 0 1 0; limit lower=-1.57 upper=1.57 effort=30 velocity=7.0 -> lower=-1.0 upper=1.0 effort=35.55 velocity=20.06; origin xyz=0.08 0.04 0 rpy=0.12 0.45 0 -> xyz=0 0 -0.213 rpy=0 0 0; parent front_left_knee_motor_link -> front_left_knee_link
- joint front_left_foot_joint: origin xyz=0 0 -0.05 rpy=0 0 0 -> xyz=0.15055376357544295 0 -0.15067370133261354 rpy=0 0 0
- joint front_left_hip_joint: axis (none) -> 1 0 0; limit lower=-1.57 upper=1.57 effort=30 velocity=7.0 -> lower=-1.0472 upper=1.0472 effort=23.7 velocity=30.1; origin xyz=0 0 0.0 rpy=0 0 0 -> xyz=0.1934 0.0465 0 rpy=0 0 0; parent front_body -> trunk
- joint front_left_knee_joint: origin xyz=0 0 0 rpy=0.3 0.1 0 -> xyz=0 0.0955 0 rpy=0 0 0; parent front_left_hip_motor_link -> front_left_hip_link
- joint front_right_ankle_joint: axis 1 1 0 -> 0 1 0; limit lower=-1.57 upper=1.57 effort=30 velocity=7.0 -> lower=-1.0 upper=1.0 effort=35.55 velocity=20.06; origin xyz=0.08 -0.04 0 rpy=-0.12 0.45 0 -> xyz=0 0 -0.213 rpy=0 0 0; parent front_right_knee_motor_link -> front_right_knee_link
- joint front_right_foot_joint: origin xyz=0 0 -0.05 rpy=0 0 0 -> xyz=0.15055376357544295 0 -0.15067370133261354 rpy=0 0 0
- joint front_right_hip_joint: axis (none) -> 1 0 0; limit lower=-1.57 upper=1.57 effort=30 velocity=7.0 -> lower=-1.0472 upper=1.0472 effort=23.7 velocity=30.1; origin xyz=0 0 0.0 rpy=0 0 0 -> xyz=0.1934 -0.0465 0 rpy=0 0 0; parent front_body -> trunk
- joint front_right_knee_joint: origin xyz=0 0 0 rpy=-0.3 0.1 0 -> xyz=0 -0.0955 0 rpy=0 0 0; parent front_right_hip_motor_link -> front_right_hip_link
- joint imu_joint: origin xyz=0 0 0.05 -> xyz=0 0 0.05 rpy=0 0 0; parent base_link -> trunk
- joint rear_left_ankle_joint: axis 1 1 0 -> 0 1 0; limit lower=-1.57 upper=1.57 effort=30 velocity=7.0 -> lower=-1.0 upper=1.0 effort=35.55 velocity=20.06; origin xyz=0.08 0.04 0 rpy=0.12 0.45 0 -> xyz=0 0 -0.213 rpy=0 0 0; parent rear_left_knee_motor_link -> rear_left_knee_link
- joint rear_left_foot_joint: origin xyz=0 0 -0.05 rpy=0 0 0 -> xyz=0.15055376357544295 0 -0.15067370133261354 rpy=0 0 0
- joint rear_left_hip_joint: axis (none) -> 1 0 0; limit lower=-1.57 upper=1.57 effort=30 velocity=7.0 -> lower=-1.0472 upper=1.0472 effort=23.7 velocity=30.1; origin xyz=0 0 0.0 rpy=0 0 0 -> xyz=-0.1934 0.0465 0 rpy=0 0 0; parent rear_body -> trunk
- joint rear_left_knee_joint: origin xyz=0 0 0 rpy=0.3 0.1 0 -> xyz=0 0.0955 0 rpy=0 0 0; parent rear_left_hip_motor_link -> rear_left_hip_link
- joint rear_right_ankle_joint: axis 1 1 0 -> 0 1 0; limit lower=-1.57 upper=1.57 effort=30 velocity=7.0 -> lower=-1.0 upper=1.0 effort=35.55 velocity=20.06; origin xyz=0.08 -0.04 0 rpy=-0.12 0.45 0 -> xyz=0 0 -0.213 rpy=0 0 0; parent rear_right_knee_motor_link -> rear_right_knee_link
- joint rear_right_foot_joint: origin xyz=0 0 -0.05 rpy=0 0 0 -> xyz=0.15055376357544295 0 -0.15067370133261354 rpy=0 0 0
- joint rear_right_hip_joint: axis (none) -> 1 0 0; limit lower=-1.57 upper=1.57 effort=30 velocity=7.0 -> lower=-1.0472 upper=1.0472 effort=23.7 velocity=30.1; origin xyz=0 0 0.0 rpy=0 0 0 -> xyz=-0.1934 -0.0465 0 rpy=0 0 0; parent rear_body -> trunk
- joint rear_right_knee_joint: origin xyz=0 0 0 rpy=-0.3 0.1 0 -> xyz=0 -0.0955 0 rpy=0 0 0; parent rear_right_hip_motor_link -> rear_right_hip_link

Commit message: update something

File: src/first_robot/description/camera.xacro (robot description, xacro)
@@ -4,28 +4,22 @@
         <parent link="base_link" />
         <child link="camera_link" />
-        <origin xyz="0.326 0 0.043"  rpy="0 0 0"/>
+        <origin xyz="0.190 0 0.043"  rpy="0 0 0"/>
     </joint>
-    <joint name="camera_optical_joint" type="fixed">
-        <parent link="camera_link" />
-        <child link="camera_link_optical" />
-        <origin xyz="0.05 0 0" rpy="${-pi/2} 0 ${-pi/2}" />
-    </joint>
-    <link name="camera_link_optical"></link>
     <link name="camera_link">
         <visual>
             <origin rpy="0 0 0" xyz="0 0 0"/>
             <geometry>
-                <sphere radius="0.001"/>
+                <sphere radius="0.005"/>
             </geometry>
-            <material name="cyan" />
+            <material name="red" />
         </visual>
         <collision>
             <origin rpy="0 0 0" xyz="0 0 0"/>
             <geometry>
-                <sphere radius="0.001"/>
+                <sphere radius="0.005"/>
             </geometry>
         </collision>
         <inertial>
-            <mass value="0.001"/>
+            <mass value="0.005"/>
             <origin rpy="0 0 0" xyz="0 0 0"/>
             <inertia ixx="0.0001" ixy="0" ixz="0" iyy="0.0001" iyz="0" izz="0.0001"/>

File: src/first_robot/description/constants.xacro (robot description, xacro)
@@ -52,5 +52,5 @@
     <xacro:property name="ankle_width" value="0.016"/>
     <xacro:property name="ankle_height" value="0.016"/>
-    <xacro:property name="foot_radius" value="0.02"/>
+    <xacro:property name="foot_radius" value="0.03"/>
     <xacro:property name="stick_radius" value="0.01"/>
     <xacro:property name="stick_length" value="0.2"/>

File: src/first_robot/description/gz_control.xacro (robot description, xacro)
@@ -14,4 +14,20 @@
       </joint>
     </xacro:macro>
+    <!-- Front Left Leg -->
+    <xacro:define_joint_interfaces joint_name="front_left_hip_joint" />
+    <xacro:define_joint_interfaces joint_name="front_left_knee_joint" />
+    <xacro:define_joint_interfaces joint_name="front_left_ankle_joint" />
+    <!-- Front Right Leg -->
+    <xacro:define_joint_interfaces joint_name="front_right_hip_joint" />
+    <xacro:define_joint_interfaces joint_name="front_right_knee_joint" />
+    <xacro:define_joint_interfaces joint_name="front_right_ankle_joint" />
+    <!-- Rear Left Leg -->
+    <xacro:define_joint_interfaces joint_name="rear_left_hip_joint" />
+    <xacro:define_joint_interfaces joint_name="rear_left_knee_joint" />
+    <xacro:define_joint_interfaces joint_name="rear_left_ankle_joint" />
+    <!-- Rear Right Leg -->
+    <xacro:define_joint_interfaces joint_name="rear_right_hip_joint" />
+    <xacro:define_joint_interfaces joint_name="rear_right_knee_joint" />
+    <xacro:define_joint_interfaces joint_name="rear_right_ankle_joint" />
   </ros2_control>
   <gazebo>

File: src/first_robot/description/imu_link.xacro (robot description, xacro)
@@ -3,25 +3,26 @@
     <link name="imu_link">
         <inertial>
-            <mass value="0.001"/>
-            <origin rpy="0 0 0" xyz="0 0 0"/>
-            <inertia ixx="0.0001" ixy="0" ixz="0" iyy="0.0001" iyz="0" izz="0.0001"/>
+            <mass value="0.001" />
+            <origin rpy="0 0 0" xyz="0 0 0" />
+            <inertia ixx="0.0001" ixy="0" ixz="0" iyy="0.0001" iyz="0" izz="0.0001" />
         </inertial>
         <visual>
-            <origin rpy="0 0 0" xyz="0 0 0"/>
+            <origin rpy="0 0 0" xyz="0 0 0" />
             <geometry>
-                <box size="0.001 0.001 0.001"/>
+                <box size="0.001 0.001 0.01" />
             </geometry>
+            <material name="yellow" />
         </visual>
         <collision>
-            <origin rpy="0 0 0" xyz="0 0 0"/>
+            <origin rpy="0 0 0" xyz="0 0 0" />
             <geometry>
-                <box size=".001 .001 .001"/>
+                <box size=".001 .001 .01" />
             </geometry>
         </collision>
     </link>
     <joint name="imu_joint" type="fixed">
-        <parent link="trunk"/>
-        <child link="imu_link"/>
-        <origin xyz="0 0 0.05" rpy="0 0 0" />
+        <parent link="trunk" />
+        <child link="imu_link" />
+        <origin xyz="0 0 0.1" rpy="0 0 0" />
         <!-- Đặt IMU gần trọng tâm -->
     </joint>

File: src/first_robot/description/leg_block_v2.xacro (robot description, xacro)
@@ -2,8 +2,8 @@
 <robot xmlns:xacro="http://www.ros.org/wiki/xacro">
   <!-- Định nghĩa macro cho một chân -->
-  <!-- prefix: Tên của chân lf: front_left, rf: front_right, lh: rear_left, rh: rear_right     -->
-  <!-- side: Chân đối xứng với chân này 1: bên phải, -1: bên trái. Dùng để nhân chia với tọa độ -->
-  <!-- use_dae: Sử dụng mesh hay không True: sử dụng, False: không sử dụng -->
-  <!-- pos: Chân trước hay chân sau (1: chân trước, -1: chân sau) -->
+  <!-- prefix  Tên của chân lf  front left  rf  front right  lh  rear left  rh  rear right     -->
+  <!-- side  Chân đối xứng với chân này 1 bên phải  âm 1  bên trái  Dùng để nhân chia với tọa độ -->
+  <!-- use dae  Sử dụng mesh hay không True  sử dụng  False  không sử dụng -->
+  <!-- pos  Chân trước hay chân sau  1  chân trước  âm 1  chân sau-->
   <xacro:macro name="leg" params="prefix side pos use_dae">
     <!-- bắt đầu phần háng -->
@@ -11,23 +11,23 @@
     <link name="${prefix}_hip_link">
       <visual name="${prefix}_hip_visual">
-        <!-- Chân trái và phía trước -->
+        <!-- Chân phải và phía trước -->
         <xacro:if value="${(side == 1) and (pos == 1)}">
-          <origin rpy="0 0 0" xyz="0 0 0"/>
+          <origin rpy="${PI/2.0} 2.0 0" xyz="0 0 0"/>
         </xacro:if>
         <!-- Chân trái và phía sau -->
         <xacro:if value="${(side == 1) and (pos == -1)}">
-          <origin rpy="${PI} 0 0" xyz="0 0 0"/>
+          <origin rpy="${PI/2.0} 2.0 0" xyz="0 0 0"/>
         </xacro:if>
-        <!-- Chân phải và phía trước -->
+        <!-- Chân trái và phía trước -->
         <xacro:if value="${(side == -1) and (pos == 1)}">
-          <origin rpy="0 ${PI} 0" xyz="0 0 0"/>
+          <origin rpy="${PI/2.0} 2.0 0" xyz="0 0 0"/>
         </xacro:if>
         <!-- Chân phải và phía sau -->
         <xacro:if value="${(side == -1) and (pos == -1)}">
-          <origin rpy="${PI} ${PI} 0" xyz="0 0 0"/>
+          <origin rpy="${PI/2.0} 2.0 0" xyz="0 0 0"/>
         </xacro:if>
         <geometry>
           <cylinder length="${hip_length}" radius="${hip_radius}"/>
-          <!-- dài 2cm, cố định thân trên và các chân -->
+          <!-- dài 2cm  cố định thân trên và các chân -->
         </geometry>
         <material name="blue"/>
@@ -91,5 +91,5 @@
       </inertial>
     </link>
-    <!-- knee Joint (Đùi, quay về sau ) -->
+    <!-- knee Joint  Đùi  quay về sau  -->
     <joint name="${prefix}_knee_joint" description="Knee joint side ${side} and pos ${pos}" type="revolute">
       <origin rpy="0 0 0" xyz="0 ${knee_offset*-side} 0"/>
@@ -121,10 +121,10 @@
       </collision>
       <inertial>
-        <origin rpy="00.785 0" xyz="${ankle_com_x} ${ankle_com_y} ${ankle_com_z}"/>
+        <origin rpy="0 0.785 0" xyz="${ankle_com_x} ${ankle_com_y} ${ankle_com_z}"/>
         <mass value="${ankle_mass}"/>
         <inertia ixx="${ankle_ixx}" ixy="${ankle_ixy}" ixz="${ankle_ixz}" iyy="${ankle_iyy}" iyz="${ankle_iyz}" izz="${ankle_izz}"/>
       </inertial>
     </link>
-    <!-- ankle Joint (Cẳng chân, quay về trước 45°) -->
+    <!-- ankle Joint  Cẳng chân  quay về trước 45  -->
     <joint name="${prefix}_ankle_joint" type="revolute">
       <origin rpy="0 0 0" xyz="0 0 ${-ankle_length}"/>
@@ -142,5 +142,5 @@
         <origin rpy="0 0 0" xyz="0 0 0"/>
         <geometry>
-          <sphere radius="${foot_radius-0.01}"/>
+          <sphere radius="${foot_radius}"/>
         </geometry>
         <material name="black"/>
@@ -159,29 +159,8 @@
     <!-- Foot Joint -->
     <joint name="${prefix}_foot_joint" type="fixed">
-       <origin rpy="0 0 0" xyz="${ankle_length/2*sin(0.785)} 0 ${-ankle_length*cos(0.785)}"/>
+       <origin rpy="0 0 0" xyz="${(ankle_length)/2*sin(0.785) } 0 ${-(ankle_length)*cos(0.785) - 0.02}"/>
       <parent link="${prefix}_ankle_link"/>
       <child link="${prefix}_foot_link"/>
     </joint>
- <!-- *** Kết thúc phần bàn chân *** -->
-    <ros2_control name="${prefix}" type="system">
-      <hardware>
-        <plugin>gz_ros2_control/GazeboSimSystem</plugin>
-      </hardware>
-      <joint name="${prefix}_hip_joint">
-        <command_interface name="effort"/>
-        <state_interface name="position"/>
-        <state_interface name="velocity"/>
-      </joint>
-      <joint name="${prefix}_knee_joint">
-        <command_interface name="effort"/>
-        <state_interface name="position"/>
-        <state_interface name="velocity"/>
-      </joint>
-      <joint name="${prefix}_ankle_joint">
-        <command_interface name="effort"/>
-        <state_interface name="position"/>
-        <state_interface name="velocity"/>
-      </joint>
-    </ros2_control>
     <!-- Transmission cho các joint -->
     <transmission name="${prefix}_knee_trans">

File: src/first_robot/description/robot_core.xacro (robot description, xacro)
@@ -10,5 +10,4 @@
       <material name="white" />
     </visual>
-    <!-- collision & inertial -->
   </link>
   <joint name="floating_base" type="fixed">
@@ -17,5 +16,5 @@
     <origin xyz="0 0 0" rpy="0 0 0"/>
   </joint>
-  <!-- Trunk : Thân robot -->
+  <!-- Trunk  Thân robot -->
   <link name="trunk">
     <visual name="trunk_visual">
@@ -38,54 +37,4 @@
     </inertial>
     </link>
-    <!-- Front Body -->
-    <link name="front_body">
-      <visual name="front_body_visual">
-        <geometry>
-          <box size="0.05 0.1 0.05"/>
-        </geometry>
-        <material name="pink"/>
-      </visual>
-      <collision name="front_body_collision">
-        <geometry>
-          <box size="0.05 0.1 0.025"/>
-        </geometry>
-      </collision>
-      <inertial>
-        <mass value="1.0"/>
-        <inertia ixx="0.01" ixy="0" ixz="0" iyy="0.01" iyz="0" izz="0.01"/>
-      </inertial>
-    </link>
-    <!-- Joint nối base_link và front_body -->
-    <joint name="front_body_joint" type="fixed">
-      <parent link="base_link"/>
-      <child link="front_body"/>
-      <origin xyz="0.1 0 0" rpy="0 0 0"/>
-      <!-- Đẩy về trước cho cân đối -->
-    </joint>
-    <!-- Rear Body -->
-    <link name="rear_body">
-      <visual name="rear_body_visual">
-        <geometry>
-          <box size="0.02 0.02 0.1"/>
-        </geometry>
-        <material name="purple"/>
-      </visual>
-      <collision name="rear_body_collision">
-        <geometry>
-          <box size="0.02 0.02 0.1"/>
-        </geometry>
-      </collision>
-      <inertial>
-        <mass value="2.0"/>
-        <inertia ixx="0.01" ixy="0" ixz="0" iyy="0.01" iyz="0" izz="0.01"/>
-      </inertial>
-    </link>
-    <!-- Joint nối base_link và rear_body -->
-    <joint name="rear_body_joint" type="fixed">
-      <parent link="base_link"/>
-      <child link="rear_body"/>
-      <origin xyz="-0.1 0 0" rpy="0 0 0"/>
-      <!-- Đẩy về sau cho cân đối -->
-    </joint>
     <!-- IMPORT LEG PATTERN -->
     <xacro:include filename="$(find first_robot)/description/leg_block_v2.xacro"/>

File: src/robot.urdf (robot description, URDF)
Before this commit: robot my_robot, 24 links, 23 joints
Links:
- removed link camera_link_optical
- removed link front_body
- removed link rear_body
- link camera_link: mass 0.001 -> 0.005; geometry collision sphere radius=0.005; visual sphere radius=0.005
- link front_left_foot_link: geometry collision sphere radius=0.02; visual sphere radius=0.02
- link front_right_foot_link: geometry collision sphere radius=0.02; visual sphere radius=0.02
- link imu_link: geometry collision box size=.001 .001 .01; visual box size=0.001 0.001 0.01
- link rear_left_foot_link: geometry collision sphere radius=0.02; visual sphere radius=0.02
- link rear_right_foot_link: geometry collision sphere radius=0.02; visual sphere radius=0.02
Joints:
- removed joint camera_optical_joint
- removed joint front_body_joint
- removed joint rear_body_joint
- joint camera_joint: origin xyz=0.326 0 0.043 rpy=0 0 0 -> xyz=0.190 0 0.043 rpy=0 0 0
- joint front_left_foot_joint: origin xyz=0.15055376357544295 0 -0.15067370133261354 rpy=0 0 0 -> xyz=0.07527688178772148 0 -0.17067370133261353 rpy=0 0 0
- joint front_right_foot_joint: origin xyz=0.15055376357544295 0 -0.15067370133261354 rpy=0 0 0 -> xyz=0.07527688178772148 0 -0.17067370133261353 rpy=0 0 0
- joint imu_joint: origin xyz=0 0 0.05 rpy=0 0 0 -> xyz=0 0 0.1 rpy=0 0 0
- joint rear_left_foot_joint: origin xyz=0.15055376357544295 0 -0.15067370133261354 rpy=0 0 0 -> xyz=0.07527688178772148 0 -0.17067370133261353 rpy=0 0 0
- joint rear_right_foot_joint: origin xyz=0.15055376357544295 0 -0.15067370133261354 rpy=0 0 0 -> xyz=0.07527688178772148 0 -0.17067370133261353 rpy=0 0 0

Commit message: add sample mesh from unitree go2

File: src/first_robot/description/camera.xacro (robot description, xacro)
@@ -4,5 +4,5 @@
         <parent link="base_link" />
         <child link="camera_link" />
-        <origin xyz="0.190 0 0.043"  rpy="0 0 0"/>
+        <origin xyz="0.25 0 0.043"  rpy="0 0 0"/>
     </joint>
     <link name="camera_link">

File: src/first_robot/description/constants.xacro (robot description, xacro)
@@ -57,5 +57,5 @@
     <!-- dynamics inertial value -->
     <!-- trunk -->
-    <xacro:property name="trunk_mass" value="6.921"/>
+    <xacro:property name="trunk_mass" value="4.921"/>
     <xacro:property name="trunk_com_x" value="0.021112"/>
     <xacro:property name="trunk_com_y" value="0.00"/>
@@ -118,5 +118,5 @@
     <!-- dynamics inertial value -->
     <!-- trunk -->
-    <xacro:property name="trunk_mass" value="6.921"/>
+    <xacro:property name="trunk_mass" value="4.921"/>
     <xacro:property name="trunk_com_x" value="0.021112"/>
     <xacro:property name="trunk_com_y" value="0.00"/>
@@ -140,5 +140,5 @@
     <xacro:property name="hip_izz" value="0.000596"/>
     <!-- knee -->
-    <xacro:property name="knee_mass" value="1.152"/>
+    <xacro:property name="knee_mass" value="0.135862"/>
     <xacro:property name="knee_com_x" value="-0.00374"/>
     <xacro:property name="knee_com_y" value="-0.0223"/>

File: src/first_robot/description/lidar_2d_camera.xacro (robot description, xacro)
@@ -4,5 +4,5 @@
         <parent link="base_link" />
         <child link="lidar_link" />
-        <origin xyz="0.05 0 0.045" rpy="0 0 0" />
+        <origin xyz="0 0 0" rpy="0 0 0" />
     </joint>
     <link name="lidar_link">

File: src/first_robot/description/robot_core.xacro (robot description, xacro)
@@ -21,5 +21,6 @@
       <origin rpy="0 0 0" xyz="0 0 0"/>
       <geometry>
-        <box size="${trunk_length} ${trunk_width} ${trunk_height}"/>
+          <!-- <box size="${trunk_length} ${trunk_width} ${trunk_height}"/> -->
+          <mesh filename="file://$(find first_robot)/meshes/trunk.dae" scale="1 1 1"/>
       </geometry>
       <material name="silver"/>
@@ -38,5 +39,5 @@
     </link>
     <!-- IMPORT LEG PATTERN -->
-    <xacro:include filename="$(find first_robot)/description/leg_block_v2.xacro"/>
+    <xacro:include filename="$(find first_robot)/description/leg_block_v3.xacro"/>
     <!-- Gọi macro leg cho từng chân -->
     <xacro:leg prefix="front_left" side="-1" use_dae="False" pos="1" />
