Commit message: run simple robot for jazzy

File: src/first_robot/description/gz_control.xacro (robot description, xacro)
@@ -1,21 +1,29 @@
 <?xml version="1.0"?>
 <robot xmlns:xacro="http://www.ros.org/wiki/xacro" >
-    <gazebo>
-        <plugin name="ros2_control" filename="libgz_ros2_control_system.so">
-            <!-- Wheel Information -->
-            <left_joint>left_wheel_joint</left_joint>
-            <right_joint>right_wheel_joint</right_joint>
-            <wheel_separation>0.35</wheel_separation>
-            <wheel_diameter>0.1</wheel_diameter>
-            <!-- Limits -->
-            <max_wheel_torque>200</max_wheel_torque>
-            <max_wheel_acceleration>10.0</max_wheel_acceleration>
-            <!-- Output -->
-            <odometry_frame>odom</odometry_frame>
-            <robot_base_frame>base_link</robot_base_frame>
-            <publish_odom>true</publish_odom>
-            <publish_odom_tf>true</publish_odom_tf>
-            <publish_wheel_tf>true</publish_wheel_tf>
-        </plugin>
-    </gazebo>
+    <xacro:arg name="use_mock_hardware" default="false" />
+    <ros2_control name="FirstRobot" type="system">
+        <!-- <xacro:unless value="${use_mock_hardware}">
+          <hardware>
+            <plugin>first_robot/DiffBotSystemHardware</plugin>
+            <param name="example_param_hw_start_duration_sec">0</param>
+            <param name="example_param_hw_stop_duration_sec">3.0</param>
+          </hardware>
+        </xacro:unless> -->
+        <xacro:if value="true">
+          <hardware>
+            <plugin>mock_components/GenericSystem</plugin>
+            <param name="calculate_dynamics">true</param>
+          </hardware>
+        </xacro:if>
+        <joint name="left_wheel_joint">
+          <command_interface name="velocity"/>
+          <state_interface name="position"/>
+          <state_interface name="velocity"/>
+        </joint>
+        <joint name="right_wheel_joint">
+          <command_interface name="velocity"/>
+          <state_interface name="position"/>
+          <state_interface name="velocity"/>
+        </joint>
+      </ros2_control>
 </robot>

File: src/first_robot/description/robot.urdf.xacro (robot description, xacro)
@@ -1,4 +1,6 @@
 <?xml version="1.0"?>
 <robot xmlns:xacro="http://www.ros.org/wiki/xacro"  name="robot">
+    <xacro:arg name="prefix" default="" />
+    <xacro:arg name="use_mock_hardware" default="false" />
     <xacro:include filename="robot_core.xacro" />
     <xacro:include filename="gz_control.xacro" />

Commit message: update \to run gazebo but not works

File: src/first_robot/description/gz_control.xacro (robot description, xacro)
@@ -1,7 +1,7 @@
 <?xml version="1.0"?>
-<robot xmlns:xacro="http://www.ros.org/wiki/xacro" >
-    <xacro:arg name="use_mock_hardware" default="false" />
-    <ros2_control name="FirstRobot" type="system">
-        <!-- <xacro:unless value="${use_mock_hardware}">
+<robot xmlns:xacro="http://www.ros.org/wiki/xacro">
+  <xacro:arg name="use_mock_hardware" default="false" />
+  <ros2_control name="FirstRobot" type="system">
+    <!-- <xacro:unless value="${use_mock_hardware}">
           <hardware>
             <plugin>first_robot/DiffBotSystemHardware</plugin>
@@ -10,20 +10,31 @@
           </hardware>
         </xacro:unless> -->
-        <xacro:if value="true">
-          <hardware>
-            <plugin>mock_components/GenericSystem</plugin>
-            <param name="calculate_dynamics">true</param>
-          </hardware>
-        </xacro:if>
-        <joint name="left_wheel_joint">
-          <command_interface name="velocity"/>
-          <state_interface name="position"/>
-          <state_interface name="velocity"/>
-        </joint>
-        <joint name="right_wheel_joint">
-          <command_interface name="velocity"/>
-          <state_interface name="position"/>
-          <state_interface name="velocity"/>
-        </joint>
-      </ros2_control>
+    <xacro:if value="true">
+      <hardware>
+        <plugin>mock_components/GenericSystem</plugin>
+        <param name="calculate_dynamics">true</param>
+      </hardware>
+    </xacro:if>
+    <joint name="left_wheel_joint">
+      <command_interface name="velocity" />
+      <state_interface name="position" />
+      <state_interface name="velocity" />
+    </joint>
+    <joint name="right_wheel_joint">
+      <command_interface name="velocity" />
+      <state_interface name="position" />
+      <state_interface name="velocity" />
+    </joint>
+  </ros2_control>
+  <!-- <gazebo>
+    <plugin name="gazebo_ros2_control" filename="libgazebo_ros2_control.so">
+      <robot_namespace>/</robot_namespace>
+    </plugin>
+  </gazebo> -->
+  <plugin filename="libgz_ros2_control-system.so" name="gz_ros2_control::GazeboRosControlPlugin">
+    <ros>
+      <namespace>/</namespace>
+      <parameter name="robot_description">robot_description</parameter>
+    </ros>
+  </plugin>
 </robot>

File: src/first_robot/description/lidar_2d_camera.xacro (robot description, xacro)
@@ -31,12 +31,15 @@
     <gazebo reference="laser_frame">
         <material>Gazebo/Black</material>
-        <sensor name="gpu_lidar" type="gpu_lidar">
-            <pose> 0 0 0 0 0 0 </pose>
-            <visualize>false</visualize>
-            <update_rate>10</update_rate>
+        <sensor name="lidar" type="gpu_lidar">
+            <always_on>true</always_on>
+            <update_rate>30</update_rate>
+            <visualize>true</visualize>
+            <pose>0 0 0 0 0 0</pose>
+            <topic>/lidar_scan</topic>
             <ray>
                 <scan>
                     <horizontal>
                         <samples>360</samples>
+                        <resolution>1</resolution>
                         <min_angle>-3.14</min_angle>
                         <max_angle>3.14</max_angle>
@@ -44,15 +47,13 @@
                 </scan>
                 <range>
-                    <min>0.3</min>
-                    <max>12</max>
+                    <min>0.1</min>
+                    <max>10.0</max>
                 </range>
+                <noise>
+                    <type>gaussian</type>
+                    <mean>0.0</mean>
+                    <stddev>0.01</stddev>
+                </noise>
             </ray>
-            <plugin name="laser_controller" filename="libgazebo_ros_ray_sensor.so">
-                <ros>
-                    <argument>~/out:=scan</argument>
-                </ros>
-                <output_type>sensor_msgs/LaserScan</output_type>
-                <frame_name>laser_frame</frame_name>
-            </plugin>
         </sensor>
     </gazebo>

Commit message: add joints config for gazebo

File: src/first_robot/description/gz_control.xacro (robot description, xacro)
@@ -3,20 +3,26 @@
   <xacro:arg name="use_mock_hardware" default="false" />
   <ros2_control name="FirstRobot" type="system">
-    <xacro:if value="true">
-      <hardware>
-        <plugin>mock_components/GenericSystem</plugin>
-        <!-- <plugin>gazebo_ros2_control/GazeboSystem</plugin> -->
-        <param name="calculate_dynamics">true</param>
-      </hardware>
-    </xacro:if>
+    <hardware>
+      <xacro:if value="true">
+        <plugin>gz_ros2_control/GazeboSimSystem</plugin>
+      </xacro:if>
+    </hardware>
     <joint name="left_wheel_joint">
-      <command_interface name="velocity" />
-      <state_interface name="position" />
-      <state_interface name="velocity" />
+      <command_interface name="position">
+        <param name="min">-1</param>
+        <param name="max">1</param>
+      </command_interface>
+      <state_interface name="position"/>
+      <command_interface name="velocity"/>
+      <state_interface name="velocity"/>
     </joint>
     <joint name="right_wheel_joint">
-      <command_interface name="velocity" />
-      <state_interface name="position" />
-      <state_interface name="velocity" />
+      <command_interface name="position">
+        <param name="min">-1</param>
+        <param name="max">1</param>
+      </command_interface>
+      <state_interface name="position"/>
+      <command_interface name="velocity"/>
+      <state_interface name="velocity"/>
     </joint>
   </ros2_control>

File: src/first_robot/description/robot_core.xacro (robot description, xacro)
@@ -1,16 +1,16 @@
 <?xml version="1.0"?>
-<robot xmlns:xacro="http://www.ros.org/wiki/xacro" >
-    <xacro:include filename="inertial_macros.xacro"/>
+<robot xmlns:xacro="http://www.ros.org/wiki/xacro">
+    <xacro:include filename="inertial_macros.xacro" />
     <material name="white">
         <color rgba="1 1 1 1" />
     </material>
     <material name="orange">
-        <color rgba="1 0.3 0.1 1"/>
+        <color rgba="1 0.3 0.1 1" />
     </material>
     <material name="blue">
-        <color rgba="0.2 0.2 1 1"/>
+        <color rgba="0.2 0.2 1 1" />
     </material>
     <material name="black">
-        <color rgba="0 0 0 1"/>
+        <color rgba="0 0 0 1" />
     </material>
     <!-- BASE LINK -->
@@ -19,93 +19,109 @@
     <!-- CHASSIS LINK -->
     <joint name="chassis_joint" type="fixed">
-        <parent link="base_link"/>
-        <child link="chassis"/>
-        <origin xyz="-0.1 0 0"/>
+        <parent link="base_link" />
+        <child link="chassis" />
+        <origin xyz="-0.1 0 0" />
     </joint>
     <link name="chassis">
         <visual>
-            <origin xyz="0.15 0 0.075"/>
+            <origin xyz="0.15 0 0.075" />
             <geometry>
-                <box size="0.3 0.3 0.15"/>
+                <box size="0.3 0.3 0.15" />
             </geometry>
-            <material name="white"/>
+            <material name="white" />
         </visual>
         <collision>
-            <origin xyz="0.15 0 0.075"/>
+            <origin xyz="0.15 0 0.075" />
             <geometry>
-                <box size="0.3 0.3 0.15"/>
+                <box size="0.3 0.3 0.15" />
             </geometry>
         </collision>
         <xacro:inertial_box mass="0.5" x="0.3" y="0.3" z="0.15">
-            <origin xyz="0.15 0 0.075" rpy="0 0 0"/>
+            <origin xyz="0.15 0 0.075" rpy="0 0 0" />
         </xacro:inertial_box>
     </link>
     <!-- LEFT WHEEL LINK -->
     <joint name="left_wheel_joint" type="continuous">
-        <parent link="base_link"/>
-        <child link="left_wheel"/>
+        <hardwareInterface>hardware_interface/velocity</hardwareInterface>
+        <parent link="base_link" />
+        <child link="left_wheel" />
         <origin xyz="0 0.175 0" rpy="-${pi/2} 0 0" />
-        <axis xyz="0 0 1"/>
+        <axis xyz="0 0 1" />
     </joint>
     <link name="left_wheel">
         <visual>
             <geometry>
-                <cylinder radius="0.05" length="0.04"/>
+                <cylinder radius="0.05" length="0.04" />
             </geometry>
-            <material name="blue"/>
+            <material name="blue" />
         </visual>
         <collision>
             <geometry>
-                <cylinder radius="0.05" length="0.04"/>
+                <cylinder radius="0.05" length="0.04" />
             </geometry>
         </collision>
         <xacro:inertial_cylinder mass="0.1" length="0.04" radius="0.05">
-            <origin xyz="0 0 0" rpy="0 0 0"/>
+            <origin xyz="0 0 0" rpy="0 0 0" />
         </xacro:inertial_cylinder>
     </link>
     <!-- RIGHT WHEEL LINK -->
     <joint name="right_wheel_joint" type="continuous">
-        <parent link="base_link"/>
-        <child link="right_wheel"/>
+        <hardwareInterface>hardware_interface/velocity</hardwareInterface>
+        <parent link="base_link" />
+        <child link="right_wheel" />
         <origin xyz="0 -0.175 0" rpy="${pi/2} 0 0" />
-        <axis xyz="0 0 -1"/>
+        <axis xyz="0 0 -1" />
     </joint>
     <link name="right_wheel">
         <visual>
             <geometry>
-                <cylinder radius="0.05" length="0.04"/>
+                <cylinder radius="0.05" length="0.04" />
             </geometry>
-            <material name="blue"/>
+            <material name="blue" />
         </visual>
         <collision>
             <geometry>
-                <cylinder radius="0.05" length="0.04"/>
+                <cylinder radius="0.05" length="0.04" />
             </geometry>
         </collision>
         <xacro:inertial_cylinder mass="0.1" length="0.04" radius="0.05">
-            <origin xyz="0 0 0" rpy="0 0 0"/>
+            <origin xyz="0 0 0" rpy="0 0 0" />
         </xacro:inertial_cylinder>
     </link>
     <!-- CASTER WHEEL LINK -->
     <joint name="caster_wheel_joint" type="fixed">
-        <parent link="chassis"/>
-        <child link="caster_wheel"/>
-        <origin xyz="0.24 0 0"/>
+        <parent link="chassis" />
+        <child link="caster_wheel" />
+        <origin xyz="0.24 0 0" />
     </joint>
     <link name="caster_wheel">
         <visual>
             <geometry>
-                <sphere radius="0.05"/>
+                <sphere radius="0.05" />
             </geometry>
-            <material name="black"/>
+            <material name="black" />
         </visual>
         <collision>
             <geometry>
-                <sphere radius="0.05"/>
+                <sphere radius="0.05" />
             </geometry>
         </collision>
         <xacro:inertial_sphere mass="0.1" radius="0.05">
-            <origin xyz="0 0 0" rpy="0 0 0"/>
+            <origin xyz="0 0 0" rpy="0 0 0" />
         </xacro:inertial_sphere>
     </link>
+    <transmission name="left_wheel_trans">
+        <type>transmission_interface/SimpleTransmission</type>
+        <actuator name="left_wheel_motor">
+            <mechanicalReduction>1</mechanicalReduction>
+        </actuator>
+        <joint name="left_wheel_joint" />
+    </transmission>
+    <transmission name="right_wheel_trans">
+        <type>transmission_interface/SimpleTransmission</type>
+        <actuator name="right_wheel_motor">
+            <mechanicalReduction>1</mechanicalReduction>
+        </actuator>
+        <joint name="right_wheel_joint" />
+    </transmission>
 </robot>

Commit message: add camera, lidar not works for jazzy harmonic

File: src/first_robot/description/gz_control.xacro (robot description, xacro)
@@ -26,4 +26,22 @@
       <state_interface name="velocity"/>
     </joint>
+    <joint name="left_rear_wheel_joint">
+      <command_interface name="position">
+        <param name="min">-1</param>
+        <param name="max">1</param>
+      </command_interface>
+      <state_interface name="position"/>
+      <command_interface name="velocity"/>
+      <state_interface name="velocity"/>
+    </joint>
+    <joint name="right_rear_wheel_joint">
+      <command_interface name="position">
+        <param name="min">-1</param>
+        <param name="max">1</param>
+      </command_interface>
+      <state_interface name="position"/>
+      <command_interface name="velocity"/>
+      <state_interface name="velocity"/>
+    </joint>
   </ros2_control>
   <gazebo>

File: src/first_robot/description/robot.urdf.xacro (robot description, xacro)
@@ -6,3 +6,4 @@
     <xacro:include filename="gz_control.xacro" />
     <xacro:include filename="lidar_2d_camera.xacro" />
+    <xacro:include filename="camera.xacro" />
 </robot>

File: src/first_robot/description/robot_core.xacro (robot description, xacro)
@@ -15,5 +15,5 @@
     </material>
     <material name="red">
-        <color rgba="1 0 0 1"/>
+        <color rgba="1 0 0 1" />
     </material>
     <!-- BASE LINK -->
@@ -46,5 +46,5 @@
     <!-- LEFT WHEEL LINK -->
     <joint name="left_wheel_joint" type="continuous">
-        <dynamics damping="0.5"/>
+        <dynamics damping="0.5" />
         <hardwareInterface>hardware_interface/velocity</hardwareInterface>
         <parent link="base_link" />
@@ -71,5 +71,5 @@
     <!-- RIGHT WHEEL LINK -->
     <joint name="right_wheel_joint" type="continuous">
-        <dynamics damping="0.5"/>
+        <dynamics damping="0.5" />
         <hardwareInterface>hardware_interface/velocity</hardwareInterface>
         <parent link="base_link" />
@@ -79,4 +79,52 @@
     </joint>
     <link name="right_wheel">
+        <visual>
+            <geometry>
+                <cylinder radius="0.05" length="0.04" />
+            </geometry>
+            <material name="blue" />
+        </visual>
+        <collision>
+            <geometry>
+                <cylinder radius="0.05" length="0.04" />
+            </geometry>
+        </collision>
+        <xacro:inertial_cylinder mass="0.1" length="0.04" radius="0.05">
+            <origin xyz="0 0 0" rpy="0 0 0" />
+        </xacro:inertial_cylinder>
+    </link>
+    <joint name="left_rear_wheel_joint" type="continuous">
+        <dynamics damping="0.5" />
+        <hardwareInterface>hardware_interface/velocity</hardwareInterface>
+        <parent link="base_link" />
+        <child link="left_rear_wheel" />
+        <origin xyz="0.2 0.175 0" rpy="-${pi/2} 0 0" />
+        <axis xyz="0 0 1" />
+    </joint>
+    <link name="left_rear_wheel">
+        <visual>
+            <geometry>
+                <cylinder radius="0.05" length="0.04" />
+            </geometry>
+            <material name="blue" />
+        </visual>
+        <collision>
+            <geometry>
+                <cylinder radius="0.05" length="0.04" />
+            </geometry>
+        </collision>
+        <xacro:inertial_cylinder mass="0.1" length="0.04" radius="0.05">
+            <origin xyz="0 0 0" rpy="0 0 0" />
+        </xacro:inertial_cylinder>
+    </link>
+    <joint name="right_rear_wheel_joint" type="continuous">
+        <dynamics damping="0.5" />
+        <hardwareInterface>hardware_interface/velocity</hardwareInterface>
+        <parent link="base_link" />
+        <child link="right_rear_wheel" />
+        <origin xyz="0.2 -0.175 0" rpy="${pi/2} 0 0" />
+        <axis xyz="0 0 -1" />
+    </joint>
+    <link name="right_rear_wheel">
         <visual>
             <geometry>
@@ -130,3 +178,17 @@
         <joint name="right_wheel_joint" />
     </transmission>
+    <transmission name="left_rear_wheel_trans">
+        <type>transmission_interface/SimpleTransmission</type>
+        <actuator name="left_rear_wheel_motor">
+            <mechanicalReduction>3</mechanicalReduction>
+        </actuator>
+        <joint name="left_rear_wheel_joint" />
+    </transmission>
+    <transmission name="right_rear_wheel_trans">
+        <type>transmission_interface/SimpleTransmission</type>
+        <actuator name="right_rear_wheel_motor">
+            <mechanicalReduction>3</mechanicalReduction>
+        </actuator>
+        <joint name="right_rear_wheel_joint" />
+    </transmission>
 </robot>

Commit message: successfully add slam toolbox for map localization

File: src/first_robot/description/gz_control.xacro (robot description, xacro)
@@ -1,5 +1,5 @@
 <?xml version="1.0"?>
 <robot xmlns:xacro="http://www.ros.org/wiki/xacro">
-  <xacro:arg name="use_mock_hardware" default="false" />
+  <xacro:arg name="use_mock_hardware" default="true" />
   <ros2_control name="FirstRobot" type="system">
     <hardware>

File: src/first_robot/description/lidar_2d_camera.xacro (robot description, xacro)
@@ -2,44 +2,61 @@
 <robot xmlns:xacro="http://www.ros.org/wiki/xacro" >
     <joint name="laser_joint" type="fixed">
-        <parent link="chassis"/>
-        <child link="laser_frame"/>
-        <origin xyz="0.1 0 0.175" rpy="0 0 0"/>
+        <parent link="base_link" />
+        <child link="lidar_link" />
+        <origin xyz="0.1 0 0.175" rpy="0 0 0" />
     </joint>
-    <link name="laser_frame">
+    <link name="lidar_link">
         <visual>
             <geometry>
-                <cylinder radius="0.05" length="0.04"/>
+                <cylinder radius="0.05" length="0.04" />
             </geometry>
-            <material name="red"/>
+            <material name="red" />
         </visual>
         <collision>
             <geometry>
-                <cylinder radius="0.05" length="0.04"/>
+                <cylinder radius="0.05" length="0.04" />
             </geometry>
         </collision>
         <xacro:inertial_cylinder mass="0.1" length="0.04" radius="0.05">
-            <origin xyz="0 0 0" rpy="0 0 0"/>
+            <origin xyz="0 0 0" rpy="0 0 0" />
         </xacro:inertial_cylinder>
     </link>
-    <gazebo reference="laser_frame">
-        <material>Gazebo/Red</material>
-        <sensor name="gpu_lidar" type="gpu_lidar">
-            <pose>0 0 0 0 0 0</pose>
-            <update_rate>30</update_rate>
+    <gazebo reference="lidar_link">
+        <sensor name="lidar_link" type="gpu_lidar">
+            <always_on>true</always_on>
+            <update_rate>2</update_rate>
+            <topic>/scan</topic>
             <visualize>true</visualize>
-            <topic>scan</topic>
+            <frame_id>lidar_link</frame_id>
+            <gz_frame_id>lidar_link</gz_frame_id>
+            <ign_frame_id>lidar_link</ign_frame_id>
+            <ros>
+                <namespace>/</namespace>
+                <remapping>scan:=scan</remapping>
+            </ros>
             <ray>
                 <scan>
                     <horizontal>
-                        <samples>360</samples>
-                        <min_angle>-3.14</min_angle>
-                        <max_angle>3.14</max_angle>
+                        <samples>720</samples>
+                        <resolution>1</resolution>
+                        <min_angle>-1.5708</min_angle>
+                        <max_angle>1.5708</max_angle>
                     </horizontal>
                 </scan>
                 <range>
-                    <min>0.3</min>
-                    <max>12</max>
+                    <min>0.1</min>
+                    <max>10.0</max>
                 </range>
+                <noise>
+                    <type>gaussian</type>
+                    <mean>0.0</mean>
+                    <stddev>0.01</stddev>
+                </noise>
             </ray>
+            <!-- <plugin
+                filename="gz-sim-sensors-system"
+                name="gz::sim::systems::Sensors">
+                <render_engine>ogre</render_engine>
+            </plugin> -->
         </sensor>
     </gazebo>

File: src/first_robot/description/robot.urdf.xacro (robot description, xacro)
@@ -1,6 +1,6 @@
 <?xml version="1.0"?>
-<robot xmlns:xacro="http://www.ros.org/wiki/xacro" name="robot">
+<robot xmlns:xacro="http://www.ros.org/wiki/xacro" name="my_robot">
     <xacro:arg name="prefix" default="" />
-    <xacro:arg name="use_mock_hardware" default="false" />
+    <xacro:arg name="use_mock_hardware" default="true" />
     <xacro:include filename="robot_core.xacro" />
     <xacro:include filename="gz_control.xacro" />
