Commit message: update champ

File: src/first_robot/description/gz_control.xacro (robot description, xacro)
@@ -1,3 +1,2 @@
-<?xml version="1.0"?>
 <robot xmlns:xacro="http://www.ros.org/wiki/xacro">
   <xacro:arg name="use_mock_hardware" default="true" />
@@ -8,5 +7,4 @@
     </hardware>
     <!-- Joint Definitions -->
-    <!-- Repeat for all leg joints -->
     <xacro:macro name="define_joint_interfaces" params="joint_name">
       <joint name="${joint_name}">
@@ -18,23 +16,22 @@
     <!-- Front Left Leg -->
     <xacro:define_joint_interfaces joint_name="left_front_hip_joint"/>
-    <xacro:define_joint_interfaces joint_name="left_front_knee_joint"/>
-    <xacro:define_joint_interfaces joint_name="left_front_ankle_joint"/>
+    <xacro:define_joint_interfaces joint_name="left_front_upper_leg_joint"/>
+    <xacro:define_joint_interfaces joint_name="left_front_lower_leg_joint"/>
     <!-- Front Right Leg -->
     <xacro:define_joint_interfaces joint_name="right_front_hip_joint"/>
-    <xacro:define_joint_interfaces joint_name="right_front_knee_joint"/>
-    <xacro:define_joint_interfaces joint_name="right_front_ankle_joint"/>
+    <xacro:define_joint_interfaces joint_name="right_front_upper_leg_joint"/>
+    <xacro:define_joint_interfaces joint_name="right_front_lower_leg_joint"/>
     <!-- Rear Left Leg -->
     <xacro:define_joint_interfaces joint_name="left_rear_hip_joint"/>
-    <xacro:define_joint_interfaces joint_name="left_rear_knee_joint"/>
-    <xacro:define_joint_interfaces joint_name="left_rear_ankle_joint"/>
+    <xacro:define_joint_interfaces joint_name="left_rear_upper_leg_joint"/>
+    <xacro:define_joint_interfaces joint_name="left_rear_lower_leg_joint"/>
     <!-- Rear Right Leg -->
     <xacro:define_joint_interfaces joint_name="right_rear_hip_joint"/>
-    <xacro:define_joint_interfaces joint_name="right_rear_knee_joint"/>
-    <xacro:define_joint_interfaces joint_name="right_rear_ankle_joint"/>
+    <xacro:define_joint_interfaces joint_name="right_rear_upper_leg_joint"/>
+    <xacro:define_joint_interfaces joint_name="right_rear_lower_leg_joint"/>
   </ros2_control>
-  <!-- Gazebo plugin config -->
   <gazebo>
     <plugin filename="gz_ros2_control-system" name="gz_ros2_control::GazeboSimROS2ControlPlugin">
-      <parameters>$(find first_robot)/config/controller_test_snipdog.yaml</parameters>
+      <parameters>$(find first_robot)/config/ros_control.yaml</parameters>
     </plugin>
   </gazebo>

File: src/first_robot/description/leg_block.xacro (robot description, xacro)
@@ -92,5 +92,5 @@
   </joint>
   <!-- Knee Joint -->
-  <joint name="${prefix}_knee_joint" type="revolute">
+  <joint name="${prefix}_upper_leg_joint" type="revolute">
     <parent link="${prefix}_knee_motor_link"/>
     <child link="${prefix}_shank"/>
@@ -143,5 +143,5 @@
   </joint>
   <!-- Ankle Joint -->
-  <joint name="${prefix}_ankle_joint" type="revolute">
+  <joint name="${prefix}_lower_leg_joint" type="revolute">
     <parent link="${prefix}_ankle_motor_link"/>
     <child link="${prefix}_foot"/>

File: src/first_robot/description/robot.urdf.xacro (robot description, xacro)
@@ -1,12 +1,11 @@
 <?xml version="1.0"?>
 <robot xmlns:xacro="http://www.ros.org/wiki/xacro" name="my_robot">
+   <!-- need to compose all to single file? run: xacro first_robot/description/robot.urdf.xacro > robot.urdf -->
     <xacro:arg name="prefix" default="" />
     <xacro:arg name="use_mock_hardware" default="true" />
     <xacro:include filename="inertial_base.xacro" />
-    <!-- ROBOT BANH XE  -->
-    <!-- <xacro:include filename="robot_core_ver_four_wheel.xacro" /> -->
     <!-- ROBOT DOG  -->
     <xacro:include filename="robot_core.xacro" />
-    <xacro:include filename="gz_control_snipdog.xacro" />
+    <xacro:include filename="gz_control.xacro" />
     <xacro:include filename="lidar_2d_camera.xacro" />
     <xacro:include filename="camera.xacro" />

File: src/first_robot/description/transmission_block.xacro (robot description, xacro)
@@ -14,5 +14,5 @@
   <transmission name="${prefix}_knee_trans">
     <type>transmission_interface/SimpleTransmission</type>
-    <joint name="${prefix}_knee_joint">
+    <joint name="${prefix}_upper_leg_joint">
       <hardwareInterface>hardware_interface/PositionJointInterface</hardwareInterface>
     </joint>
@@ -24,5 +24,5 @@
   <transmission name="${prefix}_ankle_trans">
     <type>transmission_interface/SimpleTransmission</type>
-    <joint name="${prefix}_ankle_joint">
+    <joint name="${prefix}_lower_leg_joint">
       <hardwareInterface>hardware_interface/PositionJointInterface</hardwareInterface>
     </joint>

Commit message: improve naming convention

File: src/first_robot/description/gz_control.xacro (robot description, xacro)
@@ -9,25 +9,25 @@
     <xacro:macro name="define_joint_interfaces" params="joint_name">
       <joint name="${joint_name}">
-        <command_interface name="position"/>
-        <state_interface name="position"/>
-        <state_interface name="velocity"/>
+        <command_interface name="position" />
+        <state_interface name="position" />
+        <state_interface name="velocity" />
       </joint>
     </xacro:macro>
     <!-- Front Left Leg -->
-    <xacro:define_joint_interfaces joint_name="left_front_hip_joint"/>
-    <xacro:define_joint_interfaces joint_name="left_front_upper_leg_joint"/>
-    <xacro:define_joint_interfaces joint_name="left_front_lower_leg_joint"/>
+    <xacro:define_joint_interfaces joint_name="left_front_hip_joint" />
+    <xacro:define_joint_interfaces joint_name="left_front_knee_joint" />
+    <xacro:define_joint_interfaces joint_name="left_front_ankle_joint" />
     <!-- Front Right Leg -->
-    <xacro:define_joint_interfaces joint_name="right_front_hip_joint"/>
-    <xacro:define_joint_interfaces joint_name="right_front_upper_leg_joint"/>
-    <xacro:define_joint_interfaces joint_name="right_front_lower_leg_joint"/>
+    <xacro:define_joint_interfaces joint_name="right_front_hip_joint" />
+    <xacro:define_joint_interfaces joint_name="right_front_knee_joint" />
+    <xacro:define_joint_interfaces joint_name="right_front_ankle_joint" />
     <!-- Rear Left Leg -->
-    <xacro:define_joint_interfaces joint_name="left_rear_hip_joint"/>
-    <xacro:define_joint_interfaces joint_name="left_rear_upper_leg_joint"/>
-    <xacro:define_joint_interfaces joint_name="left_rear_lower_leg_joint"/>
+    <xacro:define_joint_interfaces joint_name="left_rear_hip_joint" />
+    <xacro:define_joint_interfaces joint_name="left_rear_knee_joint" />
+    <xacro:define_joint_interfaces joint_name="left_rear_ankle_joint" />
     <!-- Rear Right Leg -->
-    <xacro:define_joint_interfaces joint_name="right_rear_hip_joint"/>
-    <xacro:define_joint_interfaces joint_name="right_rear_upper_leg_joint"/>
-    <xacro:define_joint_interfaces joint_name="right_rear_lower_leg_joint"/>
+    <xacro:define_joint_interfaces joint_name="right_rear_hip_joint" />
+    <xacro:define_joint_interfaces joint_name="right_rear_knee_joint" />
+    <xacro:define_joint_interfaces joint_name="right_rear_ankle_joint" />
   </ros2_control>
   <gazebo>

File: src/first_robot/description/leg_block.xacro (robot description, xacro)
@@ -1,6 +1,12 @@
 <?xml version="1.0"?>
 <robot xmlns:xacro="http://ros.org/wiki/xacro">
-<xacro:macro name="leg" params="prefix x y">
-  <!-- Macro định nghĩa phần inertial (khối lượng, khối tâm, quán tính) -->
+  <xacro:property name="thigh_length" value="0.18" /> <!-- Length of thigh link m -->
+  <xacro:property name="shank_length" value="0.18" /> <!-- Length of shank link m -->
+  <xacro:property name="motor_mass" value="0.03" /> <!-- Mass of motor links kg -->
+  <xacro:property name="motor_radius" value="0.012" /> <!-- Radius of motor cylinders m -->
+  <xacro:property name="motor_length" value="0.02" /> <!-- Length of motor cylinders m -->
+  <xacro:property name="foot_radius" value="0.03" /> <!-- Radius of foot sphere m -->
+  <!--  INERTIAL MACRO  -->
+  <!-- Macro to calculate inertia for box-shaped links -->
   <xacro:macro name="inertial_box_leg" params="mass box_size">
     <inertial>
@@ -14,167 +20,183 @@
     </inertial>
   </xacro:macro>
-  <!-- Hip Motor Link -->
-  <link name="${prefix}_hip_motor_link">
-    <visual>
-      <origin xyz="0 0 0.005"/>
-      <geometry>
-        <cylinder length="0.02" radius="0.015"/>
-      </geometry>
-      <material name="grey"/>
-    </visual>
-    <collision>
-      <origin xyz="0 0 0.005"/>
-      <geometry>
-        <cylinder length="0.02" radius="0.015"/>
-      </geometry>
-    </collision>
-    <inertial>
-      <mass value="0.05"/>
-      <inertia ixx="0.00001" ixy="0.0" ixz="0.0" iyy="0.00001" iyz="0.0" izz="0.00001"/>
-    </inertial>
-  </link>
-  <!-- Fixed joint gắn hip motor vào chassis -->
-  <joint name="${prefix}_hip_motor_fixed" type="fixed">
-    <parent link="chassis"/>
-    <child link="${prefix}_hip_motor_link"/>
-    <origin xyz="${x} ${y} -0.005"/>
-  </joint>
-  <!-- Hip Joint -->
-  <joint name="${prefix}_hip_joint" type="revolute">
-    <parent link="${prefix}_hip_motor_link"/>
-    <child link="${prefix}_thigh"/>
-    <origin xyz="0 0 0"/>
-    <axis xyz="0 1 0"/>
-    <limit effort="5" velocity="2.0" lower="1.57" upper="-1.57"/><!-- Đảo dấu -->
-  </joint>
-  <!-- Thigh Link -->
-  <link name="${prefix}_thigh">
-    <visual>
-      <origin xyz="0 0 -0.06"/>
-      <geometry>
-        <box size="0.03 0.03 0.12"/> <!-- Giảm kích thước -->
-      </geometry>
-      <material name="blue"/>
-    </visual>
-    <collision>
-      <origin xyz="0 0 -0.06"/>
-      <geometry>
-        <box size="0.03 0.03 0.12"/>
-      </geometry>
-    </collision>
-    <xacro:inertial_box_leg mass="0.1" box_size="${[0.03, 0.03, 0.12]}"/> <!-- Giảm khối lượng -->
-  </link>
-  <!-- Knee Motor Link -->
-  <link name="${prefix}_knee_motor_link">
-    <visual>
-      <origin xyz="0 0 -0.01"/>
-      <geometry>
-        <cylinder length="0.02" radius="0.012"/>
-      </geometry>
-      <material name="grey"/>
-    </visual>
-    <collision>
-      <origin xyz="0 0 -0.01"/>
-      <geometry>
-        <cylinder length="0.02" radius="0.012"/>
-      </geometry>
-    </collision>
-    <inertial>
-      <mass value="0.03"/>
-      <inertia ixx="0.00001" ixy="0.0" ixz="0.0" iyy="0.00001" iyz="0.0" izz="0.00001"/>
-    </inertial>
-  </link>
-  <!-- Fixed joint gắn knee motor vào thigh -->
-  <joint name="${prefix}_knee_motor_fixed" type="fixed">
-    <parent link="${prefix}_thigh"/>
-    <child link="${prefix}_knee_motor_link"/>
-    <origin xyz="0 0 -0.12" rpy="0 0.3 0"/> <!-- Thêm góc nghiêng -->
-  </joint>
-  <!-- Knee Joint -->
-  <joint name="${prefix}_upper_leg_joint" type="revolute">
-    <parent link="${prefix}_knee_motor_link"/>
-    <child link="${prefix}_shank"/>
-    <origin xyz="0 0 0"/>
-    <axis xyz="0 1 0"/>
-    <limit effort="5" velocity="2.0" lower="-2.0" upper="2.0"/> <!-- Mở rộng góc -->
-  </joint>
-  <!-- Shank Link -->
-  <link name="${prefix}_shank">
-    <visual>
-      <origin xyz="0 0 -0.06"/>
-      <geometry>
-        <box size="0.02 0.02 0.12"/> <!-- Giảm kích thước -->
-      </geometry>
-      <material name="red"/>
-    </visual>
-    <collision>
-      <origin xyz="0 0 -0.06"/>
-      <geometry>
-        <box size="0.02 0.02 0.12"/>
-      </geometry>
-    </collision>
-    <xacro:inertial_box_leg mass="0.1" box_size="${[0.02, 0.02, 0.12]}"/> <!-- Giảm khối lượng -->
-  </link>
-  <!-- Ankle Motor Link -->
-  <link name="${prefix}_ankle_motor_link">
-    <visual>
-      <origin xyz="0 0 -0.01"/>
-      <geometry>
-        <cylinder length="0.02" radius="0.012"/>
-      </geometry>
-      <material name="grey"/>
-    </visual>
-    <collision>
-      <origin xyz="0 0 -0.01"/>
-      <geometry>
-        <cylinder length="0.02" radius="0.012"/>
-      </geometry>
-    </collision>
-    <inertial>
-      <mass value="0.03"/>
-      <inertia ixx="0.00001" ixy="0.0" ixz="0.0" iyy="0.00001" iyz="0.0" izz="0.00001"/>
-    </inertial>
-  </link>
-  <!-- Fixed joint gắn ankle motor vào shank -->
-  <joint name="${prefix}_ankle_motor_fixed" type="fixed">
-    <parent link="${prefix}_shank"/>
-    <child link="${prefix}_ankle_motor_link"/>
-    <origin xyz="0 0 -0.12" rpy="0 0.3 0"/> <!-- Thêm góc nghiêng -->
-  </joint>
-  <!-- Ankle Joint -->
-  <joint name="${prefix}_lower_leg_joint" type="revolute">
-    <parent link="${prefix}_ankle_motor_link"/>
-    <child link="${prefix}_foot"/>
-    <origin xyz="0 0 0"/>
-    <axis xyz="0 1 0"/>
-    <limit effort="5" velocity="2.0" lower="-2.0" upper="2.0"/> <!-- Mở rộng góc -->
-  </joint>
-  <!-- Foot Link -->
-  <link name="${prefix}_foot">
-    <visual>
-      <geometry>
-        <sphere radius="0.03"/>
-      </geometry>
-      <material name="black"/>
-    </visual>
-    <collision>
-      <geometry>
-        <sphere radius="0.03"/>
-      </geometry>
-    </collision>
-    <xacro:inertial_sphere mass="0.1" radius="0.03">
-       <origin xyz="0 0 0" rpy="0 0 0" />
-    </xacro:inertial_sphere>
-  </link>
-  <gazebo reference="${prefix}_foot">
-    <mu1>1.2</mu1> <!-- Tăng ma sát ngang -->
-    <mu2>1.2</mu2> <!-- Tăng ma sát dọc -->
-  </gazebo>
-  <!-- IMPORT LEG PATTERN -->
-  <xacro:include filename="$(find first_robot)/description/transmission_block.xacro"/>
-  <xacro:transmission_block prefix="left_front"/>
-  <xacro:transmission_block prefix="right_front"/>
-  <xacro:transmission_block prefix="left_rear"/>
-  <xacro:transmission_block prefix="right_rear"/>
-</xacro:macro>
+  <!--  LEG MACRO  -->
+  <!-- Macro to define a single leg with hip thigh knee shank ankle and foot -->
+  <xacro:macro name="leg" params="prefix x y">
+    <!--  HIP SECTION  -->
+    <!-- Hip motor link  Small cylindrical motor attached to chassis -->
+    <link name="${prefix}_hip_motor">
+      <visual>
+        <origin xyz="0 0 0.005" />
+        <geometry>
+          <cylinder length="${motor_length}" radius="${motor_radius}" />
+        </geometry>
+        <material name="grey" />
+      </visual>
+      <collision>
+        <origin xyz="0 0 0.005" />
+        <geometry>
+          <cylinder length="${motor_length}" radius="${motor_radius}" />
+        </geometry>
+      </collision>
+      <inertial>
+        <mass value="${motor_mass}" />
+        <inertia ixx="0.00001" ixy="0.0" ixz="0.0" iyy="0.00001" iyz="0.0" izz="0.00001" />
+      </inertial>
+    </link>
+    <!-- Hip motor mount  Fixed joint attaching hip motor to chassis -->
+    <joint name="${prefix}_hip_motor_mount" type="fixed">
+      <parent link="chassis" />
+      <child link="${prefix}_hip_motor" />
+      <origin xyz="${x} ${y} -0.005" />
+    </joint>
+    <!-- Hip joint  Revolute joint for thigh rotation, limited to forward motion -->
+    <joint name="${prefix}_hip_joint" type="revolute">
+      <parent link="${prefix}_hip_motor" />
+      <child link="${prefix}_thigh" />
+      <origin xyz="0 0 0" />
+      <axis xyz="0 1 0" /> <!-- Rotation around y-axis -->
+      <limit effort="5" velocity="2.0" lower="-1.57" upper="0" /> <!-- Forward motion only -->
+    </joint>
+    <!-- Thigh link  Box-shaped link connecting hip to knee -->
+    <link name="${prefix}_thigh">
+      <visual>
+        <origin xyz="0 0 -${thigh_length/2}" /> <!-- Center of thigh -->
+        <geometry>
+          <box size="0.03 0.03 ${thigh_length}" />
+        </geometry>
+        <material name="blue" />
+      </visual>
+      <collision>
+        <origin xyz="0 0 -${thigh_length/2}" />
+        <geometry>
+          <box size="0.03 0.03 ${thigh_length}" />
+        </geometry>
+      </collision>
+      <xacro:inertial_box_leg mass="0.15" box_size="${[0.03, 0.03, thigh_length]}" />
+    </link>
+    <!--  KNEE SECTION  -->
+    <!-- Knee motor link  Small cylindrical motor attached to thigh -->
+    <link name="${prefix}_knee_motor">
+      <visual>
+        <origin xyz="0 0 -0.01" />
+        <geometry>
+          <cylinder length="${motor_length}" radius="${motor_radius}" />
+        </geometry>
+        <material name="grey" />
+      </visual>
+      <collision>
+        <origin xyz="0 0 -0.01" />
+        <geometry>
+          <cylinder length="${motor_length}" radius="${motor_radius}" />
+        </geometry>
+      </collision>
+      <inertial>
+        <mass value="${motor_mass}" />
+        <inertia ixx="0.00001" ixy="0.0" ixz="0.0" iyy="0.00001" iyz="0.0" izz="0.00001" />
+      </inertial>
+    </link>
+    <!-- Knee motor mount  Fixed joint attaching knee motor to thigh -->
+    <joint name="${prefix}_knee_motor_mount" type="fixed">
+      <parent link="${prefix}_thigh" />
+      <child link="${prefix}_knee_motor" />
+      <origin xyz="0 0 -${thigh_length}" rpy="0 -0.3 0" /> <!-- Tilt forward for natural posture -->
+    </joint>
+    <!-- Knee joint  Revolute joint for shank rotation, limited to forward motion -->
+    <joint name="${prefix}_knee_joint" type="revolute">
+      <parent link="${prefix}_knee_motor" />
+      <child link="${prefix}_shank" />
+      <origin xyz="0 0 0" />
+      <axis xyz="0 1 0" /> <!-- Rotation around y axis -->
+      <limit effort="5" velocity="2.0" lower="-2.5" upper="0" /> <!-- Forward motion only -->
+    </joint>
+    <!-- Shank link  Box-shaped link connecting knee to ankle -->
+    <link name="${prefix}_shank">
+      <visual>
+        <origin xyz="0 0 -${shank_length/2}" />
+        <geometry>
+          <box size="0.02 0.02 ${shank_length}" />
+        </geometry>
+        <material name="red" />
+      </visual>
+      <collision>
+        <origin xyz="0 0 -${shank_length/2}" />
+        <geometry>
+          <box size="0.02 0.02 ${shank_length}" />
+        </geometry>
+      </collision>
+      <xacro:inertial_box_leg mass="0.15" box_size="${[0.02, 0.02, shank_length]}" />
+    </link>
+    <!--  ANKLE SECTION  -->
+    <!-- Ankle motor link  Small cylindrical motor attached to shank -->
+    <link name="${prefix}_ankle_motor">
+      <visual>
+        <origin xyz="0 0 -0.01" />
+        <geometry>
+          <cylinder length="${motor_length}" radius="${motor_radius}" />
+        </geometry>
+        <material name="grey" />
+      </visual>
+      <collision>
+        <origin xyz="0 0 -0.01" />
+        <geometry>
+          <cylinder length="${motor_length}" radius="${motor_radius}" />
+        </geometry>
+      </collision>
+      <inertial>
+        <mass value="${motor_mass}" />
+        <inertia ixx="0.00001" ixy="0.0" ixz="0.0" iyy="0.00001" iyz="0.0" izz="0.00001" />
+      </inertial>
+    </link>
+    <!-- Ankle motor mount  Fixed joint attaching ankle motor to shank -->
+    <joint name="${prefix}_ankle_motor_mount" type="fixed">
+      <parent link="${prefix}_shank" />
+      <child link="${prefix}_ankle_motor" />
+      <origin xyz="0 0 -${shank_length}" rpy="0 -0.3 0" /> <!-- Tilt forward for natural posture -->
+    </joint>
+    <!-- Ankle joint  Revolute joint for foot rotation -->
+    <joint name="${prefix}_ankle_joint" type="revolute">
+      <parent link="${prefix}_ankle_motor" />
+      <child link="${prefix}_foot" />
+      <origin xyz="0 0 0" />
+      <axis xyz="0 1 0" /> <!-- Rotation around y-axis -->
+      <limit effort="5" velocity="2.0" lower="-2.0" upper="2.0" />
+    </joint>
+    <!-- Foot link  Spherical foot for ground contact -->
+    <link name="${prefix}_foot">
+      <visual>
+        <geometry>
+          <sphere radius="${foot_radius}" />
+        </geometry>
+        <material name="black" />
+      </visual>
+      <collision>
+        <geometry>
+          <sphere radius="${foot_radius}" />
+        </geometry>
+      </collision>
+      <xacro:inertial_sphere mass="0.1" radius="${foot_radius}">
+        <origin xyz="0 0 0" rpy="0 0 0" />
+      </xacro:inertial_sphere>
+    </link>
+    <!-- Gazebo settings for foot friction -->
+    <gazebo reference="${prefix}_foot">
+      <mu1>0.8</mu1> <!-- Giảm ma sát ngang -->
+      <mu2>0.8</mu2> <!-- Giảm ma sát dọc -->
+    </gazebo>
+    <transmission name="${prefix}_hip_trans">
+      <type>transmission_interface/SimpleTransmission</type>
+      <joint name="${prefix}_hip_joint" />
+      <actuator name="${prefix}_hip_actuator" />
+    </transmission>
+    <transmission name="${prefix}_knee_trans">
+      <type>transmission_interface/SimpleTransmission</type>
+      <joint name="${prefix}_knee_joint" />
+      <actuator name="${prefix}_knee_actuator" />
+    </transmission>
+    <transmission name="${prefix}_ankle_trans">
+      <type>transmission_interface/SimpleTransmission</type>
+      <joint name="${prefix}_ankle_joint" />
+      <actuator name="${prefix}_ankle_actuator" />
+    </transmission>
+  </xacro:macro>
 </robot>
