Commit message: improve naming convention

File: src/robot.urdf (robot description, URDF)
Before this commit: robot my_robot, 27 links, 26 joints
Links:
- removed link left_front_ankle_motor_link
- removed link left_front_hip_motor_link
- removed link left_front_knee_motor_link
- removed link left_rear_ankle_motor_link
- removed link left_rear_hip_motor_link
- removed link left_rear_knee_motor_link
- removed link right_front_ankle_motor_link
- removed link right_front_hip_motor_link
- removed link right_front_knee_motor_link
- removed link right_rear_ankle_motor_link
- removed link right_rear_hip_motor_link
- removed link right_rear_knee_motor_link
- added link camera_link; visual box size=0.010 0.03 0.03
- added link camera_link_optical
- added link imu_link, mass 0.01
- added link left_front_ankle_motor, mass 0.03; collision cylinder length=0.02 radius=0.012; visual cylinder length=0.02 radius=0.012
- added link left_front_hip_motor, mass 0.03; collision cylinder length=0.02 radius=0.012; visual cylinder length=0.02 radius=0.012
- added link left_front_knee_motor, mass 0.03; collision cylinder length=0.02 radius=0.012; visual cylinder length=0.02 radius=0.012
- added link left_rear_ankle_motor, mass 0.03; collision cylinder length=0.02 radius=0.012; visual cylinder length=0.02 radius=0.012
- added link left_rear_hip_motor, mass 0.03; collision cylinder length=0.02 radius=0.012; visual cylinder length=0.02 radius=0.012
- added link left_rear_knee_motor, mass 0.03; collision cylinder length=0.02 radius=0.012; visual cylinder length=0.02 radius=0.012
- added link lidar_link, mass 0.1; collision cylinder length=0.04 radius=0.05; visual cylinder length=0.04 radius=0.05
- added link right_front_ankle_motor, mass 0.03; collision cylinder length=0.02 radius=0.012; visual cylinder length=0.02 radius=0.012
- added link right_front_hip_motor, mass 0.03; collision cylinder length=0.02 radius=0.012; visual cylinder length=0.02 radius=0.012
- added link right_front_knee_motor, mass 0.03; collision cylinder length=0.02 radius=0.012; visual cylinder length=0.02 radius=0.012
- added link right_rear_ankle_motor, mass 0.03; collision cylinder length=0.02 radius=0.012; visual cylinder length=0.02 radius=0.012
- added link right_rear_hip_motor, mass 0.03; collision cylinder length=0.02 radius=0.012; visual cylinder length=0.02 radius=0.012
- added link right_rear_knee_motor, mass 0.03; collision cylinder length=0.02 radius=0.012; visual cylinder length=0.02 radius=0.012
- link left_front_shank: mass 0.2 -> 0.15; geometry collision box size=0.02 0.02 0.18; visual box size=0.02 0.02 0.18
- link left_front_thigh: mass 0.2 -> 0.15; geometry collision box size=0.03 0.03 0.18; visual box size=0.03 0.03 0.18
- link left_rear_shank: mass 0.2 -> 0.15; geometry collision box size=0.02 0.02 0.18; visual box size=0.02 0.02 0.18
- link left_rear_thigh: mass 0.2 -> 0.15; geometry collision box size=0.03 0.03 0.18; visual box size=0.03 0.03 0.18
- link right_front_shank: mass 0.2 -> 0.15; geometry collision box size=0.02 0.02 0.18; visual box size=0.02 0.02 0.18
- link right_front_thigh: mass 0.2 -> 0.15; geometry collision box size=0.03 0.03 0.18; visual box size=0.03 0.03 0.18
- link right_rear_shank: mass 0.2 -> 0.15; geometry collision box size=0.02 0.02 0.18; visual box size=0.02 0.02 0.18
- link right_rear_thigh: mass 0.2 -> 0.15; geometry collision box size=0.03 0.03 0.18; visual box size=0.03 0.03 0.18
Joints:
- removed joint left_front_ankle_motor_fixed
- removed joint left_front_hip_motor_fixed
- removed joint left_front_knee_motor_fixed
- removed joint left_front_lower_leg_joint
- removed joint left_front_upper_leg_joint
- removed joint left_rear_ankle_motor_fixed
- removed joint left_rear_hip_motor_fixed
- removed joint left_rear_knee_motor_fixed
- removed joint left_rear_lower_leg_joint
- removed joint left_rear_upper_leg_joint
- removed joint right_front_ankle_motor_fixed
- removed joint right_front_hip_motor_fixed
- removed joint right_front_knee_motor_fixed
- removed joint right_front_lower_leg_joint
- removed joint right_front_upper_leg_joint
- removed joint right_rear_ankle_motor_fixed
- removed joint right_rear_hip_motor_fixed
- removed joint right_rear_knee_motor_fixed
- removed joint right_rear_lower_leg_joint
- removed joint right_rear_upper_leg_joint
- added joint camera_joint: type fixed, parent chassis, child camera_link, origin xyz=0.25 0 0.08 rpy=0 0 0
- added joint camera_optical_joint: type fixed, parent camera_link, child camera_link_optical, origin xyz=0.25 0 0 rpy=-1.5707963267948966 0 -1.5707963267948966
- added joint imu_joint: type fixed, parent base_link, child imu_link, origin xyz=0 0 0.1
- added joint laser_joint: type fixed, parent base_link, child lidar_link, origin xyz=0.1 0 0.175 rpy=0 0 0
- added joint left_front_ankle_joint: type revolute, parent left_front_ankle_motor, child left_front_foot, origin xyz=0 0 0, axis 0 1 0, limit lower=-2.0 upper=2.0 effort=5 velocity=2.0
- added joint left_front_ankle_motor_mount: type fixed, parent left_front_shank, child left_front_ankle_motor, origin xyz=0 0 -0.18 rpy=0 -0.3 0
- added joint left_front_hip_motor_mount: type fixed, parent chassis, child left_front_hip_motor, origin xyz=0.15 0.1 -0.005
- added joint left_front_knee_joint: type revolute, parent left_front_knee_motor, child left_front_shank, origin xyz=0 0 0, axis 0 1 0, limit lower=-2.5 upper=0 effort=5 velocity=2.0
- added joint left_front_knee_motor_mount: type fixed, parent left_front_thigh, child left_front_knee_motor, origin xyz=0 0 -0.18 rpy=0 -0.3 0
- added joint left_rear_ankle_joint: type revolute, parent left_rear_ankle_motor, child left_rear_foot, origin xyz=0 0 0, axis 0 1 0, limit lower=-2.0 upper=2.0 effort=5 velocity=2.0
- added joint left_rear_ankle_motor_mount: type fixed, parent left_rear_shank, child left_rear_ankle_motor, origin xyz=0 0 -0.18 rpy=0 -0.3 0
- added joint left_rear_hip_motor_mount: type fixed, parent chassis, child left_rear_hip_motor, origin xyz=-0.15 0.1 -0.005
- added joint left_rear_knee_joint: type revolute, parent left_rear_knee_motor, child left_rear_shank, origin xyz=0 0 0, axis 0 1 0, limit lower=-2.5 upper=0 effort=5 velocity=2.0
- added joint left_rear_knee_motor_mount: type fixed, parent left_rear_thigh, child left_rear_knee_motor, origin xyz=0 0 -0.18 rpy=0 -0.3 0
- added joint right_front_ankle_joint: type revolute, parent right_front_ankle_motor, child right_front_foot, origin xyz=0 0 0, axis 0 1 0, limit lower=-2.0 upper=2.0 effort=5 velocity=2.0
- added joint right_front_ankle_motor_mount: type fixed, parent right_front_shank, child right_front_ankle_motor, origin xyz=0 0 -0.18 rpy=0 -0.3 0
- added joint right_front_hip_motor_mount: type fixed, parent chassis, child right_front_hip_motor, origin xyz=0.15 -0.1 -0.005
- added joint right_front_knee_joint: type revolute, parent right_front_knee_motor, child right_front_shank, origin xyz=0 0 0, axis 0 1 0, limit lower=-2.5 upper=0 effort=5 velocity=2.0
- added joint right_front_knee_motor_mount: type fixed, parent right_front_thigh, child right_front_knee_motor, origin xyz=0 0 -0.18 rpy=0 -0.3 0
- added joint right_rear_ankle_joint: type revolute, parent right_rear_ankle_motor, child right_rear_foot, origin xyz=0 0 0, axis 0 1 0, limit lower=-2.0 upper=2.0 effort=5 velocity=2.0
- added joint right_rear_ankle_motor_mount: type fixed, parent right_rear_shank, child right_rear_ankle_motor, origin xyz=0 0 -0.18 rpy=0 -0.3 0
- added joint right_rear_hip_motor_mount: type fixed, parent chassis, child right_rear_hip_motor, origin xyz=-0.15 -0.1 -0.005
- added joint right_rear_knee_joint: type revolute, parent right_rear_knee_motor, child right_rear_shank, origin xyz=0 0 0, axis 0 1 0, limit lower=-2.5 upper=0 effort=5 velocity=2.0
- added joint right_rear_knee_motor_mount: type fixed, parent right_rear_thigh, child right_rear_knee_motor, origin xyz=0 0 -0.18 rpy=0 -0.3 0
- joint left_front_hip_joint: limit lower=-1.57 upper=1.57 effort=5 velocity=2.0 -> lower=-1.57 upper=0 effort=5 velocity=2.0; parent left_front_hip_motor_link -> left_front_hip_motor
- joint left_rear_hip_joint: limit lower=-1.57 upper=1.57 effort=5 velocity=2.0 -> lower=-1.57 upper=0 effort=5 velocity=2.0; parent left_rear_hip_motor_link -> left_rear_hip_motor
- joint right_front_hip_joint: limit lower=-1.57 upper=1.57 effort=5 velocity=2.0 -> lower=-1.57 upper=0 effort=5 velocity=2.0; parent right_front_hip_motor_link -> right_front_hip_motor
- joint right_rear_hip_joint: limit lower=-1.57 upper=1.57 effort=5 velocity=2.0 -> lower=-1.57 upper=0 effort=5 velocity=2.0; parent right_rear_hip_motor_link -> right_rear_hip_motor

Commit message: update st

File: src/first_robot/description/gz_control.xacro (robot description, xacro)
@@ -2,4 +2,16 @@
   <xacro:arg name="use_mock_hardware" default="true" />
   <xacro:arg name="use_gazebo" default="true" />
+  <gazebo>
+    <plugin filename="gz-sim-pose-publisher-system" name="gz::sim::systems::PosePublisher">
+      <publish_link_pose>true</publish_link_pose>
+      <publish_sensor_pose>true</publish_sensor_pose>
+      <publish_collision_pose>false</publish_collision_pose>
+      <publish_visual_pose>false</publish_visual_pose>
+      <publish_nested_model_pose>false</publish_nested_model_pose>
+      <use_pose_vector_msg>true</use_pose_vector_msg>
+      <static_publisher>true</static_publisher>
+      <static_update_frequency>100</static_update_frequency>
+    </plugin>
+  </gazebo>
   <ros2_control name="FirstRobot" type="system">
     <hardware>
@@ -10,5 +22,4 @@
       <joint name="${joint_name}">
         <command_interface name="effort" />
-        <command_interface name="position" />
         <state_interface name="position" />
         <state_interface name="velocity" />
@@ -35,5 +46,108 @@
     <plugin filename="gz_ros2_control-system" name="gz_ros2_control::GazeboSimROS2ControlPlugin">
       <parameters>$(find first_robot)/config/ros_control.yaml</parameters>
+       <robot_param_node>robot_state_publisher</robot_param_node>
     </plugin>
   </gazebo>
+   <gazebo reference="trunk">
+    <mu1>0.2</mu1>
+    <mu2>0.2</mu2>
+    <kp>10000.0</kp>
+    <kd>1.0</kd>
+  </gazebo>
+  <!-- FL leg -->
+  <gazebo reference="front_left_hip_link">
+    <mu1>0.2</mu1>
+    <mu2>0.2</mu2>
+  </gazebo>
+  <gazebo reference="front_left_knee_link">
+    <mu1>0.2</mu1>
+    <mu2>0.2</mu2>
+    <self_collide>1</self_collide>
+    <kp>10000.0</kp>
+    <kd>1.0</kd>
+  </gazebo>
+  <gazebo reference="front_left_ankle_link">
+    <mu1>0.2</mu1>
+    <mu2>0.2</mu2>
+    <self_collide>1</self_collide>
+  </gazebo>
+  <gazebo reference="front_left_foot_link">
+    <mu1>0.6</mu1>
+    <mu2>0.6</mu2>
+    <self_collide>1</self_collide>
+    <kp>10000.0</kp>
+    <kd>1.0</kd>
+  </gazebo>
+  <!-- FR leg -->
+  <gazebo reference="front_right_hip_link">
+    <mu1>0.2</mu1>
+    <mu2>0.2</mu2>
+  </gazebo>
+  <gazebo reference="front_right_knee_link">
+    <mu1>0.2</mu1>
+    <mu2>0.2</mu2>
+    <self_collide>1</self_collide>
+    <kp>10000.0</kp>
+    <kd>1.0</kd>
+  </gazebo>
+  <gazebo reference="front_right_ankle_link">
+    <mu1>0.2</mu1>
+    <mu2>0.2</mu2>
+    <self_collide>1</self_collide>
+  </gazebo>
+  <gazebo reference="front_right_foot_link">
+    <mu1>0.6</mu1>
+    <mu2>0.6</mu2>
+    <self_collide>1</self_collide>
+    <kp>10000.0</kp>
+    <kd>1.0</kd>
+  </gazebo>
+  <!-- RL leg -->
+  <gazebo reference="rear_left_hip_link">
+    <mu1>0.2</mu1>
+    <mu2>0.2</mu2>
+  </gazebo>
+  <gazebo reference="rear_left_knee_link">
+    <mu1>0.2</mu1>
+    <mu2>0.2</mu2>
+    <self_collide>1</self_collide>
+    <kp>10000.0</kp>
+    <kd>1.0</kd>
+  </gazebo>
+  <gazebo reference="rear_left_ankle_link">
+    <mu1>0.2</mu1>
+    <mu2>0.2</mu2>
+    <self_collide>1</self_collide>
+  </gazebo>
+  <gazebo reference="rear_left_foot_link">
+    <mu1>0.6</mu1>
+    <mu2>0.6</mu2>
+    <self_collide>1</self_collide>
+    <kp>10000.0</kp>
+    <kd>1.0</kd>
+  </gazebo>
+  <!-- RR leg -->
+  <gazebo reference="rear_right_hip_link">
+    <mu1>0.2</mu1>
+    <mu2>0.2</mu2>
+  </gazebo>
+  <gazebo reference="rear_right_knee_link">
+    <mu1>0.2</mu1>
+    <mu2>0.2</mu2>
+    <self_collide>1</self_collide>
+    <kp>10000.0</kp>
+    <kd>1.0</kd>
+  </gazebo>
+  <gazebo reference="rear_right_ankle_link">
+    <mu1>0.2</mu1>
+    <mu2>0.2</mu2>
+    <self_collide>1</self_collide>
+  </gazebo>
+  <gazebo reference="rear_right_foot_link">
+    <mu1>0.6</mu1>
+    <mu2>0.6</mu2>
+    <self_collide>1</self_collide>
+    <kp>10000.0</kp>
+    <kd>1.0</kd>
+  </gazebo>
 </robot>

File: src/first_robot/description/leg_block_v3.xacro (robot description, xacro)
@@ -145,5 +145,5 @@
     <!-- ankle Joint  Cẳng chân  quay về trước 45  -->
     <joint name="${prefix}_ankle_joint" initial_position="-1.0" type="revolute">
-      <origin rpy="0 -0.90 0" xyz="0 0 ${-ankle_length}" />
+      <origin rpy="0 -0.6 0" xyz="0 0 ${-ankle_length}" />
       <parent link="${prefix}_knee_link" />
       <child link="${prefix}_ankle_link" />
