Commit message: update sthing

File: src/first_robot/description/constants.xacro (robot description, xacro)
@@ -57,5 +57,5 @@
     <!-- dynamics inertial value -->
     <!-- trunk -->
-    <xacro:property name="trunk_mass" value="4.921"/>
+    <xacro:property name="trunk_mass" value="4.0"/>
     <xacro:property name="trunk_com_x" value="0.021112"/>
     <xacro:property name="trunk_com_y" value="0.00"/>
@@ -118,5 +118,5 @@
     <!-- dynamics inertial value -->
     <!-- trunk -->
-    <xacro:property name="trunk_mass" value="4.921"/>
+    <xacro:property name="trunk_mass" value="2.2"/>
     <xacro:property name="trunk_com_x" value="0.021112"/>
     <xacro:property name="trunk_com_y" value="0.00"/>

File: src/first_robot/description/leg_block_v3.xacro (robot description, xacro)
@@ -13,59 +13,62 @@
         <!-- Chân phải và phía trước -->
         <xacro:if value="${(side == 1) and (pos == 1)}">
-          <origin rpy="${PI/2.0} 2.0 0" xyz="0 0 0"/>
+          <origin rpy="${PI} 0 0" xyz="0 0 0" />
         </xacro:if>
         <!-- Chân trái và phía sau -->
         <xacro:if value="${(side == 1) and (pos == -1)}">
-          <origin rpy="${PI/2.0} 2.0 0" xyz="0 0 0"/>
+          <origin rpy="${PI} ${PI} 0" xyz="0 0 0" />
         </xacro:if>
         <!-- Chân trái và phía trước -->
         <xacro:if value="${(side == -1) and (pos == 1)}">
-          <origin rpy="${PI/2.0} 2.0 0" xyz="0 0 0"/>
+          <origin rpy="0 0 0" xyz="0 0 0" />
         </xacro:if>
         <!-- Chân phải và phía sau -->
         <xacro:if value="${(side == -1) and (pos == -1)}">
-          <origin rpy="${PI/2.0} 2.0 0" xyz="0 0 0"/>
+          <origin rpy="0 ${PI} 0" xyz="0 0 0" />
         </xacro:if>
         <geometry>
           <!-- <cylinder length="${hip_length}" radius="${hip_radius}"/> -->
-          <mesh filename="file://$(find first_robot)/meshes/hip.dae" scale="1 1 1"/>
+          <mesh filename="file://$(find first_robot)/meshes/hip.dae" scale="1 1 1" />
           <!-- dài 2cm  cố định thân trên và các chân -->
         </geometry>
-        <material name="blue"/>
+        <material name="blue" />
       </visual>
       <collision name="${prefix}_hip_collision">
-        <origin rpy="${PI/2.0} 2.0 0" xyz="0 ${hip_offset*side} 0"/>
-        <geometry>
-          <cylinder length="${hip_length + 0.01}" radius="${hip_radius + 0.01}"/>
-        </geometry>
-      </collision>
-      <inertial>
-        <origin rpy="0 0 0" xyz="${hip_com_x*pos} ${hip_com_y*side} ${hip_com_z}"/>
-        <mass value="${hip_mass}"/>
-        <inertia ixx="${hip_ixx}" ixy="${hip_ixy*side*pos}" ixz="${hip_ixz*pos}" iyy="${hip_iyy}" iyz="${hip_iyz*side}" izz="${hip_izz}"/>
-      </inertial>
-    </link>
-    <joint name="${prefix}_hip_joint" description="Hip joint side ${side} and pos ${pos}" type="revolute">
-      <parent link="trunk"/>
-      <child link="${prefix}_hip_link"/>
+        <origin rpy="0 0 0" xyz="0 ${hip_offset*side} 0" />
+        <geometry>
+          <cylinder length="${hip_length + 0.01}" radius="${hip_radius + 0.01}" />
+        </geometry>
+      </collision>
+      <inertial>
+        <origin rpy="0 0 0" xyz="${hip_com_x*pos} ${hip_com_y*side} ${hip_com_z}" />
+        <mass value="${hip_mass}" />
+        <inertia ixx="${hip_ixx}" ixy="${hip_ixy*side*pos}" ixz="${hip_ixz*pos}" iyy="${hip_iyy}"
+          iyz="${hip_iyz*side}" izz="${hip_izz}" />
+      </inertial>
+    </link>
+    <joint name="${prefix}_hip_joint" description="Hip joint side ${side} and pos ${pos}"
+      type="revolute">
+      <parent link="trunk" />
+      <child link="${prefix}_hip_link" />
       <!-- Chân trái và phía trước -->
       <xacro:if value="${(side == 1) and (pos == 1)}">
-        <origin rpy="0 0 0" xyz="${leg_offset_x} ${-leg_offset_y} 0"/>
+        <origin rpy="0 0 0" xyz="${leg_offset_x} ${-leg_offset_y} 0" />
       </xacro:if>
       <!-- Chân trái và phía sau -->
       <xacro:if value="${(side == 1) and (pos == -1)}">
-        <origin rpy="0 0 0" xyz="${-leg_offset_x} ${-leg_offset_y} 0"/>
+        <origin rpy="0 0 0" xyz="${-leg_offset_x} ${-leg_offset_y} 0" />
       </xacro:if>
       <!-- Chân phải và phía trước -->
       <xacro:if value="${(side == -1) and (pos == 1)}">
-        <origin rpy="0 0 0" xyz="${leg_offset_x} ${leg_offset_y} 0"/>
+        <origin rpy="0 0 0" xyz="${leg_offset_x} ${leg_offset_y} 0" />
       </xacro:if>
       <!-- Chân phải và phía sau -->
       <xacro:if value="${(side == -1) and (pos == -1)}">
-        <origin rpy="0 0 0" xyz="${-leg_offset_x} ${leg_offset_y} 0"/>
-      </xacro:if>
-      <axis xyz="1 0 0"/>
-      <dynamics damping="${damping}" friction="${friction}"/>
-      <limit effort="${hip_torque_max}" velocity="${hip_velocity_max}" lower="${hip_position_min}" upper="${hip_position_max}"/>
+        <origin rpy="0 0 0" xyz="${-leg_offset_x} ${leg_offset_y} 0" />
+      </xacro:if>
+      <axis xyz="1 0 0" />
+      <dynamics damping="${damping}" friction="${friction}" />
+      <limit effort="${hip_torque_max}" velocity="${hip_velocity_max}" lower="${hip_position_min}"
+        upper="${hip_position_max}" />
       <!-- Vị trí gắn khớp háng vào body-->
     </joint>
@@ -74,40 +77,43 @@
     <link name="${prefix}_knee_link">
       <visual name="${prefix}_knee_visual">
-        <origin rpy="0 0 0" xyz="0 0 0"/>
+        <origin rpy="0 0 0" xyz="0 0 0" />
         <geometry>
           <!-- <box size="${knee_length} ${knee_width} ${knee_height}"/> -->
           <xacro:if value="${(side == 1) }">
-            <mesh filename="file://$(find first_robot)/meshes/knee_mirror.dae" scale="1 1 1"/>
+            <mesh filename="file://$(find first_robot)/meshes/knee_mirror.dae" scale="1 1 1" />
             <!-- <origin rpy="${PI/2.0} 2.0 0" xyz="0 0 0"/> -->
           </xacro:if>
           <xacro:if value="${(side == -1) }">
-            <mesh filename="file://$(find first_robot)/meshes/knee.dae" scale="1 1 1"/>
+            <mesh filename="file://$(find first_robot)/meshes/knee.dae" scale="1 1 1" />
             <!-- <origin rpy="${PI/2.0} 2.0 0" xyz="0 0 0"/> -->
           </xacro:if>
         </geometry>
-        <material name="green"/>
+        <material name="green" />
       </visual>
       <collision name="${prefix}_knee_collision">
-        <origin rpy="0 0 0" xyz="0 0 0"/>
-        <geometry>
-          <box size="${knee_length + 0.01} ${knee_width + 0.01} ${knee_height + 0.01}"/>
-        </geometry>
-      </collision>
-      <inertial>
-        <origin rpy="0 0 0" xyz="${knee_com_x} ${knee_com_y*-side} ${knee_com_z}"/>
-        <mass value="${knee_mass}"/>
-        <inertia ixx="${knee_ixx}" ixy="${knee_ixy*-side}" ixz="${knee_ixz}" iyy="${knee_iyy}" iyz="${knee_iyz*-side}" izz="${knee_izz}"/>
+        <origin rpy="0 0 0" xyz="0 0 0" />
+        <geometry>
+          <box size="${knee_length + 0.01} ${knee_width + 0.01} ${knee_height + 0.01}" />
+        </geometry>
+      </collision>
+      <inertial>
+        <origin rpy="0 0 0" xyz="${knee_com_x} ${knee_com_y*-side} ${knee_com_z}" />
+        <mass value="${knee_mass}" />
+        <inertia ixx="${knee_ixx}" ixy="${knee_ixy*-side}" ixz="${knee_ixz}" iyy="${knee_iyy}"
+          iyz="${knee_iyz*-side}" izz="${knee_izz}" />
       </inertial>
     </link>
     <!-- knee Joint  Đùi  quay về sau  -->
-    <joint name="${prefix}_knee_joint" description="Knee joint side ${side} and pos ${pos}" type="revolute">
-      <origin rpy="0 0.45 0" xyz="0 ${knee_offset*-side} 0"/>
-      <parent link="${prefix}_hip_link"/>
+    <joint name="${prefix}_knee_joint" description="Knee joint side ${side} and pos ${pos}"
+      type="revolute">
+      <origin rpy="0 0.45 0" xyz="0 ${knee_offset*-side} 0" />
+      <parent link="${prefix}_hip_link" />
       <!-- Gắn vào motor háng mô phỏng -->
-      <child link="${prefix}_knee_link"/>
-      <axis xyz="0 1 0"/>
-      <dynamics damping="${damping}" friction="${friction}"/>
-      <limit lower="-1.57" upper="1.57" effort="30" velocity="7.0"/>
-      <limit effort="${knee_torque_max}" velocity="${knee_velocity_max}" lower="${knee_position_min}" upper="${knee_position_max}"/>
+      <child link="${prefix}_knee_link" />
+      <axis xyz="0 1 0" />
+      <dynamics damping="${damping}" friction="${friction}" />
+      <limit lower="-1.57" upper="1.57" effort="30" velocity="7.0" />
+      <limit effort="${knee_torque_max}" velocity="${knee_velocity_max}"
+        lower="${knee_position_min}" upper="${knee_position_max}" />
     </joint>
     <!-- *** Kết thúc phần đùi chân *** -->
@@ -116,32 +122,34 @@
     <link name="${prefix}_ankle_link">
       <visual name="${prefix}_ankle_visual">
-        <origin rpy="0 0 0" xyz="0 0 0"/>
+        <origin rpy="0 0 0" xyz="0 0 0" />
         <geometry>
           <!-- <box size="${ankle_length} ${ankle_width} ${ankle_height}"/> -->
-          <mesh filename="file://$(find first_robot)/meshes/ankle.dae" scale="1 1 1"/>
+          <mesh filename="file://$(find first_robot)/meshes/ankle.dae" scale="1 1 1" />
         </geometry>
         <!-- Màu tím -->
-        <material name="purple"/>
+        <material name="purple" />
       </visual>
       <collision name="${prefix}_ankle_collision">
-        <origin rpy="0 0 0" xyz="0 0 0"/>
-        <geometry>
-          <box size="${ankle_length + 0.01} ${ankle_width + 0.01} ${ankle_height + 0.01}"/>
-        </geometry>
-      </collision>
-      <inertial>
-        <origin rpy="0 0 0" xyz="${ankle_com_x} ${ankle_com_y} ${ankle_com_z}"/>
-        <mass value="${ankle_mass}"/>
-        <inertia ixx="${ankle_ixx}" ixy="${ankle_ixy}" ixz="${ankle_ixz}" iyy="${ankle_iyy}" iyz="${ankle_iyz}" izz="${ankle_izz}"/>
+        <origin rpy="0 0 0" xyz="0 0 0" />
+        <geometry>
+          <box size="${ankle_length + 0.01} ${ankle_width + 0.01} ${ankle_height + 0.01}" />
+        </geometry>
+      </collision>
+      <inertial>
+        <origin rpy="0 0 0" xyz="${ankle_com_x} ${ankle_com_y} ${ankle_com_z}" />
+        <mass value="${ankle_mass}" />
+        <inertia ixx="${ankle_ixx}" ixy="${ankle_ixy}" ixz="${ankle_ixz}" iyy="${ankle_iyy}"
+          iyz="${ankle_iyz}" izz="${ankle_izz}" />
       </inertial>
     </link>
     <!-- ankle Joint  Cẳng chân  quay về trước 45  -->
     <joint name="${prefix}_ankle_joint" type="revolute">
-      <origin rpy="0 -0.45 0" xyz="0 0 ${-ankle_length}"/>
-      <parent link="${prefix}_knee_link"/>
-      <child link="${prefix}_ankle_link"/>
-      <axis xyz="0 1 0"/>
-      <dynamics damping="${damping}" friction="${friction}"/>
-      <limit effort="${ankle_torque_max}" velocity="${ankle_velocity_max}" lower="${ankle_position_min}" upper="${ankle_position_max}"/>
+      <origin rpy="0 -0.8 0" xyz="0 0 ${-ankle_length}" />
+      <parent link="${prefix}_knee_link" />
+      <child link="${prefix}_ankle_link" />
+      <axis xyz="0 1 0" />
+      <dynamics damping="${damping}" friction="${friction}" />
+      <limit effort="${ankle_torque_max}" velocity="${ankle_velocity_max}"
+        lower="${ankle_position_min}" upper="${ankle_position_max}" />
     </joint>
     <!-- *** Kết thúc phần cẳng chân *** -->
@@ -150,32 +158,34 @@
     <link name="${prefix}_foot_link">
       <visual name="${prefix}_foot_visual">
-        <origin rpy="0 0 0" xyz="0 0 0"/>
-        <geometry>
-          <mesh filename="file://$(find first_robot)/meshes/foot.dae" scale="1 1 1"/>
+        <origin rpy="0 0 0" xyz="0 0 0" />
+        <geometry>
+          <mesh filename="file://$(find first_robot)/meshes/foot.dae" scale="1 1 1" />
           <!-- <sphere radius="${foot_radius}"/> -->
         </geometry>
-        <material name="black"/>
+        <material name="black" />
       </visual>
       <collision name="${prefix}_foot_collision">
-        <origin rpy="0 0 0" xyz="0 0 0"/>
-        <geometry>
-          <sphere radius="${foot_radius}"/>
-        </geometry>
-      </collision>
-      <inertial>
-        <mass value="${foot_mass}"/>
-        <inertia ixx="${(2*foot_mass)/5.0*(foot_radius*foot_radius)}" ixy="0.0" ixz="0.0" iyy="${(2*foot_mass)/5.0*(foot_radius*foot_radius)}" iyz="0.0" izz="${(2*foot_mass)/5.0*(foot_radius*foot_radius)}"/>
+        <origin rpy="0 0 0" xyz="0 0 0" />
+        <geometry>
+          <sphere radius="${foot_radius}" />
+        </geometry>
+      </collision>
+      <inertial>
+        <mass value="${foot_mass}" />
+        <inertia ixx="${(2*foot_mass)/5.0*(foot_radius*foot_radius)}" ixy="0.0" ixz="0.0"
+          iyy="${(2*foot_mass)/5.0*(foot_radius*foot_radius)}" iyz="0.0"
+          izz="${(2*foot_mass)/5.0*(foot_radius*foot_radius)}" />
       </inertial>
     </link>
     <!-- Foot Joint -->
     <joint name="${prefix}_foot_joint" type="fixed">
-      <origin rpy="0 0 0" xyz="0 0 -0.213"/>
-      <parent link="${prefix}_ankle_link"/>
-      <child link="${prefix}_foot_link"/>
+      <origin rpy="0 0 0" xyz="0 0 -0.213" />
+      <parent link="${prefix}_ankle_link" />
+      <child link="${prefix}_foot_link" />
     </joint>
     <!-- Transmission cho các joint -->
     <transmission name="${prefix}_knee_trans">
       <type>transmission_interface/SimpleTransmission</type>
-      <joint name="${prefix}_knee_joint"/>
+      <joint name="${prefix}_knee_joint" />
       <actuator name="${prefix}_knee_motor">
         <mechanical_reduction>1</mechanical_reduction>
@@ -184,5 +194,5 @@
     <transmission name="${prefix}_ankle_trans">
       <type>transmission_interface/SimpleTransmission</type>
-      <joint name="${prefix}_ankle_joint"/>
+      <joint name="${prefix}_ankle_joint" />
       <actuator name="${prefix}_ankle_motor">
         <mechanical_reduction>1</mechanical_reduction>

File: src/first_robot/description/robot_core.xacro (robot description, xacro)
@@ -4,44 +4,50 @@
   <link name="base_link">
     <visual name="base_link_visual">
-      <origin rpy="0 0 0" xyz="0 0 0"/>
+      <origin rpy="0 0 0" xyz="0 0 0" />
       <geometry>
-        <box size="0.001 0.001 0.001"/>
+        <box size="0.001 0.001 0.001" />
       </geometry>
       <material name="white" />
     </visual>
+    <inertial>
+      <origin xyz="0 0 0" />
+      <mass value="0.1" />
+      <inertia ixx="0.001" iyy="0.001" izz="0.001" ixy="0" ixz="0" iyz="0" />
+    </inertial>
   </link>
   <joint name="floating_base" type="fixed">
-    <parent link="base_link"/>
-    <child link="trunk"/>
-    <origin xyz="0 0 0" rpy="0 0 0"/>
+    <parent link="base_link" />
+    <child link="trunk" />
+    <origin xyz="0 0 0" rpy="0 0 0" />
   </joint>
   <!-- Trunk  Thân robot -->
   <link name="trunk">
     <visual name="trunk_visual">
-      <origin rpy="0 0 0" xyz="0 0 0"/>
+      <origin rpy="0 0 0" xyz="0 0 0" />
       <geometry>
-          <!-- <box size="${trunk_length} ${trunk_width} ${trunk_height}"/> -->
-          <mesh filename="file://$(find first_robot)/meshes/trunk.dae" scale="1 1 1"/>
+        <!-- <box size="${trunk_length} ${trunk_width} ${trunk_height}"/> -->
+        <mesh filename="file://$(find first_robot)/meshes/trunk.dae" scale="1 1 1" />
       </geometry>
-      <material name="silver"/>
+      <material name="silver" />
     </visual>
     <collision name="trunk_collision">
-      <origin rpy="0 0 0" xyz="0 0 0"/>
+      <origin rpy="0 0 0" xyz="0 0 0" />
       <geometry>
-        <box size="${trunk_length} ${trunk_width} ${trunk_height}"/>
+        <box size="${trunk_length} ${trunk_width} ${trunk_height}" />
       </geometry>
     </collision>
     <inertial>
-      <origin rpy="0 0 0" xyz="${trunk_com_x} ${trunk_com_y} ${trunk_com_z}"/>
-      <mass value="${trunk_mass}"/>
-      <inertia ixx="${trunk_ixx}" ixy="${trunk_ixy}" ixz="${trunk_ixz}" iyy="${trunk_iyy}" iyz="${trunk_iyz}" izz="${trunk_izz}"/>
+      <origin rpy="0 0 0" xyz="${trunk_com_x} ${trunk_com_y} ${trunk_com_z}" />
+      <mass value="${trunk_mass}" />
+      <inertia ixx="${trunk_ixx}" ixy="${trunk_ixy}" ixz="${trunk_ixz}" iyy="${trunk_iyy}"
+        iyz="${trunk_iyz}" izz="${trunk_izz}" />
     </inertial>
-    </link>
-    <!-- IMPORT LEG PATTERN -->
-    <xacro:include filename="$(find first_robot)/description/leg_block_v3.xacro"/>
-    <!-- Gọi macro leg cho từng chân -->
-    <xacro:leg prefix="front_left" side="-1" use_dae="False" pos="1" />
-    <xacro:leg prefix="front_right" side="1" use_dae="False" pos="1"/>
-    <xacro:leg prefix="rear_left" side="-1" use_dae="False" pos="-1" />
-    <xacro:leg prefix="rear_right" side="1" use_dae="False" pos="-1" />
-  </robot>
+  </link>
+  <!-- IMPORT LEG PATTERN -->
+  <xacro:include filename="$(find first_robot)/description/leg_block_v3.xacro" />
+  <!-- Gọi macro leg cho từng chân -->
+  <xacro:leg prefix="front_left" side="-1" use_dae="False" pos="1" />
+  <xacro:leg prefix="front_right" side="1" use_dae="False" pos="1" />
+  <xacro:leg prefix="rear_left" side="-1" use_dae="False" pos="-1" />
+  <xacro:leg prefix="rear_right" side="1" use_dae="False" pos="-1" />
+</robot>

File: src/robot.urdf (robot description, URDF)
Before this commit: robot my_robot, 21 links, 20 joints
Links:
- link base_link: mass None -> 0.1
- link front_left_ankle_link: geometry collision box size=0.223 0.026000000000000002 0.026000000000000002; visual mesh filename=file:///home/phieu/ros2-learning/src/install/first_robot/sh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 scale=1 1 1
- link front_left_foot_link: geometry collision sphere radius=0.02; visual mesh filename=file:///home/phieu/ros2-learning/src/install/first_robot/sh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 scale=1 1 1
- link front_left_hip_link: geometry collision cylinder length=0.05 radius=0.056; visual mesh filename=file:///home/phieu/ros2-learning/src/install/first_robot/sh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 scale=1 1 1
- link front_left_knee_link: mass 1.152 -> 0.135862; geometry collision box size=0.223 0.0345 0.044000000000000004; visual mesh filename=file:///home/phieu/ros2-learning/src/install/first_robot/sh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 scale=1 1 1
- link front_right_ankle_link: geometry collision box size=0.223 0.026000000000000002 0.026000000000000002; visual mesh filename=file:///home/phieu/ros2-learning/src/install/first_robot/sh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 scale=1 1 1
- link front_right_foot_link: geometry collision sphere radius=0.02; visual mesh filename=file:///home/phieu/ros2-learning/src/install/first_robot/sh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 scale=1 1 1
- link front_right_hip_link: geometry collision cylinder length=0.05 radius=0.056; visual mesh filename=file:///home/phieu/ros2-learning/src/install/first_robot/sh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 scale=1 1 1
- link front_right_knee_link: mass 1.152 -> 0.135862; geometry collision box size=0.223 0.0345 0.044000000000000004; visual mesh filename=file:///home/phieu/ros2-learning/src/install/first_robot/sh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 scale=1 1 1
- link rear_left_ankle_link: geometry collision box size=0.223 0.026000000000000002 0.026000000000000002; visual mesh filename=file:///home/phieu/ros2-learning/src/install/first_robot/sh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 scale=1 1 1
- link rear_left_foot_link: geometry collision sphere radius=0.02; visual mesh filename=file:///home/phieu/ros2-learning/src/install/first_robot/sh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 scale=1 1 1
- link rear_left_hip_link: geometry collision cylinder length=0.05 radius=0.056; visual mesh filename=file:///home/phieu/ros2-learning/src/install/first_robot/sh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 scale=1 1 1
- link rear_left_knee_link: mass 1.152 -> 0.135862; geometry collision box size=0.223 0.0345 0.044000000000000004; visual mesh filename=file:///home/phieu/ros2-learning/src/install/first_robot/sh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 scale=1 1 1
- link rear_right_ankle_link: geometry collision box size=0.223 0.026000000000000002 0.026000000000000002; visual mesh filename=file:///home/phieu/ros2-learning/src/install/first_robot/sh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 scale=1 1 1
- link rear_right_foot_link: geometry collision sphere radius=0.02; visual mesh filename=file:///home/phieu/ros2-learning/src/install/first_robot/sh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 scale=1 1 1
- link rear_right_hip_link: geometry collision cylinder length=0.05 radius=0.056; visual mesh filename=file:///home/phieu/ros2-learning/src/install/first_robot/sh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 scale=1 1 1
- link rear_right_knee_link: mass 1.152 -> 0.135862; geometry collision box size=0.223 0.0345 0.044000000000000004; visual mesh filename=file:///home/phieu/ros2-learning/src/install/first_robot/sh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 scale=1 1 1
- link trunk: mass 6.921 -> 4.921; geometry collision box size=0.3762 0.0935 0.114; visual mesh filename=file:///home/phieu/ros2-learning/src/install/first_robot/sh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 scale=1 1 1
Joints:
- joint camera_joint: origin xyz=0.190 0 0.043 rpy=0 0 0 -> xyz=0.25 0 0.043 rpy=0 0 0
- joint front_left_ankle_joint: origin xyz=0 0 -0.213 rpy=0 0 0 -> xyz=0 0 -0.213 rpy=0 -1.57 0
- joint front_left_foot_joint: origin xyz=0.07527688178772148 0 -0.17067370133261353 rpy=0 0 0 -> xyz=0 0 -0.213 rpy=0 0 0
- joint front_left_knee_joint: origin xyz=0 0.0955 0 rpy=0 0 0 -> xyz=0 0.0955 0 rpy=0 0.45 0
- joint front_right_ankle_joint: origin xyz=0 0 -0.213 rpy=0 0 0 -> xyz=0 0 -0.213 rpy=0 -1.57 0
- joint front_right_foot_joint: origin xyz=0.07527688178772148 0 -0.17067370133261353 rpy=0 0 0 -> xyz=0 0 -0.213 rpy=0 0 0
- joint front_right_knee_joint: origin xyz=0 -0.0955 0 rpy=0 0 0 -> xyz=0 -0.0955 0 rpy=0 0.45 0
- joint laser_joint: origin xyz=0.05 0 0.045 rpy=0 0 0 -> xyz=0 0 0 rpy=0 0 0
- joint rear_left_ankle_joint: origin xyz=0 0 -0.213 rpy=0 0 0 -> xyz=0 0 -0.213 rpy=0 -1.57 0
- joint rear_left_foot_joint: origin xyz=0.07527688178772148 0 -0.17067370133261353 rpy=0 0 0 -> xyz=0 0 -0.213 rpy=0 0 0
- joint rear_left_knee_joint: origin xyz=0 0.0955 0 rpy=0 0 0 -> xyz=0 0.0955 0 rpy=0 0.45 0
- joint rear_right_ankle_joint: origin xyz=0 0 -0.213 rpy=0 0 0 -> xyz=0 0 -0.213 rpy=0 -1.57 0
- joint rear_right_foot_joint: origin xyz=0.07527688178772148 0 -0.17067370133261353 rpy=0 0 0 -> xyz=0 0 -0.213 rpy=0 0 0
- joint rear_right_knee_joint: origin xyz=0 -0.0955 0 rpy=0 0 0 -> xyz=0 -0.0955 0 rpy=0 0.45 0
