Commit message: temp update

File: src/first_robot/description/constants.xacro (robot description, xacro)
@@ -61,10 +61,10 @@
     <xacro:property name="trunk_com_y" value="0.00"/>
     <xacro:property name="trunk_com_z" value="-0.005366"/>
-    <xacro:property name="trunk_ixx" value="0.02448"/>
-    <xacro:property name="trunk_ixy" value="0.00012166"/>
-    <xacro:property name="trunk_ixz" value="0.0014849"/>
-    <xacro:property name="trunk_iyy" value="0.098077"/>
-    <xacro:property name="trunk_iyz" value="-3.12E-05"/>
-    <xacro:property name="trunk_izz" value="0.107"/>
+    <xacro:property name="trunk_ixx" value="0.0168128557"/>
+    <xacro:property name="trunk_ixy" value="-0.0002296769"/>
+    <xacro:property name="trunk_ixz" value="-0.0002945293"/>
+    <xacro:property name="trunk_iyy" value="0.063009565"/>
+    <xacro:property name="trunk_iyz" value="-4.18731e-05"/>
+    <xacro:property name="trunk_izz" value="0.0716547275"/>
     <!-- simplified collision value -->
     <xacro:property name="trunk_width" value="0.0935"/>
@@ -102,8 +102,8 @@
     <xacro:property name="ankle_offset_z" value="-0.213"/>
     <!-- joint limits -->
-    <xacro:property name="damping" value="0.01"/>
-    <xacro:property name="friction" value="0.2"/>
-    <xacro:property name="hip_position_max" value="1.0472"/>
-    <xacro:property name="hip_position_min" value="-1.0472"/>
+    <xacro:property name="damping" value="0.5"/>
+    <xacro:property name="friction" value="0.1"/>
+    <xacro:property name="hip_position_max" value="0.863"/>
+    <xacro:property name="hip_position_min" value="-0.686"/>
     <xacro:property name="hip_velocity_max" value="30.1"/>
     <xacro:property name="hip_torque_max" value="23.7"/>
@@ -112,6 +112,6 @@
     <xacro:property name="knee_velocity_max" value="30.1"/>
     <xacro:property name="knee_torque_max" value="23.7"/>
-    <xacro:property name="ankle_position_max" value="1.0"/>
-    <xacro:property name="ankle_position_min" value="-1.0"/>
+    <xacro:property name="ankle_position_max" value="-0.888"/>
+    <xacro:property name="ankle_position_min" value="-2.818"/>
     <xacro:property name="ankle_velocity_max" value="20.06"/>
     <xacro:property name="ankle_torque_max" value="35.55"/>

File: src/first_robot/description/gz_control.xacro (robot description, xacro)
@@ -9,4 +9,5 @@
     <xacro:macro name="define_joint_interfaces" params="joint_name">
       <joint name="${joint_name}">
+        <command_interface name="effort" />
         <command_interface name="position" />
         <state_interface name="position" />

File: src/first_robot/description/leg_block_v3.xacro (robot description, xacro)
@@ -47,5 +47,5 @@
       </inertial>
     </link>
-    <joint name="${prefix}_hip_joint" description="Hip joint side ${side} and pos ${pos}"
+    <joint name="${prefix}_hip_joint" initial_position="0.0" description="Hip joint side ${side} and pos ${pos}"
       type="revolute">
       <parent link="trunk" />
@@ -105,5 +105,5 @@
     </link>
     <!-- knee Joint  Đùi  quay về sau  -->
-    <joint name="${prefix}_knee_joint" description="Knee joint side ${side} and pos ${pos}"
+    <joint name="${prefix}_knee_joint" initial_position="0.5" description="Knee joint side ${side} and pos ${pos}"
       type="revolute">
       <origin rpy="0 0.45 0" xyz="0 ${knee_offset*-side} 0" />
@@ -113,5 +113,5 @@
       <axis xyz="0 1 0" />
       <dynamics damping="${damping}" friction="${friction}" />
-      <limit lower="-1.57" upper="1.57" effort="30" velocity="7.0" />
+      <!-- <limit lower="-1.57" upper="1.57" effort="30" velocity="7.0" /> -->
       <limit effort="${knee_torque_max}" velocity="${knee_velocity_max}"
         lower="${knee_position_min}" upper="${knee_position_max}" />
@@ -144,6 +144,6 @@
     </link>
     <!-- ankle Joint  Cẳng chân  quay về trước 45  -->
-    <joint name="${prefix}_ankle_joint" type="revolute">
-      <origin rpy="0 -0.8 0" xyz="0 0 ${-ankle_length}" />
+    <joint name="${prefix}_ankle_joint" initial_position="-1.0" type="revolute">
+      <origin rpy="0 -0.90 0" xyz="0 0 ${-ankle_length}" />
       <parent link="${prefix}_knee_link" />
       <child link="${prefix}_ankle_link" />

File: src/first_robot/description/robot_core.xacro (robot description, xacro)
@@ -6,5 +6,5 @@
       <origin rpy="0 0 0" xyz="0 0 0" />
       <geometry>
-        <box size="0.001 0.001 0.001" />
+        <box size="0.3762 0.0935 0.114" />
       </geometry>
       <material name="white" />
@@ -12,5 +12,5 @@
     <inertial>
       <origin xyz="0 0 0" />
-      <mass value="0.1" />
+      <mass value="2.2" />
       <inertia ixx="0.001" iyy="0.001" izz="0.001" ixy="0" ixz="0" iyz="0" />
     </inertial>
@@ -19,5 +19,5 @@
     <parent link="base_link" />
     <child link="trunk" />
-    <origin xyz="0 0 0" rpy="0 0 0" />
+    <origin xyz="-0.021112 0 0" rpy="0 0 0" />
   </joint>
   <!-- Trunk  Thân robot -->

File: src/robot.urdf (robot description, URDF)
Before this commit: robot my_robot, 21 links, 20 joints
Links:
- link trunk: mass 4.921 -> 2.2
Joints:
- joint front_left_ankle_joint: limit lower=-1.0 upper=1.0 effort=35.55 velocity=20.06 -> lower=-2.818 upper=-0.888 effort=35.55 velocity=20.06; origin xyz=0 0 -0.213 rpy=0 -1.57 0 -> xyz=0 0 -0.213 rpy=0 -0.90 0
- joint front_left_hip_joint: limit lower=-1.0472 upper=1.0472 effort=23.7 velocity=30.1 -> lower=-0.686 upper=0.863 effort=23.7 velocity=30.1
- joint front_left_knee_joint: limit lower=-1.57 upper=1.57 effort=30 velocity=7.0 -> lower=-1.5708 upper=3.4907 effort=23.7 velocity=30.1
- joint front_right_ankle_joint: limit lower=-1.0 upper=1.0 effort=35.55 velocity=20.06 -> lower=-2.818 upper=-0.888 effort=35.55 velocity=20.06; origin xyz=0 0 -0.213 rpy=0 -1.57 0 -> xyz=0 0 -0.213 rpy=0 -0.90 0
- joint front_right_hip_joint: limit lower=-1.0472 upper=1.0472 effort=23.7 velocity=30.1 -> lower=-0.686 upper=0.863 effort=23.7 velocity=30.1
- joint front_right_knee_joint: limit lower=-1.57 upper=1.57 effort=30 velocity=7.0 -> lower=-1.5708 upper=3.4907 effort=23.7 velocity=30.1
- joint rear_left_ankle_joint: limit lower=-1.0 upper=1.0 effort=35.55 velocity=20.06 -> lower=-2.818 upper=-0.888 effort=35.55 velocity=20.06; origin xyz=0 0 -0.213 rpy=0 -1.57 0 -> xyz=0 0 -0.213 rpy=0 -0.90 0
- joint rear_left_hip_joint: limit lower=-1.0472 upper=1.0472 effort=23.7 velocity=30.1 -> lower=-0.686 upper=0.863 effort=23.7 velocity=30.1
- joint rear_left_knee_joint: limit lower=-1.57 upper=1.57 effort=30 velocity=7.0 -> lower=-1.5708 upper=3.4907 effort=23.7 velocity=30.1
- joint rear_right_ankle_joint: limit lower=-1.0 upper=1.0 effort=35.55 velocity=20.06 -> lower=-2.818 upper=-0.888 effort=35.55 velocity=20.06; origin xyz=0 0 -0.213 rpy=0 -1.57 0 -> xyz=0 0 -0.213 rpy=0 -0.90 0
- joint rear_right_hip_joint: limit lower=-1.0472 upper=1.0472 effort=23.7 velocity=30.1 -> lower=-0.686 upper=0.863 effort=23.7 velocity=30.1
- joint rear_right_knee_joint: limit lower=-1.57 upper=1.57 effort=30 velocity=7.0 -> lower=-1.5708 upper=3.4907 effort=23.7 velocity=30.1

Commit message: little  update

File: src/first_robot/description/constants.xacro (robot description, xacro)
@@ -118,5 +118,5 @@
     <!-- dynamics inertial value -->
     <!-- trunk -->
-    <xacro:property name="trunk_mass" value="2.2"/>
+    <xacro:property name="trunk_mass" value="4.2"/>
     <xacro:property name="trunk_com_x" value="0.021112"/>
     <xacro:property name="trunk_com_y" value="0.00"/>
@@ -129,5 +129,5 @@
     <xacro:property name="trunk_izz" value="0.107"/>
     <!-- hip (left front) -->
-    <xacro:property name="hip_mass" value="0.678"/>
+    <xacro:property name="hip_mass" value="0.478"/>
     <xacro:property name="hip_com_x" value="-0.0054"/>
     <xacro:property name="hip_com_y" value="0.00194"/>
@@ -140,5 +140,5 @@
     <xacro:property name="hip_izz" value="0.000596"/>
     <!-- knee -->
-    <xacro:property name="knee_mass" value="0.135862"/>
+    <xacro:property name="knee_mass" value="0.435862"/>
     <xacro:property name="knee_com_x" value="-0.00374"/>
     <xacro:property name="knee_com_y" value="-0.0223"/>
