Commit message: update champ config

File: src/first_robot/description/leg_block_v3.xacro (robot description, xacro)
@@ -47,5 +47,6 @@
       </inertial>
     </link>
-    <joint name="${prefix}_hip_joint" initial_position="0.0" description="Hip joint side ${side} and pos ${pos}"
+    <joint name="${prefix}_hip_joint" initial_position="0.0"
+      description="Hip joint side ${side} and pos ${pos}"
       type="revolute">
       <parent link="trunk" />
@@ -105,7 +106,8 @@
     </link>
     <!-- knee Joint  Đùi  quay về sau  -->
-    <joint name="${prefix}_knee_joint" initial_position="0.5" description="Knee joint side ${side} and pos ${pos}"
+    <joint name="${prefix}_knee_joint" initial_position="0.0"
+      description="Knee joint side ${side} and pos ${pos}"
       type="revolute">
-      <origin rpy="0 0.45 0" xyz="0 ${knee_offset*-side} 0" />
+      <origin rpy="0 0 0" xyz="0 ${knee_offset*-side} 0" />
       <parent link="${prefix}_hip_link" />
       <!-- Gắn vào motor háng mô phỏng -->
@@ -144,6 +146,6 @@
     </link>
     <!-- ankle Joint  Cẳng chân  quay về trước 45  -->
-    <joint name="${prefix}_ankle_joint" initial_position="-1.0" type="revolute">
-      <origin rpy="0 -0.6 0" xyz="0 0 ${-ankle_length}" />
+    <joint name="${prefix}_ankle_joint" initial_position="0.0" type="revolute">
+      <origin rpy="0 0 0" xyz="0 0 ${-ankle_length}" />
       <parent link="${prefix}_knee_link" />
       <child link="${prefix}_ankle_link" />
@@ -152,4 +154,26 @@
       <limit effort="${ankle_torque_max}" velocity="${ankle_velocity_max}"
         lower="${ankle_position_min}" upper="${ankle_position_max}" />
+      <gazebo>
+        <plugin name="${prefix}_ankle_controller" filename="libgazebo_ros_joint_position_controller.so">
+          <robotNamespace>/first_robot</robotNamespace>
+          <jointName>${prefix}_ankle_joint</jointName>
+          <commandTopic>/${prefix}_ankle_controller/command</commandTopic>
+          <updateRate>30</updateRate>
+          <pid>
+            <p>100.0</p>
+            <i>0.0</i>
+            <d>10.0</d>
+          </pid>
+        </plugin>
+        <!-- Plugin cảm biến lực mô phỏng -->
+        <plugin name="${prefix}_force_torque_sensor" filename="libgazebo_ros_force_torque_sensor.so">
+          <robotNamespace>/first_robot</robotNamespace>
+          <jointName>${prefix}_ankle_joint</jointName>
+          <topicName>/${prefix}_force_torque_sensor</topicName>
+        </plugin>
+      </gazebo>
+      <sensor name="${prefix}_force_torque" type="force_torque">
+        <update_rate>30</update_rate>
+      </sensor>
     </joint>
     <!-- *** Kết thúc phần cẳng chân *** -->

Commit message: update new model

File: src/first_robot/description/leg_block_v3.xacro (robot description, xacro)
@@ -43,11 +43,8 @@
         <origin rpy="0 0 0" xyz="${hip_com_x*pos} ${hip_com_y*side} ${hip_com_z}" />
         <mass value="${hip_mass}" />
-        <inertia ixx="${hip_ixx}" ixy="${hip_ixy*side*pos}" ixz="${hip_ixz*pos}" iyy="${hip_iyy}"
-          iyz="${hip_iyz*side}" izz="${hip_izz}" />
-      </inertial>
-    </link>
-    <joint name="${prefix}_hip_joint" initial_position="0.0"
-      description="Hip joint side ${side} and pos ${pos}"
-      type="revolute">
+        <inertia ixx="${hip_ixx}" ixy="${hip_ixy*side*pos}" ixz="${hip_ixz*pos}" iyy="${hip_iyy}" iyz="${hip_iyz*side}" izz="${hip_izz}" />
+      </inertial>
+    </link>
+    <joint name="${prefix}_hip_joint" initial_position="0.0" description="Hip joint side ${side} and pos ${pos}" type="revolute">
       <parent link="trunk" />
       <child link="${prefix}_hip_link" />
@@ -70,6 +67,5 @@
       <axis xyz="1 0 0" />
       <dynamics damping="${damping}" friction="${friction}" />
-      <limit effort="${hip_torque_max}" velocity="${hip_velocity_max}" lower="${hip_position_min}"
-        upper="${hip_position_max}" />
+      <limit effort="${hip_torque_max}" velocity="${hip_velocity_max}" lower="${hip_position_min}" upper="${hip_position_max}" />
       <!-- Vị trí gắn khớp háng vào body-->
     </joint>
@@ -82,9 +78,9 @@
           <!-- <box size="${knee_length} ${knee_width} ${knee_height}"/> -->
           <xacro:if value="${(side == 1) }">
-            <mesh filename="file://$(find first_robot)/meshes/knee_mirror.dae" scale="1 1 1" />
+            <mesh filename="file://$(find first_robot)/meshes/knee_mirror_new.dae" scale="1 1 1" />
             <!-- <origin rpy="${PI/2.0} 2.0 0" xyz="0 0 0"/> -->
           </xacro:if>
           <xacro:if value="${(side == -1) }">
-            <mesh filename="file://$(find first_robot)/meshes/knee.dae" scale="1 1 1" />
+            <mesh filename="file://$(find first_robot)/meshes/knee_new.dae" scale="1 1 1" />
             <!-- <origin rpy="${PI/2.0} 2.0 0" xyz="0 0 0"/> -->
           </xacro:if>
@@ -101,12 +97,9 @@
         <origin rpy="0 0 0" xyz="${knee_com_x} ${knee_com_y*-side} ${knee_com_z}" />
         <mass value="${knee_mass}" />
-        <inertia ixx="${knee_ixx}" ixy="${knee_ixy*-side}" ixz="${knee_ixz}" iyy="${knee_iyy}"
-          iyz="${knee_iyz*-side}" izz="${knee_izz}" />
+        <inertia ixx="${knee_ixx}" ixy="${knee_ixy*-side}" ixz="${knee_ixz}" iyy="${knee_iyy}" iyz="${knee_iyz*-side}" izz="${knee_izz}" />
       </inertial>
     </link>
     <!-- knee Joint  Đùi  quay về sau  -->
-    <joint name="${prefix}_knee_joint" initial_position="0.0"
-      description="Knee joint side ${side} and pos ${pos}"
-      type="revolute">
+    <joint name="${prefix}_knee_joint" initial_position="0.0" description="Knee joint side ${side} and pos ${pos}" type="revolute">
       <origin rpy="0 0 0" xyz="0 ${knee_offset*-side} 0" />
       <parent link="${prefix}_hip_link" />
@@ -116,6 +109,5 @@
       <dynamics damping="${damping}" friction="${friction}" />
       <!-- <limit lower="-1.57" upper="1.57" effort="30" velocity="7.0" /> -->
-      <limit effort="${knee_torque_max}" velocity="${knee_velocity_max}"
-        lower="${knee_position_min}" upper="${knee_position_max}" />
+      <limit effort="${knee_torque_max}" velocity="${knee_velocity_max}" lower="${knee_position_min}" upper="${knee_position_max}" />
     </joint>
     <!-- *** Kết thúc phần đùi chân *** -->
@@ -127,5 +119,13 @@
         <geometry>
           <!-- <box size="${ankle_length} ${ankle_width} ${ankle_height}"/> -->
-          <mesh filename="file://$(find first_robot)/meshes/ankle.dae" scale="1 1 1" />
+          <mesh filename="file://$(find first_robot)/meshes/ankle_new.dae" scale="1 1 1" />
+          <xacro:if value="${(side == 1) }">
+            <mesh filename="file://$(find first_robot)/meshes/ankle_new.dae" scale="1 1 1" />
+            <!-- <origin rpy="${PI/2.0} 2.0 0" xyz="0 0 0"/> -->
+          </xacro:if>
+          <xacro:if value="${(side == -1) }">
+            <mesh filename="file://$(find first_robot)/meshes/ankle_mirror_new.dae" scale="1 1 1" />
+            <!-- <origin rpy="${PI/2.0} 2.0 0" xyz="0 0 0"/> -->
+          </xacro:if>
         </geometry>
         <!-- Màu tím -->
@@ -141,6 +141,5 @@
         <origin rpy="0 0 0" xyz="${ankle_com_x} ${ankle_com_y} ${ankle_com_z}" />
         <mass value="${ankle_mass}" />
-        <inertia ixx="${ankle_ixx}" ixy="${ankle_ixy}" ixz="${ankle_ixz}" iyy="${ankle_iyy}"
-          iyz="${ankle_iyz}" izz="${ankle_izz}" />
+        <inertia ixx="${ankle_ixx}" ixy="${ankle_ixy}" ixz="${ankle_ixz}" iyy="${ankle_iyy}" iyz="${ankle_iyz}" izz="${ankle_izz}" />
       </inertial>
     </link>
@@ -152,6 +151,5 @@
       <axis xyz="0 1 0" />
       <dynamics damping="${damping}" friction="${friction}" />
-      <limit effort="${ankle_torque_max}" velocity="${ankle_velocity_max}"
-        lower="${ankle_position_min}" upper="${ankle_position_max}" />
+      <limit effort="${ankle_torque_max}" velocity="${ankle_velocity_max}" lower="${ankle_position_min}" upper="${ankle_position_max}" />
       <gazebo>
         <plugin name="${prefix}_ankle_controller" filename="libgazebo_ros_joint_position_controller.so">
@@ -197,7 +195,5 @@
       <inertial>
         <mass value="${foot_mass}" />
-        <inertia ixx="${(2*foot_mass)/5.0*(foot_radius*foot_radius)}" ixy="0.0" ixz="0.0"
-          iyy="${(2*foot_mass)/5.0*(foot_radius*foot_radius)}" iyz="0.0"
-          izz="${(2*foot_mass)/5.0*(foot_radius*foot_radius)}" />
+        <inertia ixx="${(2*foot_mass)/5.0*(foot_radius*foot_radius)}" ixy="0.0" ixz="0.0" iyy="${(2*foot_mass)/5.0*(foot_radius*foot_radius)}" iyz="0.0" izz="${(2*foot_mass)/5.0*(foot_radius*foot_radius)}" />
       </inertial>
     </link>

File: src/first_robot/description/robot_core.xacro (robot description, xacro)
@@ -6,5 +6,5 @@
       <origin rpy="0 0 0" xyz="0 0 0" />
       <geometry>
-        <box size="0.3762 0.0935 0.114" />
+        <box size="0.3762 0.02 0.05" />
       </geometry>
       <material name="white" />
@@ -27,5 +27,5 @@
       <geometry>
         <!-- <box size="${trunk_length} ${trunk_width} ${trunk_height}"/> -->
-        <mesh filename="file://$(find first_robot)/meshes/trunk.dae" scale="1 1 1" />
+        <mesh filename="file://$(find first_robot)/meshes/trunk_new.dae" scale="1 1 1" />
       </geometry>
       <material name="silver" />

Commit message: refactor meshs

File: src/first_robot/description/leg_block_v3.xacro (robot description, xacro)
@@ -32,5 +32,5 @@
           <!-- dài 2cm  cố định thân trên và các chân -->
         </geometry>
-        <material name="blue" />
+        <!-- <material name="blue" /> -->
       </visual>
       <collision name="${prefix}_hip_collision">
@@ -78,9 +78,9 @@
           <!-- <box size="${knee_length} ${knee_width} ${knee_height}"/> -->
           <xacro:if value="${(side == 1) }">
-            <mesh filename="file://$(find first_robot)/meshes/knee_mirror_new.dae" scale="1 1 1" />
+            <mesh filename="file://$(find first_robot)/meshes/knee_left.dae" scale="1 1 1" />
             <!-- <origin rpy="${PI/2.0} 2.0 0" xyz="0 0 0"/> -->
           </xacro:if>
           <xacro:if value="${(side == -1) }">
-            <mesh filename="file://$(find first_robot)/meshes/knee_new.dae" scale="1 1 1" />
+            <mesh filename="file://$(find first_robot)/meshes/knee_right.dae" scale="1 1 1" />
             <!-- <origin rpy="${PI/2.0} 2.0 0" xyz="0 0 0"/> -->
           </xacro:if>
@@ -119,16 +119,14 @@
         <geometry>
           <!-- <box size="${ankle_length} ${ankle_width} ${ankle_height}"/> -->
-          <mesh filename="file://$(find first_robot)/meshes/ankle_new.dae" scale="1 1 1" />
           <xacro:if value="${(side == 1) }">
-            <mesh filename="file://$(find first_robot)/meshes/ankle_new.dae" scale="1 1 1" />
+            <mesh  filename="file://$(find first_robot)/meshes/ankle_left.dae" scale="1 1 1" />
             <!-- <origin rpy="${PI/2.0} 2.0 0" xyz="0 0 0"/> -->
           </xacro:if>
           <xacro:if value="${(side == -1) }">
-            <mesh filename="file://$(find first_robot)/meshes/ankle_mirror_new.dae" scale="1 1 1" />
-            <!-- <origin rpy="${PI/2.0} 2.0 0" xyz="0 0 0"/> -->
+            <mesh filename="file://$(find first_robot)/meshes/ankle_right.dae" scale="1 1 1" />
           </xacro:if>
         </geometry>
         <!-- Màu tím -->
-        <material name="purple" />
+        <!-- <material name="purple" /> -->
       </visual>
       <collision name="${prefix}_ankle_collision">

File: src/first_robot/description/robot_core.xacro (robot description, xacro)
@@ -29,5 +29,5 @@
         <mesh filename="file://$(find first_robot)/meshes/trunk_new.dae" scale="1 1 1" />
       </geometry>
-      <material name="silver" />
+      <!-- <material name="silver" /> -->
     </visual>
     <collision name="trunk_collision">
