Commit message: update readme

File: src/robot.urdf (robot description, URDF)
Before this commit: robot my_robot, 21 links, 20 joints
Links:
- link base_link: mass 0.1 -> 2.2; geometry visual box size=0.3762 0.02 0.05
- link front_left_hip_link: mass 0.678 -> 0.478
- link front_left_knee_link: mass 0.135862 -> 0.435862
- link front_right_hip_link: mass 0.678 -> 0.478
- link front_right_knee_link: mass 0.135862 -> 0.435862
- link rear_left_hip_link: mass 0.678 -> 0.478
- link rear_left_knee_link: mass 0.135862 -> 0.435862
- link rear_right_hip_link: mass 0.678 -> 0.478
- link rear_right_knee_link: mass 0.135862 -> 0.435862
- link trunk: mass 2.2 -> 4.2
Joints:
- joint floating_base: origin xyz=0 0 0 rpy=0 0 0 -> xyz=-0.021112 0 0 rpy=0 0 0
- joint front_left_ankle_joint: origin xyz=0 0 -0.213 rpy=0 -0.90 0 -> xyz=0 0 -0.213 rpy=0 0 0
- joint front_left_knee_joint: origin xyz=0 0.0955 0 rpy=0 0.45 0 -> xyz=0 0.0955 0 rpy=0 0 0
- joint front_right_ankle_joint: origin xyz=0 0 -0.213 rpy=0 -0.90 0 -> xyz=0 0 -0.213 rpy=0 0 0
- joint front_right_knee_joint: origin xyz=0 -0.0955 0 rpy=0 0.45 0 -> xyz=0 -0.0955 0 rpy=0 0 0
- joint rear_left_ankle_joint: origin xyz=0 0 -0.213 rpy=0 -0.90 0 -> xyz=0 0 -0.213 rpy=0 0 0
- joint rear_left_knee_joint: origin xyz=0 0.0955 0 rpy=0 0.45 0 -> xyz=0 0.0955 0 rpy=0 0 0
- joint rear_right_ankle_joint: origin xyz=0 0 -0.213 rpy=0 -0.90 0 -> xyz=0 0 -0.213 rpy=0 0 0
- joint rear_right_knee_joint: origin xyz=0 -0.0955 0 rpy=0 0.45 0 -> xyz=0 -0.0955 0 rpy=0 0 0
