Commit message: add moveit assistant support

File: src/second_robot/description/gz_control.xacro (robot description, xacro)
@@ -6,5 +6,6 @@
   <ros2_control name="SecondRobot" type="system">
     <hardware>
-      <plugin>gz_ros2_control/GazeboSimSystem</plugin>
+      <!-- <plugin>gz_ros2_control/GazeboSimSystem</plugin> -->
+      <plugin>mock_components/GenericSystem</plugin>
     </hardware>
     <!-- Joint Definitions -->

File: src/second_robot/description/robot_core.xacro (robot description, xacro)
@@ -37,4 +37,10 @@
       <material name="gray" />
     </visual>
+    <collision>
+      <geometry>
+        <sphere radius="0.025" />
+      </geometry>
+      <origin xyz="0 0 0" rpy="0 0 0" />
+    </collision>
     <inertial>
       <origin xyz="0 0 0" />
@@ -51,4 +57,5 @@
     <limit lower="-3.14" upper="3.14" effort="1.0" velocity="2.0" />
   </joint>
+  <!-- Upper Arm Link -->
   <link name="upper_arm_link">
     <visual>
@@ -56,11 +63,17 @@
         <cylinder length="${link_length}" radius="${link_radius}" />
       </geometry>
-      <origin xyz="${link_length/2} 0 0" rpy="0 0 0" />
+      <origin xyz="0 0 ${link_length/2}" rpy="0 0 0" />
       <material name="blue">
         <color rgba="0 0 1 1" />
       </material>
     </visual>
+    <collision>
+      <geometry>
+        <cylinder length="${link_length}" radius="${link_radius}" />
+      </geometry>
+      <origin xyz="0 0 ${link_length/2}" rpy="0 0 0" />
+    </collision>
     <inertial>
-      <origin xyz="${link_length/2} 0 0" />
+      <origin xyz="0 0 ${link_length/2}" rpy="0 0 0" />
       <mass value="0.15" />
       <inertia ixx="0.00012" iyy="0.00012" izz="0.00002" ixy="0" ixz="0" iyz="0" />
@@ -71,8 +84,9 @@
     <parent link="upper_arm_link" />
     <child link="forearm_link" />
-    <origin xyz="${link_length} 0 0" rpy="0 0 0" />
+    <origin xyz="0 0 ${link_length}" rpy="0 0 0" />
     <axis xyz="0 0 1" />
     <limit lower="-3.14" upper="3.14" effort="1.0" velocity="2.0" />
   </joint>
+  <!-- Forearm Link -->
   <link name="forearm_link">
     <visual>
@@ -80,11 +94,17 @@
         <cylinder length="${link_length}" radius="${link_radius}" />
       </geometry>
-      <origin xyz="${link_length/2} 0 0" rpy="0 0 0" />
+      <origin xyz="0 0 ${link_length/2}" rpy="0 0 0" />
       <material name="green">
         <color rgba="0 1 0 1" />
       </material>
     </visual>
+    <collision>
+      <geometry>
+        <cylinder length="${link_length}" radius="${link_radius}" />
+      </geometry>
+      <origin xyz="0 0 ${link_length/2}" rpy="0 0 0" />
+    </collision>
     <inertial>
-      <origin xyz="${link_length/2} 0 0" />
+      <origin xyz="0 0 ${link_length/2}" rpy="0 0 0" />
       <mass value="0.12" />
       <inertia ixx="0.00010" iyy="0.00010" izz="0.000015" ixy="0" ixz="0" iyz="0" />
@@ -95,8 +115,9 @@
     <parent link="forearm_link" />
     <child link="wrist_link" />
-    <origin xyz="${link_length} 0 0" rpy="0 0 0" />
+    <origin xyz="0 0 ${link_length}" rpy="0 0 0" />
     <axis xyz="0 0 1" />
     <limit lower="-3.14" upper="3.14" effort="1.0" velocity="2.0" />
   </joint>
+  <!-- Wrist Link -->
   <link name="wrist_link">
     <visual>
@@ -104,11 +125,17 @@
         <cylinder length="${link_length}" radius="${link_radius}" />
       </geometry>
-      <origin xyz="${link_length/2} 0 0" rpy="0 0 0" />
+      <origin xyz="0 0 ${link_length/2}" rpy="0 0 0" />
       <material name="red">
         <color rgba="1 0 0 1" />
       </material>
     </visual>
+    <collision>
+      <geometry>
+        <cylinder length="${link_length}" radius="${link_radius}" />
+      </geometry>
+      <origin xyz="0 0 ${link_length/2}" rpy="0 0 0" />
+    </collision>
     <inertial>
-      <origin xyz="${link_length/2} 0 0" />
+      <origin xyz="0 0 ${link_length/2}" rpy="0 0 0" />
       <mass value="0.08" />
       <inertia ixx="0.00007" iyy="0.00007" izz="0.00001" ixy="0" ixz="0" iyz="0" />
@@ -126,4 +153,10 @@
       </material>
     </visual>
+    <collision>
+      <geometry>
+        <sphere radius="0.015" />
+      </geometry>
+      <origin xyz="0 0 0" rpy="0 0 0" />
+    </collision>
     <inertial>
       <origin xyz="0 0 0" />
@@ -132,8 +165,9 @@
     </inertial>
   </link>
+  <!-- End Effector Joint -->
   <joint name="ee_fixed_joint" type="fixed">
     <parent link="wrist_link" />
     <child link="end_effector_link" />
-    <origin xyz="${link_length} 0 0" rpy="0 0 0" />
+    <origin xyz="0 0 ${link_length}" rpy="0 0 0" />
   </joint>
 </robot>

Commit message: initial moveit2

File: src/second_robot/description/gz_control.xacro (robot description, xacro)
@@ -8,11 +8,15 @@
       <plugin>gz_ros2_control/GazeboSimSystem</plugin>
       <!-- <plugin>mock_components/GenericSystem</plugin> -->
+      <!-- <plugin>gazebo_ros2_control/GazeboSystem</plugin> -->
     </hardware>
     <!-- Joint Definitions -->
     <xacro:macro name="define_joint_interfaces" params="joint_name">
       <joint name="${joint_name}">
-        <command_interface name="effort" />
-        <state_interface name="position" />
-        <state_interface name="velocity" />
+        <command_interface name="position">
+          <param name="min">-1</param>
+          <param name="max">1</param>
+        </command_interface>
+        <state_interface name="position"/>
+        <state_interface name="velocity"/>
       </joint>
     </xacro:macro>
@@ -25,5 +29,5 @@
     <plugin filename="gz_ros2_control-system" name="gz_ros2_control::GazeboSimROS2ControlPlugin">
       <parameters>$(find second_robot)/config/ros_control.yaml</parameters>
-       <robot_param_node>robot_state_publisher</robot_param_node>
+      <robot_param_node>robot_state_publisher</robot_param_node>
     </plugin>
   </gazebo>

File: src/second_robot/description/robot_core.xacro (robot description, xacro)
@@ -27,4 +27,5 @@
     <child link="shoulder_link" />
     <origin xyz="0 0 0" rpy="0 0 0" />
+    <limit lower="-2.0" upper="2.0" effort="5.0" velocity="1.0"/>
   </joint>
   <!-- Shoulder Link -->
@@ -171,3 +172,33 @@
     <origin xyz="0 0 ${link_length}" rpy="0 0 0" />
   </joint>
+<transmission name="trans_shoulder">
+  <type>transmission_interface/SimpleTransmission</type>
+  <joint name="shoulder_joint">
+    <hardwareInterface>hardware_interface/PositionJointInterface</hardwareInterface>
+  </joint>
+  <actuator name="shoulder_motor">
+    <hardwareInterface>hardware_interface/PositionJointInterface</hardwareInterface>
+    <mechanicalReduction>1</mechanicalReduction>
+  </actuator>
+</transmission>
+<transmission name="trans_elbow">
+  <type>transmission_interface/SimpleTransmission</type>
+  <joint name="elbow_joint">
+    <hardwareInterface>hardware_interface/PositionJointInterface</hardwareInterface>
+  </joint>
+  <actuator name="elbow_motor">
+    <hardwareInterface>hardware_interface/PositionJointInterface</hardwareInterface>
+    <mechanicalReduction>1</mechanicalReduction>
+  </actuator>
+</transmission>
+<transmission name="trans_wrist">
+  <type>transmission_interface/SimpleTransmission</type>
+  <joint name="wrist_joint">
+    <hardwareInterface>hardware_interface/PositionJointInterface</hardwareInterface>
+  </joint>
+  <actuator name="wrist_motor">
+    <hardwareInterface>hardware_interface/PositionJointInterface</hardwareInterface>
+    <mechanicalReduction>1</mechanicalReduction>
+  </actuator>
+</transmission>
 </robot>

Commit message: update moveit2 work basically

File: src/second_robot/description/gz_control.xacro (robot description, xacro)
@@ -32,3 +32,9 @@
     </plugin>
   </gazebo>
+  <gazebo reference="base_link">
+    <static>true</static>
+  </gazebo>
+   <gazebo reference="shoulder_link">
+    <static>true</static>
+  </gazebo>
 </robot>

File: src/second_robot/description/robot_core.xacro (robot description, xacro)
@@ -1,4 +1,13 @@
 <?xml version="1.0"?>
 <robot xmlns:xacro="http://www.ros.org/wiki/xacro">
+  <!-- Thêm biến xacro cho kích thước giống tay người -->
+  <xacro:property name="link_length" value="0.30" />    <!-- upper arm -->
+  <xacro:property name="forearm_length" value="0.25" /> <!-- forearm -->
+  <xacro:property name="wrist_length" value="0.125" />   <!-- wrist -->
+  <xacro:property name="link_radius" value="0.04" />
+  <!-- Góc khởi tạo khớp -->
+  <xacro:property name="shoulder_init" value="${0.785}" /> <!-- 45 độ -->
+  <xacro:property name="elbow_init" value="${1.57}" />     <!-- 90 độ -->
+  <xacro:property name="wrist_init" value="0" />
   <!-- Base Link -->
   <link name="base_link">
@@ -27,5 +36,5 @@
     <child link="shoulder_link" />
     <origin xyz="0 0 0" rpy="0 0 0" />
-    <limit lower="-2.0" upper="2.0" effort="5.0" velocity="1.0"/>
+    <limit lower="-2.0" upper="2.0" effort="5.0" velocity="1.0" />
   </joint>
   <!-- Shoulder Link -->
@@ -54,6 +63,6 @@
     <parent link="shoulder_link" />
     <child link="upper_arm_link" />
-    <origin xyz="0 0 0" rpy="0 0 0" />
-    <axis xyz="0 0 1" />
+    <origin xyz="0 0 0" rpy="0 0 ${shoulder_init}" />
+    <axis xyz="0 1 0" />
     <limit lower="-3.14" upper="3.14" effort="1.0" velocity="2.0" />
   </joint>
@@ -85,6 +94,6 @@
     <parent link="upper_arm_link" />
     <child link="forearm_link" />
-    <origin xyz="0 0 ${link_length}" rpy="0 0 0" />
-    <axis xyz="0 0 1" />
+    <origin xyz="0 0 ${link_length}" rpy="0 0 ${elbow_init}" />
+    <axis xyz="0 1 0" />
     <limit lower="-3.14" upper="3.14" effort="1.0" velocity="2.0" />
   </joint>
@@ -93,7 +102,7 @@
     <visual>
       <geometry>
-        <cylinder length="${link_length}" radius="${link_radius}" />
-      </geometry>
-      <origin xyz="0 0 ${link_length/2}" rpy="0 0 0" />
+        <cylinder length="${forearm_length}" radius="${link_radius}" />
+      </geometry>
+      <origin xyz="0 0 ${forearm_length/2}" rpy="0 0 0" />
       <material name="green">
         <color rgba="0 1 0 1" />
@@ -102,10 +111,10 @@
     <collision>
       <geometry>
-        <cylinder length="${link_length}" radius="${link_radius}" />
-      </geometry>
-      <origin xyz="0 0 ${link_length/2}" rpy="0 0 0" />
-    </collision>
-    <inertial>
-      <origin xyz="0 0 ${link_length/2}" rpy="0 0 0" />
+        <cylinder length="${forearm_length}" radius="${link_radius}" />
+      </geometry>
+      <origin xyz="0 0 ${forearm_length/2}" rpy="0 0 0" />
+    </collision>
+    <inertial>
+      <origin xyz="0 0 ${forearm_length/2}" rpy="0 0 0" />
       <mass value="0.12" />
       <inertia ixx="0.00010" iyy="0.00010" izz="0.000015" ixy="0" ixz="0" iyz="0" />
@@ -116,6 +125,6 @@
     <parent link="forearm_link" />
     <child link="wrist_link" />
-    <origin xyz="0 0 ${link_length}" rpy="0 0 0" />
-    <axis xyz="0 0 1" />
+    <origin xyz="0 0 ${forearm_length}" rpy="0 0 ${wrist_init}" />
+    <axis xyz="0 1 0" />
     <limit lower="-3.14" upper="3.14" effort="1.0" velocity="2.0" />
   </joint>
@@ -124,7 +133,7 @@
     <visual>
       <geometry>
-        <cylinder length="${link_length}" radius="${link_radius}" />
-      </geometry>
-      <origin xyz="0 0 ${link_length/2}" rpy="0 0 0" />
+        <cylinder length="${wrist_length}" radius="${link_radius}" />
+      </geometry>
+      <origin xyz="0 0 ${wrist_length/2}" rpy="0 0 0" />
       <material name="red">
         <color rgba="1 0 0 1" />
@@ -133,10 +142,10 @@
     <collision>
       <geometry>
-        <cylinder length="${link_length}" radius="${link_radius}" />
-      </geometry>
-      <origin xyz="0 0 ${link_length/2}" rpy="0 0 0" />
-    </collision>
-    <inertial>
-      <origin xyz="0 0 ${link_length/2}" rpy="0 0 0" />
+        <cylinder length="${wrist_length}" radius="${link_radius}" />
+      </geometry>
+      <origin xyz="0 0 ${wrist_length/2}" rpy="0 0 0" />
+    </collision>
+    <inertial>
+      <origin xyz="0 0 ${wrist_length/2}" rpy="0 0 0" />
       <mass value="0.08" />
       <inertia ixx="0.00007" iyy="0.00007" izz="0.00001" ixy="0" ixz="0" iyz="0" />
@@ -147,5 +156,5 @@
     <visual>
       <geometry>
-        <sphere radius="0.015" />
+        <box size="0.08 0.02 0.01" /> <!-- hình hộp nhỏ, giống lòng bàn tay -->
       </geometry>
       <origin xyz="0 0 0" rpy="0 0 0" />
@@ -156,5 +165,5 @@
     <collision>
       <geometry>
-        <sphere radius="0.015" />
+        <box size="0.08 0.02 0.01" />
       </geometry>
       <origin xyz="0 0 0" rpy="0 0 0" />
@@ -170,35 +179,35 @@
     <parent link="wrist_link" />
     <child link="end_effector_link" />
-    <origin xyz="0 0 ${link_length}" rpy="0 0 0" />
-  </joint>
-<transmission name="trans_shoulder">
-  <type>transmission_interface/SimpleTransmission</type>
-  <joint name="shoulder_joint">
-    <hardwareInterface>hardware_interface/PositionJointInterface</hardwareInterface>
-  </joint>
-  <actuator name="shoulder_motor">
-    <hardwareInterface>hardware_interface/PositionJointInterface</hardwareInterface>
-    <mechanicalReduction>1</mechanicalReduction>
-  </actuator>
-</transmission>
-<transmission name="trans_elbow">
-  <type>transmission_interface/SimpleTransmission</type>
-  <joint name="elbow_joint">
-    <hardwareInterface>hardware_interface/PositionJointInterface</hardwareInterface>
-  </joint>
-  <actuator name="elbow_motor">
-    <hardwareInterface>hardware_interface/PositionJointInterface</hardwareInterface>
-    <mechanicalReduction>1</mechanicalReduction>
-  </actuator>
-</transmission>
-<transmission name="trans_wrist">
-  <type>transmission_interface/SimpleTransmission</type>
-  <joint name="wrist_joint">
-    <hardwareInterface>hardware_interface/PositionJointInterface</hardwareInterface>
-  </joint>
-  <actuator name="wrist_motor">
-    <hardwareInterface>hardware_interface/PositionJointInterface</hardwareInterface>
-    <mechanicalReduction>1</mechanicalReduction>
-  </actuator>
-</transmission>
+    <origin xyz="0 0 ${wrist_length}" rpy="0 0 0" />
+  </joint>
+  <transmission name="trans_shoulder">
+    <type>transmission_interface/SimpleTransmission</type>
+    <joint name="shoulder_joint">
+      <hardwareInterface>hardware_interface/PositionJointInterface</hardwareInterface>
+    </joint>
+    <actuator name="shoulder_motor">
+      <hardwareInterface>hardware_interface/PositionJointInterface</hardwareInterface>
+      <mechanicalReduction>1</mechanicalReduction>
+    </actuator>
+  </transmission>
+  <transmission name="trans_elbow">
+    <type>transmission_interface/SimpleTransmission</type>
+    <joint name="elbow_joint">
+      <hardwareInterface>hardware_interface/PositionJointInterface</hardwareInterface>
+    </joint>
+    <actuator name="elbow_motor">
+      <hardwareInterface>hardware_interface/PositionJointInterface</hardwareInterface>
+      <mechanicalReduction>1</mechanicalReduction>
+    </actuator>
+  </transmission>
+  <transmission name="trans_wrist">
+    <type>transmission_interface/SimpleTransmission</type>
+    <joint name="wrist_joint">
+      <hardwareInterface>hardware_interface/PositionJointInterface</hardwareInterface>
+    </joint>
+    <actuator name="wrist_motor">
+      <hardwareInterface>hardware_interface/PositionJointInterface</hardwareInterface>
+      <mechanicalReduction>1</mechanicalReduction>
+    </actuator>
+  </transmission>
 </robot>
